Commit message: fix: add support in srdf file

File: denso_robot_moveit_config/robots/vs050/srdf/dual_denso_robot_macro.srdf.xacro (robot description, xacro)
@@ -5,5 +5,5 @@
     A URDF file must exist for this robot as well, where the joints and the links that are referenced are defined
 -->
-  <xacro:macro name="denso_robot_srdf" params="name namespace">
+  <xacro:macro name="dual_denso_robot_srdf" params="name">
     <!--GROUPS - Representation of a set of joints and links. This can be useful for specifying DOF to plan for, defining arms, end effectors, etc-->
     <!--LINKS - When a link is specified, the parent joint of that link (if it exists) is automatically included-->
@@ -11,25 +11,42 @@
     <!--CHAINS - When a chain is specified, all the links along the chain (including endpoints) are included in the group. Additionally, all the joints that are parents to included links are also included. This means that joints along the chain and the parent joint of the base link are included in the group-->
     <!--SUBGROUPS - Groups can also be formed by referencing to already defined group names-->
-    <group name="${namespace}arm">
-		<joint name="${namespace}joint_1"/>
-		<joint name="${namespace}joint_2"/>
-		<joint name="${namespace}joint_3"/>
-		<joint name="${namespace}joint_4"/>
-		<joint name="${namespace}joint_5"/>
-		<joint name="${namespace}joint_6"/>
-	</group>
+    <group name="left_arm">
+		  <joint name="left_joint_1"/>
+		  <joint name="left_joint_2"/>
+		  <joint name="left_joint_3"/>
+		  <joint name="left_joint_4"/>
+		  <joint name="left_joint_5"/>
+		  <joint name="left_joint_6"/>
+	  </group>
+    <group name="right_arm">
+		  <joint name="right_joint_1"/>
+		  <joint name="right_joint_2"/>
+		  <joint name="right_joint_3"/>
+		  <joint name="right_joint_4"/>
+		  <joint name="right_joint_5"/>
+		  <joint name="right_joint_6"/>
+	  </group>
     <!--GROUP STATES - Purpose - Define a named state for a particular group, in terms of joint values. This is useful to define states like 'folded arms'-->
     <!--END EFFECTOR - Purpose - Represent information about an end effector.-->
     <!--VIRTUAL JOINT - Purpose - this element defines a virtual joint between a robot link and an external frame of reference (considered fixed with respect to the robot)-->
-    <virtual_joint name="${namespace}fixed_base" type="fixed" parent_frame="world" child_link="${namespace}base_link" />
+    <virtual_joint name="$left_fixed_base" type="fixed" parent_frame="world" child_link="left_base_link" />
+    <virtual_joint name="$right_fixed_base" type="fixed" parent_frame="world" child_link="right_base_link" />
     <!--DISABLE COLLISIONS - By default it is assumed that any link of the robot could potentially come into collision with any other link in the robot. This tag disables collision checking between a specified pair of links. -->
-	<disable_collisions link1="${namespace}J6" link2="${namespace}J3" reason="Never"/>
-	<disable_collisions link1="${namespace}J6" link2="${namespace}J5" reason="Adjacent"/>
-	<disable_collisions link1="${namespace}J1" link2="${namespace}J2" reason="Adjacent"/>
-	<disable_collisions link1="${namespace}J1" link2="${namespace}base_link" reason="Adjacent"/>
-	<disable_collisions link1="${namespace}J2" link2="${namespace}J3" reason="Adjacent"/>
-	<disable_collisions link1="${namespace}J3" link2="${namespace}J4" reason="Adjacent"/>
-	<disable_collisions link1="${namespace}J3" link2="${namespace}J5" reason="Never"/>
-	<disable_collisions link1="${namespace}J4" link2="${namespace}J5" reason="Adjacent"/>
+    <disable_collisions link1="left_J6" link2="left_J3" reason="Never"/>
+    <disable_collisions link1="left_J6" link2="left_J5" reason="Adjacent"/>
+    <disable_collisions link1="left_J1" link2="left_J2" reason="Adjacent"/>
+    <disable_collisions link1="left_J1" link2="left_base_link" reason="Adjacent"/>
+    <disable_collisions link1="left_J2" link2="left_J3" reason="Adjacent"/>
+    <disable_collisions link1="left_J3" link2="left_J4" reason="Adjacent"/>
+    <disable_collisions link1="left_J3" link2="left_J5" reason="Never"/>
+    <disable_collisions link1="left_J4" link2="left_J5" reason="Adjacent"/>
+    <disable_collisions link1="right_J6" link2="right_J3" reason="Never"/>
+    <disable_collisions link1="right_J6" link2="right_J5" reason="Adjacent"/>
+    <disable_collisions link1="right_J1" link2="right_J2" reason="Adjacent"/>
+    <disable_collisions link1="right_J1" link2="right_base_link" reason="Adjacent"/>
+    <disable_collisions link1="right_J2" link2="right_J3" reason="Adjacent"/>
+    <disable_collisions link1="right_J3" link2="right_J4" reason="Adjacent"/>
+    <disable_collisions link1="right_J3" link2="right_J5" reason="Never"/>
+    <disable_collisions link1="right_J4" link2="right_J5" reason="Adjacent"/>
   </xacro:macro>
 </robot>
