Commit message: refactor(srdf): use kinematic chain for arm group definition
- Replace the explicit list of individual joints in the `${namespace}arm` planning group with a single `<chain>` tag spanning from `${namespace}base_link` to `${namespace}tool0`.
- This simplifies the SRDF configuration, makes it less prone to errors, and aligns with MoveIt best practices by leveraging the existing URDF tree structure.

File: denso_robot_moveit_config/robots/vs050/srdf/denso_robot_macro.srdf.xacro (robot description, xacro)
@@ -12,13 +12,5 @@
     <!--SUBGROUPS - Groups can also be formed by referencing to already defined group names-->
     <group name="${namespace}arm">
-      <joint name="${namespace}fixed_base"/>
-      <joint name="${namespace}joint_w"/>
-      <joint name="${namespace}joint_1"/>
-      <joint name="${namespace}joint_2"/>
-      <joint name="${namespace}joint_3"/>
-      <joint name="${namespace}joint_4"/>
-      <joint name="${namespace}joint_5"/>
-      <joint name="${namespace}joint_6"/>
-      <joint name="${namespace}J6-tool0"/>
+      <chain base_link="${namespace}base_link" tip_link="${namespace}tool0" />
     </group>
     <group name="${namespace}end_effector">
