Commit message: refactor: remove nome parameter in SRDFs beaause it's not useful

File: denso_robot_moveit_config/robots/cobotta/srdf/denso_robot_macro.srdf.xacro (robot description, xacro)
@@ -5,5 +5,5 @@
     A URDF file must exist for this robot as well, where the joints and the links that are referenced are defined
 -->
-  <xacro:macro name="denso_robot_srdf" params="name namespace">
+  <xacro:macro name="denso_robot_srdf" params="namespace">
     <!--GROUPS - Representation of a set of joints and links. This can be useful for specifying DOF to plan for, defining arms, end effectors, etc-->
     <!--LINKS - When a link is specified, the parent joint of that link (if it exists) is automatically included-->

File: denso_robot_moveit_config/robots/hsr065a1_n32/srdf/denso_robot_macro.srdf.xacro (robot description, xacro)
@@ -5,5 +5,5 @@
     A URDF file must exist for this robot as well, where the joints and the links that are referenced are defined
 -->
-  <xacro:macro name="denso_robot_srdf" params="name namespace">
+  <xacro:macro name="denso_robot_srdf" params="namespace">
     <!--GROUPS - Representation of a set of joints and links. This can be useful for specifying DOF to plan for, defining arms, end effectors, etc-->
     <!--LINKS - When a link is specified, the parent joint of that link (if it exists) is automatically included-->

File: denso_robot_moveit_config/srdf/denso_robot.srdf.xacro (robot description, xacro)
@@ -6,4 +6,4 @@
   <xacro:arg name="namespace" default="" />
   <xacro:include filename="$(find denso_robot_moveit_config)/robots/$(arg model)/srdf/denso_robot_macro.srdf.xacro"/>
-  <xacro:denso_robot_srdf name="$(arg namespace)$(arg model)" namespace="$(arg namespace)"/>
+  <xacro:denso_robot_srdf namespace="$(arg namespace)"/>
 </robot>

Commit message: refactor: srdf file with support for two arms in multiple models

File: denso_robot_moveit_config/robots/cobotta/srdf/denso_robot_macro.srdf.xacro (robot description, xacro)
@@ -12,10 +12,10 @@
     <!--SUBGROUPS - Groups can also be formed by referencing to already defined group names-->
     <group name="${namespace}arm">
-		<joint name="$(arg namespace)joint_1"/>
-		<joint name="$(arg namespace)joint_2"/>
-		<joint name="$(arg namespace)joint_3"/>
-		<joint name="$(arg namespace)joint_4"/>
-		<joint name="$(arg namespace)joint_5"/>
-		<joint name="$(arg namespace)joint_6"/>
+		<joint name="${namespace}joint_1"/>
+		<joint name="${namespace}joint_2"/>
+		<joint name="${namespace}joint_3"/>
+		<joint name="${namespace}joint_4"/>
+		<joint name="${namespace}joint_5"/>
+		<joint name="${namespace}joint_6"/>
 	</group>
     <!--GROUP STATES - Purpose - Define a named state for a particular group, in terms of joint values. This is useful to define states like 'folded arms'-->
@@ -24,12 +24,12 @@
     <virtual_joint name="${namespace}fixed_base" type="fixed" parent_frame="world" child_link="${namespace}base_link" />
     <!--DISABLE COLLISIONS - By default it is assumed that any link of the robot could potentially come into collision with any other link in the robot. This tag disables collision checking between a specified pair of links. -->
-	<disable_collisions link1="$(arg namespace)J6" link2="$(arg namespace)J3" reason="Never"/>
-	<disable_collisions link1="$(arg namespace)J6" link2="$(arg namespace)J5" reason="Adjacent"/>
-	<disable_collisions link1="$(arg namespace)J1" link2="$(arg namespace)J2" reason="Adjacent"/>
-	<disable_collisions link1="$(arg namespace)J1" link2="$(arg namespace)base_link" reason="Adjacent"/>
-	<disable_collisions link1="$(arg namespace)J2" link2="$(arg namespace)J3" reason="Adjacent"/>
-	<disable_collisions link1="$(arg namespace)J3" link2="$(arg namespace)J4" reason="Adjacent"/>
-	<disable_collisions link1="$(arg namespace)J3" link2="$(arg namespace)J5" reason="Never"/>
-	<disable_collisions link1="$(arg namespace)J4" link2="$(arg namespace)J5" reason="Adjacent"/>
+	<disable_collisions link1="${namespace}J6" link2="${namespace}J3" reason="Never"/>
+	<disable_collisions link1="${namespace}J6" link2="${namespace}J5" reason="Adjacent"/>
+	<disable_collisions link1="${namespace}J1" link2="${namespace}J2" reason="Adjacent"/>
+	<disable_collisions link1="${namespace}J1" link2="${namespace}base_link" reason="Adjacent"/>
+	<disable_collisions link1="${namespace}J2" link2="${namespace}J3" reason="Adjacent"/>
+	<disable_collisions link1="${namespace}J3" link2="${namespace}J4" reason="Adjacent"/>
+	<disable_collisions link1="${namespace}J3" link2="${namespace}J5" reason="Never"/>
+	<disable_collisions link1="${namespace}J4" link2="${namespace}J5" reason="Adjacent"/>
   </xacro:macro>
 </robot>

File: denso_robot_moveit_config/robots/hsr065a1_n32/srdf/denso_robot_macro.srdf.xacro (robot description, xacro)
@@ -12,8 +12,8 @@
     <!--SUBGROUPS - Groups can also be formed by referencing to already defined group names-->
     <group name="${namespace}arm">
-		<joint name="$(arg namespace)joint_1"/>
-		<joint name="$(arg namespace)joint_2"/>
-		<joint name="$(arg namespace)joint_3"/>
-		<joint name="$(arg namespace)joint_4"/>
+		<joint name="${namespace}joint_1"/>
+		<joint name="${namespace}joint_2"/>
+		<joint name="${namespace}joint_3"/>
+		<joint name="${namespace}joint_4"/>
 	</group>
     <!--GROUP STATES - Purpose - Define a named state for a particular group, in terms of joint values. This is useful to define states like 'folded arms'-->
@@ -22,13 +22,13 @@
     <virtual_joint name="${namespace}fixed_base" type="fixed" parent_frame="world" child_link="${namespace}base_link" />
     <!--DISABLE COLLISIONS - By default it is assumed that any link of the robot could potentially come into collision with any other link in the robot. This tag disables collision checking between a specified pair of links. -->
-	<disable_collisions link1="$(arg namespace)J1" link2="$(arg namespace)J2" reason="Adjacent"/>
-	<disable_collisions link1="$(arg namespace)J1" link2="$(arg namespace)J3" reason="Never"/>
-	<disable_collisions link1="$(arg namespace)J1" link2="$(arg namespace)J4" reason="Never"/>
-	<disable_collisions link1="$(arg namespace)J1" link2="$(arg namespace)base_link" reason="Adjacent"/>
-	<disable_collisions link1="$(arg namespace)J2" link2="$(arg namespace)J3" reason="Adjacent"/>
-	<disable_collisions link1="$(arg namespace)J2" link2="$(arg namespace)J4" reason="Never"/>
-	<disable_collisions link1="$(arg namespace)J2" link2="$(arg namespace)base_link" reason="Never"/>
-	<disable_collisions link1="$(arg namespace)J3" link2="$(arg namespace)J4" reason="Adjacent"/>
-	<disable_collisions link1="$(arg namespace)J4" link2="$(arg namespace)base_link" reason="Never"/>
+	<disable_collisions link1="${namespace}J1" link2="${namespace}J2" reason="Adjacent"/>
+	<disable_collisions link1="${namespace}J1" link2="${namespace}J3" reason="Never"/>
+	<disable_collisions link1="${namespace}J1" link2="${namespace}J4" reason="Never"/>
+	<disable_collisions link1="${namespace}J1" link2="${namespace}base_link" reason="Adjacent"/>
+	<disable_collisions link1="${namespace}J2" link2="${namespace}J3" reason="Adjacent"/>
+	<disable_collisions link1="${namespace}J2" link2="${namespace}J4" reason="Never"/>
+	<disable_collisions link1="${namespace}J2" link2="${namespace}base_link" reason="Never"/>
+	<disable_collisions link1="${namespace}J3" link2="${namespace}J4" reason="Adjacent"/>
+	<disable_collisions link1="${namespace}J4" link2="${namespace}base_link" reason="Never"/>
   </xacro:macro>
 </robot>
