Commit message: feat: ajustments to the urdf files of others robots to support two arms and basic_camera support in cobotta

File: denso_robot_descriptions/robots/cobotta/urdf/denso_robot_joint_limits.xacro (robot description, xacro)
@@ -2,5 +2,5 @@
 <robot xmlns:xacro="http://www.ros.org/wiki/xacro">
 	<xacro:macro name="denso_robot_control_limits" params="namespace">
-		<joint name="$(arg namespace)joint_1">
+		<joint name="${namespace}joint_1">
 			<command_interface name="position">
 				<param name="min">-2.617994</param>
@@ -15,5 +15,5 @@
 			<state_interface name="effort"/>
 		</joint>
-		<joint name="$(arg namespace)joint_2">
+		<joint name="${namespace}joint_2">
 			<command_interface name="position">
 				<param name="min">-1.047198</param>
@@ -28,5 +28,5 @@
 			<state_interface name="effort"/>
 		</joint>
-		<joint name="$(arg namespace)joint_3">
+		<joint name="${namespace}joint_3">
 			<command_interface name="position">
 				<param name="min">0.314159</param>
@@ -41,5 +41,5 @@
 			<state_interface name="effort"/>
 		</joint>
-		<joint name="$(arg namespace)joint_4">
+		<joint name="${namespace}joint_4">
 			<command_interface name="position">
 				<param name="min">-2.967060</param>
@@ -54,5 +54,5 @@
 			<state_interface name="effort"/>
 		</joint>
-		<joint name="$(arg namespace)joint_5">
+		<joint name="${namespace}joint_5">
 			<command_interface name="position">
 				<param name="min">-1.658063</param>
@@ -67,5 +67,5 @@
 			<state_interface name="effort"/>
 		</joint>
-		<joint name="$(arg namespace)joint_6">
+		<joint name="${namespace}joint_6">
 			<command_interface name="position">
 				<param name="min">-2.967060</param>

File: denso_robot_descriptions/robots/cobotta/urdf/denso_robot_kinematics.xacro (robot description, xacro)
@@ -1,11 +1,11 @@
 <?xml version='1.0' encoding='UTF-8'?>
 <robot xmlns:xacro="http://www.ros.org/wiki/xacro">
-	<xacro:macro name="denso_robot_arm_kinematics" params="namespace model">
-		<link name="world"/>
-		<joint name="$(arg namespace)joint_w" type="fixed">
-			<parent link="world"/>
-			<child link="$(arg namespace)base_link"/>
+	<xacro:macro name="denso_robot_arm_kinematics" params="namespace model parent *origin">
+		<joint name="${namespace}joint_w" type="fixed">
+			<xacro:insert_block name="origin" />
+			<parent link="${parent}"/>
+			<child link="${namespace}base_link"/>
 		</joint>
-		<link name="$(arg namespace)base_link">
+		<link name="${namespace}base_link">
 			<visual>
 				<origin rpy="0 0 0" xyz="0 0 0"/>
@@ -26,5 +26,5 @@
 			</inertial>
 		</link>
-		<link name="$(arg namespace)J1">
+		<link name="${namespace}J1">
 			<visual>
 				<origin rpy="0 0 0" xyz="0 0 0"/>
@@ -45,7 +45,7 @@
 			</inertial>
 		</link>
-		<joint name="$(arg namespace)joint_1" type="revolute">
-			<parent link="$(arg namespace)base_link"/>
-			<child link="$(arg namespace)J1"/>
+		<joint name="${namespace}joint_1" type="revolute">
+			<parent link="${namespace}base_link"/>
+			<child link="${namespace}J1"/>
 			<origin rpy="0.000000 0.000000 0.000000" xyz="0.000000 0.000000 0.000000"/>
 			<axis xyz="-0.000000 -0.000000 1.000000"/>
@@ -53,5 +53,5 @@
 			<dynamics damping="0" friction="0"/>
 		</joint>
-		<link name="$(arg namespace)J2">
+		<link name="${namespace}J2">
 			<visual>
 				<origin rpy="0 0 0" xyz="0 0 0"/>
@@ -72,7 +72,7 @@
 			</inertial>
 		</link>
-		<joint name="$(arg namespace)joint_2" type="revolute">
-			<parent link="$(arg namespace)J1"/>
-			<child link="$(arg namespace)J2"/>
+		<joint name="${namespace}joint_2" type="revolute">
+			<parent link="${namespace}J1"/>
+			<child link="${namespace}J2"/>
 			<origin rpy="0.000000 0.000000 0.000000" xyz="0.000000 0.000000 0.180000"/>
 			<axis xyz="-0.000000 1.000000 -0.000000"/>
@@ -80,5 +80,5 @@
 			<dynamics damping="0" friction="0"/>
 		</joint>
-		<link name="$(arg namespace)J3">
+		<link name="${namespace}J3">
 			<visual>
 				<origin rpy="0 0 0" xyz="0 0 0"/>
@@ -99,7 +99,7 @@
 			</inertial>
 		</link>
-		<joint name="$(arg namespace)joint_3" type="revolute">
-			<parent link="$(arg namespace)J2"/>
-			<child link="$(arg namespace)J3"/>
+		<joint name="${namespace}joint_3" type="revolute">
+			<parent link="${namespace}J2"/>
+			<child link="${namespace}J3"/>
 			<origin rpy="0.000000 0.000000 0.000000" xyz="0.000000 0.000000 0.165000"/>
 			<axis xyz="-0.000000 1.000000 -0.000000"/>
@@ -107,5 +107,5 @@
 			<dynamics damping="0" friction="0"/>
 		</joint>
-		<link name="$(arg namespace)J4">
+		<link name="${namespace}J4">
 			<visual>
 				<origin rpy="0 0 0" xyz="0 0 0"/>
@@ -126,7 +126,7 @@
 			</inertial>
 		</link>
-		<joint name="$(arg namespace)joint_4" type="revolute">
-			<parent link="$(arg namespace)J3"/>
-			<child link="$(arg namespace)J4"/>
+		<joint name="${namespace}joint_4" type="revolute">
+			<parent link="${namespace}J3"/>
+			<child link="${namespace}J4"/>
 			<origin rpy="0.000000 0.000000 0.000000" xyz="-0.012000 0.020000 -0.345000"/>
 			<axis xyz="-0.000000 -0.000000 1.000000"/>
@@ -134,5 +134,5 @@
 			<dynamics damping="0" friction="0"/>
 		</joint>
-		<link name="$(arg namespace)J5">
+		<link name="${namespace}J5">
 			<visual>
 				<origin rpy="0 0 0" xyz="0 0 0"/>
@@ -153,7 +153,7 @@
 			</inertial>
 		</link>
-		<joint name="$(arg namespace)joint_5" type="revolute">
-			<parent link="$(arg namespace)J4"/>
-			<child link="$(arg namespace)J5"/>
+		<joint name="${namespace}joint_5" type="revolute">
+			<parent link="${namespace}J4"/>
+			<child link="${namespace}J5"/>
 			<origin rpy="0.000000 0.000000 0.000000" xyz="0.000000 -0.020000 0.522500"/>
 			<axis xyz="-0.000000 1.000000 -0.000000"/>
@@ -161,5 +161,5 @@
 			<dynamics damping="0" friction="0"/>
 		</joint>
-		<link name="$(arg namespace)J6">
+		<link name="${namespace}J6">
 			<visual>
 				<origin rpy="0 0 0" xyz="0 0 0"/>
@@ -180,7 +180,7 @@
 			</inertial>
 		</link>
-		<joint name="$(arg namespace)joint_6" type="revolute">
-			<parent link="$(arg namespace)J5"/>
-			<child link="$(arg namespace)J6"/>
+		<joint name="${namespace}joint_6" type="revolute">
+			<parent link="${namespace}J5"/>
+			<child link="${namespace}J6"/>
 			<origin rpy="0.000000 0.000000 0.000000" xyz="0.000000 -0.044500 0.042000"/>
 			<axis xyz="-0.000000 -0.000000 1.000000"/>

File: denso_robot_descriptions/robots/cobotta/urdf/denso_robot_macro.xacro (robot description, xacro)
@@ -67,9 +67,7 @@
       <xacro:insert_block name="origin" />
     </xacro:denso_robot_arm_kinematics>
-    <gazebo>
-	    <plugin filename="gz_ros2_control-system" name="gz_ros2_control::GazeboSimROS2ControlPlugin">
-      		<parameters>$(find denso_robot_moveit_config)/robots/$(arg model)/config/denso_robot_controllers.yaml</parameters>
-    	</plugin>
-  	</gazebo>
+    <xacro:if value="$(arg basic_camera)">
+      <xacro:basic_camera namespace="${namespace}" />
+    </xacro:if>
   </xacro:macro>
 </robot>

File: denso_robot_descriptions/robots/hsr065a1_n32/urdf/denso_robot.ros2_control.xacro (robot description, xacro)
@@ -38,5 +38,5 @@
         </xacro:unless>
       </hardware>
-      <xacro:denso_robot_control_limits namespace="$(arg namespace)" />
+      <xacro:denso_robot_control_limits namespace="${namespace}" />
     </ros2_control>
   </xacro:macro>

File: denso_robot_descriptions/robots/hsr065a1_n32/urdf/denso_robot_joint_limits.xacro (robot description, xacro)
@@ -2,5 +2,5 @@
 <robot xmlns:xacro="http://www.ros.org/wiki/xacro">
 	<xacro:macro name="denso_robot_control_limits" params="namespace">
-		<joint name="$(arg namespace)joint_1">
+		<joint name="${namespace}joint_1">
 			<command_interface name="position">
 				<param name="min">-2.268928</param>
@@ -15,5 +15,5 @@
 			<state_interface name="effort"/>
 		</joint>
-		<joint name="$(arg namespace)joint_2">
+		<joint name="${namespace}joint_2">
 			<command_interface name="position">
 				<param name="min">-2.617994</param>
@@ -28,5 +28,5 @@
 			<state_interface name="effort"/>
 		</joint>
-		<joint name="$(arg namespace)joint_3">
+		<joint name="${namespace}joint_3">
 			<command_interface name="position">
 				<param name="min">-0.100000</param>
@@ -41,5 +41,5 @@
 			<state_interface name="effort"/>
 		</joint>
-		<joint name="$(arg namespace)joint_4">
+		<joint name="${namespace}joint_4">
 			<command_interface name="position">
 				<param name="min">-6.283185</param>

File: denso_robot_descriptions/robots/hsr065a1_n32/urdf/denso_robot_kinematics.xacro (robot description, xacro)
@@ -1,11 +1,11 @@
 <?xml version='1.0' encoding='UTF-8'?>
 <robot xmlns:xacro="http://www.ros.org/wiki/xacro">
-	<xacro:macro name="denso_robot_arm_kinematics" params="namespace model">
-		<link name="world"/>
-		<joint name="$(arg namespace)joint_w" type="fixed">
-			<parent link="world"/>
-			<child link="$(arg namespace)base_link"/>
+	<xacro:macro name="denso_robot_arm_kinematics" params="namespace model parent *origin">
+		<joint name="${namespace}joint_w" type="fixed">
+			<xacro:insert_block name="origin" />
+			<parent link="${parent}"/>
+			<child link="${namespace}base_link"/>
 		</joint>
-		<link name="$(arg namespace)base_link">
+		<link name="${namespace}base_link">
 			<visual>
 				<origin rpy="0 0 0" xyz="0 0 0"/>
@@ -26,5 +26,5 @@
 			</inertial>
 		</link>
-		<link name="$(arg namespace)J1">
+		<link name="${namespace}J1">
 			<visual>
 				<origin rpy="0 0 0" xyz="0 0 0"/>
@@ -45,7 +45,7 @@
 			</inertial>
 		</link>
-		<joint name="$(arg namespace)joint_1" type="revolute">
-			<parent link="$(arg namespace)base_link"/>
-			<child link="$(arg namespace)J1"/>
+		<joint name="${namespace}joint_1" type="revolute">
+			<parent link="${namespace}base_link"/>
+			<child link="${namespace}J1"/>
 			<origin rpy="0.000000 0.000000 0.000000" xyz="0.000000 0.000000 0.000000"/>
 			<axis xyz="-0.000000 -0.000000 1.000000"/>
@@ -53,5 +53,5 @@
 			<dynamics damping="0" friction="0"/>
 		</joint>
-		<link name="$(arg namespace)J2">
+		<link name="${namespace}J2">
 			<visual>
 				<origin rpy="0 0 0" xyz="0 0 0"/>
@@ -72,7 +72,7 @@
 			</inertial>
 		</link>
-		<joint name="$(arg namespace)joint_2" type="revolute">
-			<parent link="$(arg namespace)J1"/>
-			<child link="$(arg namespace)J2"/>
+		<joint name="${namespace}joint_2" type="revolute">
+			<parent link="${namespace}J1"/>
+			<child link="${namespace}J2"/>
 			<origin rpy="0.000000 0.000000 0.000000" xyz="0.375000 0.000000 0.000000"/>
 			<axis xyz="-0.000000 -0.000000 1.000000"/>
@@ -80,5 +80,5 @@
 			<dynamics damping="0" friction="0"/>
 		</joint>
-		<link name="$(arg namespace)J3">
+		<link name="${namespace}J3">
 			<visual>
 				<origin rpy="0 0 0" xyz="0 0 0"/>
@@ -99,7 +99,7 @@
 			</inertial>
 		</link>
-		<joint name="$(arg namespace)joint_3" type="prismatic">
-			<parent link="$(arg namespace)J2"/>
-			<child link="$(arg namespace)J3"/>
+		<joint name="${namespace}joint_3" type="prismatic">
+			<parent link="${namespace}J2"/>
+			<child link="${namespace}J3"/>
 			<origin rpy="0.000000 0.000000 0.000000" xyz="-0.375000 0.000000 0.000000"/>
 			<axis xyz="0.000000 0.000000 1.000000"/>
@@ -107,5 +107,5 @@
 			<dynamics damping="0" friction="0"/>
 		</joint>
-		<link name="$(arg namespace)J4">
+		<link name="${namespace}J4">
 			<visual>
 				<origin rpy="0 0 0" xyz="0 0 0"/>
@@ -126,7 +126,7 @@
 			</inertial>
 		</link>
-		<joint name="$(arg namespace)joint_4" type="revolute">
-			<parent link="$(arg namespace)J3"/>
-			<child link="$(arg namespace)J4"/>
+		<joint name="${namespace}joint_4" type="revolute">
+			<parent link="${namespace}J3"/>
+			<child link="${namespace}J4"/>
 			<origin rpy="0.000000 0.000000 0.000000" xyz="0.650000 0.000000 0.000000"/>
 			<axis xyz="-0.000000 -0.000000 1.000000"/>

File: denso_robot_descriptions/robots/hsr065a1_n32/urdf/denso_robot_macro.xacro (robot description, xacro)
@@ -64,9 +64,4 @@
       <xacro:insert_block name="origin" />
     </xacro:denso_robot_arm_kinematics>
-    <gazebo>
-	    <plugin filename="gz_ros2_control-system" name="gz_ros2_control::GazeboSimROS2ControlPlugin">
-      		<parameters>$(find denso_robot_moveit_config)/robots/$(arg model)/config/denso_robot_controllers.yaml</parameters>
-    	</plugin>
-  	</gazebo>
   </xacro:macro>
 </robot>

File: denso_robot_descriptions/robots/vs060/urdf/denso_robot_joint_limits.xacro (robot description, xacro)
@@ -2,5 +2,5 @@
 <robot xmlns:xacro="http://www.ros.org/wiki/xacro">
 	<xacro:macro name="denso_robot_control_limits" params="namespace">
-		<joint name="$(arg namespace)joint_1">
+		<joint name="${namespace}joint_1">
 			<command_interface name="position">
 				<param name="min">-2.967060</param>
@@ -15,5 +15,5 @@
 			<state_interface name="effort"/>
 		</joint>
-		<joint name="$(arg namespace)joint_2">
+		<joint name="${namespace}joint_2">
 			<command_interface name="position">
 				<param name="min">-2.094395</param>
@@ -28,5 +28,5 @@
 			<state_interface name="effort"/>
 		</joint>
-		<joint name="$(arg namespace)joint_3">
+		<joint name="${namespace}joint_3">
 			<command_interface name="position">
 				<param name="min">-2.181662</param>
@@ -41,5 +41,5 @@
 			<state_interface name="effort"/>
 		</joint>
-		<joint name="$(arg namespace)joint_4">
+		<joint name="${namespace}joint_4">
 			<command_interface name="position">
 				<param name="min">-4.712389</param>
@@ -54,5 +54,5 @@
 			<state_interface name="effort"/>
 		</joint>
-		<joint name="$(arg namespace)joint_5">
+		<joint name="${namespace}joint_5">
 			<command_interface name="position">
 				<param name="min">-2.094395</param>
@@ -67,5 +67,5 @@
 			<state_interface name="effort"/>
 		</joint>
-		<joint name="$(arg namespace)joint_6">
+		<joint name="${namespace}joint_6">
 			<command_interface name="position">
 				<param name="min">-6.283185</param>

File: denso_robot_descriptions/robots/vs060/urdf/denso_robot_kinematics.xacro (robot description, xacro)
@@ -1,11 +1,11 @@
 <?xml version='1.0' encoding='UTF-8'?>
 <robot xmlns:xacro="http://www.ros.org/wiki/xacro">
-	<xacro:macro name="denso_robot_arm_kinematics" params="namespace model">
-		<link name="world"/>
-		<joint name="$(arg namespace)joint_w" type="fixed">
-			<parent link="world"/>
-			<child link="$(arg namespace)base_link"/>
+	<xacro:macro name="denso_robot_arm_kinematics" params="namespace model parent *origin">
+		<joint name="${namespace}joint_w" type="fixed">
+			<xacro:insert_block name="origin" />
+			<parent link="${parent}"/>
+			<child link="${namespace}base_link"/>
 		</joint>
-		<link name="$(arg namespace)base_link">
+		<link name="${namespace}base_link">
 			<visual>
 				<origin rpy="0 0 0" xyz="0 0 0"/>
@@ -26,5 +26,5 @@
 			</inertial>
 		</link>
-		<link name="$(arg namespace)J1">
+		<link name="${namespace}J1">
 			<visual>
 				<origin rpy="0 0 0" xyz="0 0 0"/>
@@ -45,7 +45,7 @@
 			</inertial>
 		</link>
-		<joint name="$(arg namespace)joint_1" type="revolute">
-			<parent link="$(arg namespace)base_link"/>
-			<child link="$(arg namespace)J1"/>
+		<joint name="${namespace}joint_1" type="revolute">
+			<parent link="${namespace}base_link"/>
+			<child link="${namespace}J1"/>
 			<origin rpy="0.000000 0.000000 0.000000" xyz="0.000000 0.000000 0.181500"/>
 			<axis xyz="-0.000000 -0.000000 1.000000"/>
@@ -53,5 +53,5 @@
 			<dynamics damping="0" friction="0"/>
 		</joint>
-		<link name="$(arg namespace)J2">
+		<link name="${namespace}J2">
 			<visual>
 				<origin rpy="0 0 0" xyz="0 0 0"/>
@@ -72,12 +72,12 @@
 			</inertial>
 		</link>
-		<joint name="$(arg namespace)joint_2" type="revolute">
-			<parent link="$(arg namespace)J1"/>
-			<child link="$(arg namespace)J2"/>
+		<joint name="${namespace}joint_2" type="revolute">
+			<parent link="${namespace}J1"/>
+			<child link="${namespace}J2"/>
 			<origin rpy="0.000000 0.000000 0.000000" xyz="0.000000 0.000000 0.163500"/>
 			<axis xyz="-0.000000 1.000000 -0.000000"/>
 			<limit effort="1000" lower="-2.0943951023932" upper="2.0943951023932" velocity="2.48709418409192"/> <!-- effort value is arbitary for make gazebo simulation runs without gravity problems -->
 		</joint>
-		<link name="$(arg namespace)J3">
+		<link name="${namespace}J3">
 			<visual>
 				<origin rpy="0 0 0" xyz="0 0 0"/>
@@ -98,7 +98,7 @@
 			</inertial>
 		</link>
-		<joint name="$(arg namespace)joint_3" type="revolute">
-			<parent link="$(arg namespace)J2"/>
-			<child link="$(arg namespace)J3"/>
+		<joint name="${namespace}joint_3" type="revolute">
+			<parent link="${namespace}J2"/>
+			<child link="${namespace}J3"/>
 			<origin rpy="0.000000 0.000000 0.000000" xyz="0.000000 0.000000 0.305000"/>
 			<axis xyz="-0.000000 1.000000 -0.000000"/>
@@ -106,5 +106,5 @@
 			<dynamics damping="0" friction="0"/>
 		</joint>
-		<link name="$(arg namespace)J4">
+		<link name="${namespace}J4">
 			<visual>
 				<origin rpy="0 0 0" xyz="0 0 0"/>
@@ -125,12 +125,12 @@
 			</inertial>
 		</link>
-		<joint name="$(arg namespace)joint_4" type="revolute">
-			<parent link="$(arg namespace)J3"/>
-			<child link="$(arg namespace)J4"/>
+		<joint name="${namespace}joint_4" type="revolute">
+			<parent link="${namespace}J3"/>
+			<child link="${namespace}J4"/>
 			<origin rpy="0.000000 0.000000 0.000000" xyz="-0.010000 0.000000 0.164500"/>
 			<axis xyz="-0.000000 -0.000000 1.000000"/>
 			<limit effort="1000" lower="-4.71238898038469" upper="4.71238898038469" velocity="3.73064127613788"/> <!-- effort value is arbitary for make gazebo simulation runs without gravity problems -->
 		</joint>
-		<link name="$(arg namespace)J5">
+		<link name="${namespace}J5">
 			<visual>
 				<origin rpy="0 0 0" xyz="0 0 0"/>
@@ -151,7 +151,7 @@
 			</inertial>
 		</link>
-		<joint name="$(arg namespace)joint_5" type="revolute">
-			<parent link="$(arg namespace)J4"/>
-			<child link="$(arg namespace)J5"/>
+		<joint name="${namespace}joint_5" type="revolute">
+			<parent link="${namespace}J4"/>
+			<child link="${namespace}J5"/>
 			<origin rpy="0.000000 0.000000 0.000000" xyz="0.000000 0.000000 0.135500"/>
 			<axis xyz="-0.000000 1.000000 -0.000000"/>
@@ -159,5 +159,5 @@
 			<dynamics damping="0" friction="0"/>
 		</joint>
-		<link name="$(arg namespace)J6">
+		<link name="${namespace}J6">
 			<visual>
 				<origin rpy="0 0 0" xyz="0 0 0"/>
@@ -178,7 +178,7 @@
 			</inertial>
 		</link>
-		<joint name="$(arg namespace)joint_6" type="revolute">
-			<parent link="$(arg namespace)J5"/>
-			<child link="$(arg namespace)J6"/>
+		<joint name="${namespace}joint_6" type="revolute">
+			<parent link="${namespace}J5"/>
+			<child link="${namespace}J6"/>
 			<origin rpy="0.000000 0.000000 0.000000" xyz="0.000000 0.000000 0.070000"/>
 			<axis xyz="-0.000000 -0.000000 1.000000"/>

File: denso_robot_descriptions/robots/vs060/urdf/denso_robot_macro.xacro (robot description, xacro)
@@ -74,12 +74,4 @@
       <xacro:insert_block name="origin" />
     </xacro:denso_robot_arm_kinematics>
-    <xacro:if value="$(arg basic_camera)">
-      <xacro:tool namespace="${namespace}" />
-    </xacro:if>
-    <gazebo>
-	    <plugin filename="gz_ros2_control-system" name="gz_ros2_control::GazeboSimROS2ControlPlugin">
-      		<parameters>$(find denso_robot_moveit_config)/robots/$(arg model)/config/denso_robot_controllers.yaml</parameters>
-    	</plugin>
-  	</gazebo>
   </xacro:macro>
 </robot>
