Commit message: feat: add end effector args to basic_camera

File: denso_robot_descriptions/robots/cobotta/urdf/denso_robot_macro.xacro (robot description, xacro)
@@ -75,5 +75,5 @@
     </xacro:denso_robot_arm_kinematics>
     <xacro:if value="$(arg basic_camera)">
-      <xacro:basic_camera namespace="${namespace}" />
+      <xacro:basic_camera namespace="${namespace}" end_effector="J6" />
     </xacro:if>
   </xacro:macro>

File: denso_robot_descriptions/robots/vs050/urdf/denso_robot_macro.xacro (robot description, xacro)
@@ -75,5 +75,5 @@
     </xacro:denso_robot_arm_kinematics>
     <xacro:if value="$(arg basic_camera)">
-      <xacro:basic_camera namespace="${namespace}" />
+      <xacro:basic_camera namespace="${namespace}" end_effector="J6" />
     </xacro:if>
   </xacro:macro>

File: denso_robot_descriptions/robots/vs060/urdf/denso_robot_macro.xacro (robot description, xacro)
@@ -75,5 +75,5 @@
     </xacro:denso_robot_arm_kinematics>
     <xacro:if value="$(arg basic_camera)">
-      <xacro:basic_camera namespace="${namespace}" />
+      <xacro:basic_camera namespace="${namespace}" end_effector="J6" />
     </xacro:if>
   </xacro:macro>

File: denso_robot_descriptions/tools/basic_camera/urdf/basic_camera.xacro (robot description, xacro)
@@ -2,5 +2,5 @@
 <robot xmlns:xacro="http://www.ros.org/wiki/xacro">
     <!-- here you define the parameters you want your xacro file to receive. -->
-    <xacro:macro name="basic_camera" params="namespace">
+    <xacro:macro name="basic_camera" params="namespace end_effector">
     <!-- if your tool has meshes, define the path to it in geometry tag. -->
     <!-- see the vs050 robot urdf implementation as an example. -->
@@ -23,5 +23,5 @@
 	<joint name="${namespace}basic_camera_joint" type="fixed">
         <!-- here you define where your tool will connect. In this case, it's at joint 6. -->
-		<parent link="${namespace}J6"/>
+		<parent link="${namespace}${end_effector}"/>
 		<child link="${namespace}basic_camera_link"/>
 		<origin rpy="0 ${radians(-90)} 0" xyz="0 0 0.01"/>
