Commit message: feat(cobotta): synchronize URDF and MoveIt configs with modernized setup
- Introduce standard `flange` and `tool0` links to the cobotta kinematics.
- Flatten the legacy YAML hierarchy in `moveit_controllers.yaml` for MoveIt 2 compatibility.
- Expand `ros2_control` hardware interfaces in `joint_limits.xacro` to include `velocity` and `effort`.
- Enforce strict trajectory controller constraints (open loop, zero velocity tolerance) in `denso_robot_controllers.yaml`.
- Update xacro macros to use the correct `www.ros.org` namespace and clean up XML indentation across files (including a minor formatting fix in vs050).

File: denso_robot_descriptions/robots/cobotta/urdf/denso_robot.ros2_control.xacro (robot description, xacro)
@@ -1,18 +1,27 @@
 <?xml version="1.0"?>
 <robot xmlns:xacro="http://www.ros.org/wiki/xacro">
-  <xacro:macro name="denso_robot_ros2_control" params="name namespace
-	robot_name
-    sim:=false fake_sensor_commands:=false
-    ip_address
-    model
-    robot_joints joint_1 joint_2 joint_3 joint_4 joint_5 joint_6
-    arm_group
-    send_format recv_format
-	controller_type
-    verbose
-    ">
+  <xacro:macro name="denso_robot_ros2_control"
+               params="name
+                       namespace
+                       robot_name
+                       sim:=false
+                       fake_sensor_commands:=false
+                       ip_address
+                       model
+                       robot_joints
+                       joint_1
+                       joint_2
+                       joint_3
+                       joint_4
+                       joint_5
+                       joint_6
+                       arm_group
+                       send_format
+                       recv_format
+                       controller_type
+                       verbose">
     <ros2_control name="${namespace}${name}" type="system">
-	<!-- joint limits include -->
-	<xacro:include filename="$(find denso_robot_descriptions)/robots/$(arg model)/urdf/denso_robot_joint_limits.xacro" />
+	  <!-- joint limits include -->
+	  <xacro:include filename="$(find denso_robot_descriptions)/robots/$(arg model)/urdf/denso_robot_joint_limits.xacro" />
       <hardware>
         <xacro:if value="${sim}">
@@ -22,5 +31,5 @@
           <plugin>denso_robot_control/DensoRobotHW</plugin>
           <param name="ip_address">${ip_address}</param>
-<!-- "robot_name" param must be consistent with the @TYPE_NAME variable of the real robot !!  -->
+          <!-- "robot_name" param must be consistent with the @TYPE_NAME variable of the real robot !!  -->
           <param name="robot_name">${robot_name}</param>
           <param name="node_name">denso_robot_control</param>
@@ -40,5 +49,5 @@
         </xacro:unless>
       </hardware>
-      <xacro:denso_robot_control_limits namespace="$(arg namespace)" />
+      <xacro:denso_robot_control_limits namespace="${namespace}" />
     </ros2_control>
   </xacro:macro>

File: denso_robot_descriptions/robots/cobotta/urdf/denso_robot_joint_limits.xacro (robot description, xacro)
@@ -1,83 +1,53 @@
 <?xml version='1.0' encoding='UTF-8'?>
 <robot xmlns:xacro="http://www.ros.org/wiki/xacro">
-	<xacro:macro name="denso_robot_control_limits" params="namespace">
-		<joint name="$(arg namespace)joint_1">
-			<command_interface name="position">
-				<param name="min">-2.617994</param>
-				<param name="max">2.617994</param>
-			</command_interface>
-			<command_interface name="velocity">
-				<param name="min">0</param>
-				<param name="max">0.03830125043501562</param>
-			</command_interface>
-			<state_interface name="position"/>
-			<state_interface name="velocity"/>
-			<state_interface name="effort"/>
-		</joint>
-		<joint name="$(arg namespace)joint_2">
-			<command_interface name="position">
-				<param name="min">-1.047198</param>
-				<param name="max">1.745329</param>
-			</command_interface>
-			<command_interface name="velocity">
-				<param name="min">0</param>
-				<param name="max">0.037256670877697</param>
-			</command_interface>
-			<state_interface name="position"/>
-			<state_interface name="velocity"/>
-			<state_interface name="effort"/>
-		</joint>
-		<joint name="$(arg namespace)joint_3">
-			<command_interface name="position">
-				<param name="min">0.314159</param>
-				<param name="max">2.443461</param>
-			</command_interface>
-			<command_interface name="velocity">
-				<param name="min">0</param>
-				<param name="max">0.068942250783028</param>
-			</command_interface>
-			<state_interface name="position"/>
-			<state_interface name="velocity"/>
-			<state_interface name="effort"/>
-		</joint>
-		<joint name="$(arg namespace)joint_4">
-			<command_interface name="position">
-				<param name="min">-2.967060</param>
-				<param name="max">2.967060</param>
-			</command_interface>
-			<command_interface name="velocity">
-				<param name="min">0</param>
-				<param name="max">0.0702189591308619</param>
-			</command_interface>
-			<state_interface name="position"/>
-			<state_interface name="velocity"/>
-			<state_interface name="effort"/>
-		</joint>
-		<joint name="$(arg namespace)joint_5">
-			<command_interface name="position">
-				<param name="min">-1.658063</param>
-				<param name="max">2.356194</param>
-			</command_interface>
-			<command_interface name="velocity">
-				<param name="min">0</param>
-				<param name="max">0.0702189591308619</param>
-			</command_interface>
-			<state_interface name="position"/>
-			<state_interface name="velocity"/>
-			<state_interface name="effort"/>
-		</joint>
-		<joint name="$(arg namespace)joint_6">
-			<command_interface name="position">
-				<param name="min">-2.967060</param>
-				<param name="max">2.967060</param>
-			</command_interface>
-			<command_interface name="velocity">
-				<param name="min">0</param>
-				<param name="max">0.105386470893922</param>
-			</command_interface>
-			<state_interface name="position"/>
-			<state_interface name="velocity"/>
-			<state_interface name="effort"/>
-		</joint>
+	<xacro:macro name="denso_robot_control_limits" params="namespace initial_positions_file">
+	  <joint name="${namespace}joint_1">
+      <command_interface name="position" />
+      <command_interface name="velocity" />
+      <state_interface name="position">
+      </state_interface>
+      <state_interface name="velocity" />
+      <state_interface name="effort"/>
+    </joint>
+    <joint name="${namespace}joint_2">
+      <command_interface name="position" />
+      <command_interface name="velocity" />
+      <state_interface name="position">
+      </state_interface>
+      <state_interface name="velocity" />
+      <state_interface name="effort"/>
+    </joint>
+    <joint name="${namespace}joint_3">
+      <command_interface name="position" />
+      <command_interface name="velocity" />
+      <state_interface name="position">
+      </state_interface>
+      <state_interface name="velocity" />
+      <state_interface name="effort"/>
+    </joint>
+    <joint name="${namespace}joint_4">
+      <command_interface name="position" />
+      <command_interface name="velocity" />
+      <state_interface name="position">
+      </state_interface>
+      <state_interface name="velocity" />
+      <state_interface name="effort"/>
+    </joint>
+    <joint name="${namespace}joint_5">
+      <command_interface name="position" />
+      <command_interface name="velocity" />
+      <state_interface name="position">
+      </state_interface>
+      <state_interface name="velocity" />
+      <state_interface name="effort"/>
+    </joint>
+    <joint name="${namespace}joint_6">
+      <command_interface name="position" />
+      <command_interface name="velocity" />
+      <state_interface name="position">
+      </state_interface>
+      <state_interface name="velocity" />
+      <state_interface name="effort"/>
+    </joint>
 	</xacro:macro>
 </robot>

File: denso_robot_descriptions/robots/cobotta/urdf/denso_robot_kinematics.xacro (robot description, xacro)
@@ -1,11 +1,11 @@
 <?xml version='1.0' encoding='UTF-8'?>
 <robot xmlns:xacro="http://www.ros.org/wiki/xacro">
-	<xacro:macro name="denso_robot_arm_kinematics" params="namespace model">
-		<link name="world"/>
-		<joint name="$(arg namespace)joint_w" type="fixed">
-			<parent link="world"/>
-			<child link="$(arg namespace)base_link"/>
-		</joint>
-		<link name="$(arg namespace)base_link">
+	<xacro:macro name="denso_robot_arm_kinematics" params="namespace model parent *origin">
+		<joint name="${namespace}joint_w" type="fixed">
+			<xacro:insert_block name="origin"  />
+			<parent link="${parent}" />
+			<child link="${namespace}base_link" />
+		</joint>
+		<link name="${namespace}base_link">
 			<visual>
 				<origin rpy="0 0 0" xyz="0 0 0"/>
@@ -26,5 +26,5 @@
 			</inertial>
 		</link>
-		<link name="$(arg namespace)J1">
+		<link name="${namespace}J1">
 			<visual>
 				<origin rpy="0 0 0" xyz="0 0 0"/>
@@ -45,7 +45,7 @@
 			</inertial>
 		</link>
-		<joint name="$(arg namespace)joint_1" type="revolute">
-			<parent link="$(arg namespace)base_link"/>
-			<child link="$(arg namespace)J1"/>
+		<joint name="${namespace}joint_1" type="revolute">
+			<parent link="${namespace}base_link"/>
+			<child link="${namespace}J1"/>
 			<origin rpy="0.000000 0.000000 0.000000" xyz="0.000000 0.000000 0.000000"/>
 			<axis xyz="-0.000000 -0.000000 1.000000"/>
@@ -53,5 +53,5 @@
 			<dynamics damping="0" friction="0"/>
 		</joint>
-		<link name="$(arg namespace)J2">
+		<link name="${namespace}J2">
 			<visual>
 				<origin rpy="0 0 0" xyz="0 0 0"/>
@@ -72,7 +72,7 @@
 			</inertial>
 		</link>
-		<joint name="$(arg namespace)joint_2" type="revolute">
-			<parent link="$(arg namespace)J1"/>
-			<child link="$(arg namespace)J2"/>
+		<joint name="${namespace}joint_2" type="revolute">
+			<parent link="${namespace}J1"/>
+			<child link="${namespace}J2"/>
 			<origin rpy="0.000000 0.000000 0.000000" xyz="0.000000 0.000000 0.180000"/>
 			<axis xyz="-0.000000 1.000000 -0.000000"/>
@@ -80,5 +80,5 @@
 			<dynamics damping="0" friction="0"/>
 		</joint>
-		<link name="$(arg namespace)J3">
+		<link name="${namespace}J3">
 			<visual>
 				<origin rpy="0 0 0" xyz="0 0 0"/>
@@ -99,7 +99,7 @@
 			</inertial>
 		</link>
-		<joint name="$(arg namespace)joint_3" type="revolute">
-			<parent link="$(arg namespace)J2"/>
-			<child link="$(arg namespace)J3"/>
+		<joint name="${namespace}joint_3" type="revolute">
+			<parent link="${namespace}J2"/>
+			<child link="${namespace}J3"/>
 			<origin rpy="0.000000 0.000000 0.000000" xyz="0.000000 0.000000 0.165000"/>
 			<axis xyz="-0.000000 1.000000 -0.000000"/>
@@ -107,5 +107,5 @@
 			<dynamics damping="0" friction="0"/>
 		</joint>
-		<link name="$(arg namespace)J4">
+		<link name="${namespace}J4">
 			<visual>
 				<origin rpy="0 0 0" xyz="0 0 0"/>
@@ -126,7 +126,7 @@
 			</inertial>
 		</link>
-		<joint name="$(arg namespace)joint_4" type="revolute">
-			<parent link="$(arg namespace)J3"/>
-			<child link="$(arg namespace)J4"/>
+		<joint name="${namespace}joint_4" type="revolute">
+			<parent link="${namespace}J3"/>
+			<child link="${namespace}J4"/>
 			<origin rpy="0.000000 0.000000 0.000000" xyz="-0.012000 0.020000 -0.345000"/>
 			<axis xyz="-0.000000 -0.000000 1.000000"/>
@@ -134,5 +134,5 @@
 			<dynamics damping="0" friction="0"/>
 		</joint>
-		<link name="$(arg namespace)J5">
+		<link name="${namespace}J5">
 			<visual>
 				<origin rpy="0 0 0" xyz="0 0 0"/>
@@ -153,7 +153,7 @@
 			</inertial>
 		</link>
-		<joint name="$(arg namespace)joint_5" type="revolute">
-			<parent link="$(arg namespace)J4"/>
-			<child link="$(arg namespace)J5"/>
+		<joint name="${namespace}joint_5" type="revolute">
+			<parent link="${namespace}J4"/>
+			<child link="${namespace}J5"/>
 			<origin rpy="0.000000 0.000000 0.000000" xyz="0.000000 -0.020000 0.522500"/>
 			<axis xyz="-0.000000 1.000000 -0.000000"/>
@@ -161,5 +161,5 @@
 			<dynamics damping="0" friction="0"/>
 		</joint>
-		<link name="$(arg namespace)J6">
+		<link name="${namespace}J6">
 			<visual>
 				<origin rpy="0 0 0" xyz="0 0 0"/>
@@ -180,7 +180,7 @@
 			</inertial>
 		</link>
-		<joint name="$(arg namespace)joint_6" type="revolute">
-			<parent link="$(arg namespace)J5"/>
-			<child link="$(arg namespace)J6"/>
+		<joint name="${namespace}joint_6" type="revolute">
+			<parent link="${namespace}J5"/>
+			<child link="${namespace}J6"/>
 			<origin rpy="0.000000 0.000000 0.000000" xyz="0.000000 -0.044500 0.042000"/>
 			<axis xyz="-0.000000 -0.000000 1.000000"/>
@@ -188,4 +188,16 @@
 			<dynamics damping="0" friction="0"/>
 		</joint>
+		<link name="${namespace}flange"/>
+		<joint name="${namespace}J6-flange" type="fixed">
+			<parent link="${namespace}J6"/>
+			<child link="${namespace}flange"/>
+			<origin rpy="0 0 0" xyz="0 0 0"/>
+		</joint>
+		<link name="${namespace}tool0"/>
+		<joint name="${namespace}J6-tool0" type="fixed">
+			<parent link="${namespace}J6"/>
+			<child link="${namespace}tool0"/>
+			<origin rpy="${radians(pi)} ${radians(-pi/2)} 0" xyz="0 0 0"/>
+		</joint>
 	</xacro:macro>
 </robot>

File: denso_robot_descriptions/robots/cobotta/urdf/denso_robot_macro.xacro (robot description, xacro)
@@ -1,4 +1,4 @@
 <?xml version="1.0"?>
-<robot xmlns:xacro="http://wiki.ros.org/xacro">
+<robot xmlns:xacro="http://www.ros.org/wiki/xacro">
   <!--
     Base Denso robot xacro macro.
@@ -9,63 +9,70 @@
     Author DENSO WAVE INCORPORATED
   -->
-  <xacro:macro name="denso_robot" params="
-    model
-    namespace
-    transmission_hw_interface:=hardware_interface/PositionJointInterface
-    sim:=false
-    ip_address
-    send_format
-    recv_format
-    verbose:=false"
-  >
-    <!-- Robot data required by the denso driver -->
-    <xacro:arg name="ip_address" default="192.168.0.1"/>
-    <xacro:arg name="robot_name" default="CVR038A1-NV6-NN"/> <!-- "robot_name" param must be consistent with the @TYPE_NAME variable of the real robot !! -->
-    <xacro:arg name="robot_joints" default="6"/> <!-- number of total joints in the kinematic chain -->
-    <xacro:arg name="joint_1" default="1"/> <!-- 0 = prismatic , 1 = revolute -->
-    <xacro:arg name="joint_2" default="1"/> <!-- 0 = prismatic , 1 = revolute -->
-    <xacro:arg name="joint_3" default="1"/> <!-- 0 = prismatic , 1 = revolute -->
-    <xacro:arg name="joint_4" default="1"/> <!-- 0 = prismatic , 1 = revolute -->
-    <xacro:arg name="joint_5" default="1"/> <!-- 0 = prismatic , 1 = revolute -->
-    <xacro:arg name="joint_6" default="1"/> <!-- 0 = prismatic , 1 = revolute -->
-    <xacro:arg name="controller_type" default="8"/> <!-- 8 = RC8 , 9 = RC9 -->
-    <xacro:arg name="arm_group" default="0"/>
-    <xacro:arg name="send_format" default="288"/>
-    <xacro:arg name="recv_format" default="292"/>
-    <xacro:arg name="verbose" default="false"/>
-    <xacro:include filename="$(find denso_robot_descriptions)/robots/$(arg model)/urdf/denso_robot_transmissions.xacro" />
-    <!-- robot kinematics include -->
-    <xacro:include filename="$(find denso_robot_descriptions)/robots/$(arg model)/urdf/denso_robot_kinematics.xacro" />
-    <!-- ros2 control include -->
-    <xacro:include filename="$(find denso_robot_descriptions)/robots/$(arg model)/urdf/denso_robot.ros2_control.xacro" />
-    <!-- ros2 control instance -->
-    <xacro:denso_robot_ros2_control
-      name="GazeboSystem" namespace="$(arg namespace)"
-      sim="$(arg sim)"
-      model="$(arg model)"
-      ip_address="$(arg ip_address)"
-      robot_name="$(arg robot_name)"
-      robot_joints="$(arg robot_joints)"
-      joint_1="$(arg joint_1)"
-      joint_2="$(arg joint_2)"
-      joint_3="$(arg joint_3)"
-      joint_4="$(arg joint_4)"
-      joint_5="$(arg joint_5)"
-      joint_6="$(arg joint_6)"
-      arm_group="$(arg arm_group)"
-      controller_type="$(arg controller_type)"
-      verbose="$(arg verbose)"
-      send_format="$(arg send_format)"
-      recv_format="$(arg recv_format)" />
-    <!-- Add URDF transmission elements (for ros_control) -->
-    <xacro:denso_robot_arm_transmission namespace="$(arg namespace)" hw_interface="$(arg transmission_hw_interface)" />
-    <!-- Placeholder for ros2_control transmission which don't yet exist -->
-    <!-- links -  main serial chain -->
-    <xacro:denso_robot_arm_kinematics namespace="$(arg namespace)" model="$(arg model)" />
-    <gazebo>
-	    <plugin filename="gz_ros2_control-system" name="gz_ros2_control::GazeboSimROS2ControlPlugin">
-      		<parameters>$(find denso_robot_moveit_config)/robots/$(arg model)/config/denso_robot_controllers.yaml</parameters>
-    	</plugin>
-  	</gazebo>
+  <xacro:macro name="denso_robot" params="model
+                                          namespace
+                                          parent
+                                          *origin
+                                          transmission_hw_interface:=hardware_interface/PositionJointInterface
+                                          sim:=false
+                                          basic_camera:=false
+                                          ip_address
+                                          send_format
+                                          recv_format
+                                          verbose:=false">
+  <!-- Robot data required by the denso driver -->
+  <xacro:arg name="ip_address" default=""/>
+  <xacro:arg name="robot_name" default="CVR038A1-NV6-NN"/> <!-- "robot_name" param must be consistent with the @TYPE_NAME variable of the real robot !! -->
+  <xacro:arg name="robot_joints" default="6"/> <!-- number of total joints in the kinematic chain -->
+  <xacro:arg name="joint_1" default="1"/> <!-- 0 = prismatic , 1 = revolute -->
+  <xacro:arg name="joint_2" default="1"/> <!-- 0 = prismatic , 1 = revolute -->
+  <xacro:arg name="joint_3" default="1"/> <!-- 0 = prismatic , 1 = revolute -->
+  <xacro:arg name="joint_4" default="1"/> <!-- 0 = prismatic , 1 = revolute -->
+  <xacro:arg name="joint_5" default="1"/> <!-- 0 = prismatic , 1 = revolute -->
+  <xacro:arg name="joint_6" default="1"/> <!-- 0 = prismatic , 1 = revolute -->
+  <xacro:arg name="controller_type" default="8"/> <!-- 8 = RC8 , 9 = RC9 -->
+  <xacro:arg name="arm_group" default="0"/>
+  <xacro:arg name="send_format" default="288"/>
+  <xacro:arg name="recv_format" default="292"/>
+  <xacro:arg name="verbose" default="false"/>
+  <xacro:include filename="$(find denso_robot_descriptions)/robots/$(arg model)/urdf/denso_robot_transmissions.xacro" />
+  <!-- robot kinematics include -->
+  <xacro:include filename="$(find denso_robot_descriptions)/robots/$(arg model)/urdf/denso_robot_kinematics.xacro" />
+  <!-- ros2 control include -->
+  <xacro:include filename="$(find denso_robot_descriptions)/robots/$(arg model)/urdf/denso_robot.ros2_control.xacro" />
+  <!-- For other tools, modify the filename parameter to the path of your tool's xacro file. -->
+  <!-- The line with tag xacro:tool passes the parameters defined in your tool's xacro file -->
+  <!-- (see basic_camera.xacro as an example implementation) -->
+  <xacro:if value="$(arg basic_camera)">
+    <xacro:include filename="$(find denso_robot_gazebo)/sensors/basic_camera/urdf/basic_camera.xacro" />
+  </xacro:if>
+  <!-- ros2 control instance -->
+  <xacro:denso_robot_ros2_control name="COBOTTA"
+                                  namespace="${namespace}"
+                                  sim="$(arg sim)"
+                                  model="$(arg model)"
+                                  ip_address="${ip_address}"
+                                  robot_name="$(arg robot_name)"
+                                  robot_joints="$(arg robot_joints)"
+                                  joint_1="$(arg joint_1)"
+                                  joint_2="$(arg joint_2)"
+                                  joint_3="$(arg joint_3)"
+                                  joint_4="$(arg joint_4)"
+                                  joint_5="$(arg joint_5)"
+                                  joint_6="$(arg joint_6)"
+                                  arm_group="$(arg arm_group)"
+                                  controller_type="$(arg controller_type)"
+                                  verbose="$(arg verbose)"
+                                  send_format="$(arg send_format)"
+                                  recv_format="$(arg recv_format)" />
+  <!-- Add URDF transmission elements (for ros_control) -->
+  <xacro:denso_robot_arm_transmission namespace="${namespace}" hw_interface="$(arg transmission_hw_interface)" />
+  <!-- Placeholder for ros2_control transmission which don't yet exist -->
+  <!-- links -  main serial chain -->
+  <xacro:denso_robot_arm_kinematics namespace="${namespace}" model="$(arg model)" parent="${parent}">
+    <xacro:insert_block name="origin" />
+  </xacro:denso_robot_arm_kinematics>
+  <xacro:if value="$(arg basic_camera)">
+    <xacro:basic_camera namespace="${namespace}" end_effector="J6" />
+  </xacro:if>
   </xacro:macro>
 </robot>

File: denso_robot_descriptions/robots/vs050/urdf/denso_robot_kinematics.xacro (robot description, xacro)
@@ -193,13 +193,13 @@
 		<link name="${namespace}flange"/>
 		<joint name="${namespace}J6-flange" type="fixed">
-      <parent link="${namespace}J6"/>
-      <child link="${namespace}flange"/>
-      <origin rpy="0 0 0" xyz="0 0 0"/>
+			<parent link="${namespace}J6"/>
+			<child link="${namespace}flange"/>
+			<origin rpy="0 0 0" xyz="0 0 0"/>
 		</joint>
 		<link name="${namespace}tool0"/>
 		<joint name="${namespace}J6-tool0" type="fixed">
-      <parent link="${namespace}J6"/>
-      <child link="${namespace}tool0"/>
-      <origin rpy="${radians(pi)} ${radians(-pi/2)} 0" xyz="0 0 0"/>
+			<parent link="${namespace}J6"/>
+			<child link="${namespace}tool0"/>
+			<origin rpy="${radians(pi)} ${radians(-pi/2)} 0" xyz="0 0 0"/>
 		</joint>
 	</xacro:macro>
