Commit message: feat(cobotta): overhaul configurations and enable cobotta in bringup
Fixes xacro namespace syntax errors (`$(arg)` to `${}`), removes the model restriction in the bringup launch, flattens MoveIt configuration YAMLs, and brings the cobotta URDF (tool0, gz_cam, parent/origin support) into full parity with the VS series.

File: denso_robot_descriptions/robots/cobotta/urdf/denso_robot.ros2_control.xacro (robot description, xacro)
@@ -1,29 +1,38 @@
 <?xml version="1.0"?>
 <robot xmlns:xacro="http://www.ros.org/wiki/xacro">
-  <xacro:macro name="denso_robot_ros2_control" params="name namespace
-	robot_name
-    sim:=false fake_sensor_commands:=false
-    ip_address
-    model
-    robot_joints joint_1 joint_2 joint_3 joint_4 joint_5 joint_6
-    arm_group
-    send_format recv_format
-	controller_type
-    verbose
-    ">
+  <xacro:macro name="denso_robot_ros2_control"
+               params="name
+                       namespace
+                       robot_name
+                       sim:=false
+                       fake_sensor_commands:=false
+                       ip_address
+                       model
+                       robot_joints
+                       joint_1
+                       joint_2
+                       joint_3
+                       joint_4
+                       joint_5
+                       joint_6
+                       arm_group
+                       send_format
+                       recv_format
+                       controller_type
+                       verbose">
     <ros2_control name="${namespace}${name}" type="system">
-	<!-- joint limits include -->
-	<xacro:include filename="$(find denso_robot_descriptions)/robots/$(arg model)/urdf/denso_robot_joint_limits.xacro" />
+      <!-- joint limits include -->
+      <xacro:include filename="$(find denso_robot_descriptions)/robots/$(arg model)/urdf/denso_robot_joint_limits.xacro" />
       <hardware>
         <xacro:if value="${sim}">
-      	  <plugin>gz_ros2_control/GazeboSimSystem</plugin>
+          <plugin>gz_ros2_control/GazeboSimSystem</plugin>
         </xacro:if>
         <xacro:unless value="${sim}">
           <plugin>denso_robot_control/DensoRobotHW</plugin>
           <param name="ip_address">${ip_address}</param>
-<!-- "robot_name" param must be consistent with the @TYPE_NAME variable of the real robot !!  -->
+          <!-- "robot_name" param must be consistent with the @TYPE_NAME variable of the real robot !! -->
           <param name="robot_name">${robot_name}</param>
           <param name="node_name">denso_robot_control</param>
-          <param name="node_namespace">${namespace}${model}</param>
+          <param name="node_namespace">${namespace}$(arg model)</param>
           <param name="robot_joints">${robot_joints}</param>
           <param name="joint_1">${joint_1}</param>
@@ -40,5 +49,5 @@
         </xacro:unless>
       </hardware>
-      <xacro:denso_robot_control_limits namespace="$(arg namespace)" />
+      <xacro:denso_robot_control_limits namespace="${namespace}" />
     </ros2_control>
   </xacro:macro>

File: denso_robot_descriptions/robots/cobotta/urdf/denso_robot_joint_limits.xacro (robot description, xacro)
@@ -2,5 +2,5 @@
 <robot xmlns:xacro="http://www.ros.org/wiki/xacro">
 	<xacro:macro name="denso_robot_control_limits" params="namespace">
-		<joint name="$(arg namespace)joint_1">
+		<joint name="${namespace}joint_1">
 			<command_interface name="position">
 				<param name="min">-2.617994</param>
@@ -11,9 +11,11 @@
 				<param name="max">0.03830125043501562</param>
 			</command_interface>
-			<state_interface name="position"/>
+			<state_interface name="position">
+				<param name="initial_value">0.0</param>
+			</state_interface>
 			<state_interface name="velocity"/>
 			<state_interface name="effort"/>
 		</joint>
-		<joint name="$(arg namespace)joint_2">
+		<joint name="${namespace}joint_2">
 			<command_interface name="position">
 				<param name="min">-1.047198</param>
@@ -24,9 +26,11 @@
 				<param name="max">0.037256670877697</param>
 			</command_interface>
-			<state_interface name="position"/>
+			<state_interface name="position">
+				<param name="initial_value">0.0</param>
+			</state_interface>
 			<state_interface name="velocity"/>
 			<state_interface name="effort"/>
 		</joint>
-		<joint name="$(arg namespace)joint_3">
+		<joint name="${namespace}joint_3">
 			<command_interface name="position">
 				<param name="min">0.314159</param>
@@ -37,9 +41,12 @@
 				<param name="max">0.068942250783028</param>
 			</command_interface>
-			<state_interface name="position"/>
+			<!-- joint_3 lower bound is 0.314159 rad — initial value must be inside [0.314159, 2.443461] -->
+			<state_interface name="position">
+				<param name="initial_value">1.5</param>
+			</state_interface>
 			<state_interface name="velocity"/>
 			<state_interface name="effort"/>
 		</joint>
-		<joint name="$(arg namespace)joint_4">
+		<joint name="${namespace}joint_4">
 			<command_interface name="position">
 				<param name="min">-2.967060</param>
@@ -50,9 +57,11 @@
 				<param name="max">0.0702189591308619</param>
 			</command_interface>
-			<state_interface name="position"/>
+			<state_interface name="position">
+				<param name="initial_value">0.0</param>
+			</state_interface>
 			<state_interface name="velocity"/>
 			<state_interface name="effort"/>
 		</joint>
-		<joint name="$(arg namespace)joint_5">
+		<joint name="${namespace}joint_5">
 			<command_interface name="position">
 				<param name="min">-1.658063</param>
@@ -63,9 +72,11 @@
 				<param name="max">0.0702189591308619</param>
 			</command_interface>
-			<state_interface name="position"/>
+			<state_interface name="position">
+				<param name="initial_value">0.0</param>
+			</state_interface>
 			<state_interface name="velocity"/>
 			<state_interface name="effort"/>
 		</joint>
-		<joint name="$(arg namespace)joint_6">
+		<joint name="${namespace}joint_6">
 			<command_interface name="position">
 				<param name="min">-2.967060</param>
@@ -76,5 +87,7 @@
 				<param name="max">0.105386470893922</param>
 			</command_interface>
-			<state_interface name="position"/>
+			<state_interface name="position">
+				<param name="initial_value">0.0</param>
+			</state_interface>
 			<state_interface name="velocity"/>
 			<state_interface name="effort"/>

File: denso_robot_descriptions/robots/cobotta/urdf/denso_robot_kinematics.xacro (robot description, xacro)
@@ -1,11 +1,11 @@
 <?xml version='1.0' encoding='UTF-8'?>
 <robot xmlns:xacro="http://www.ros.org/wiki/xacro">
-	<xacro:macro name="denso_robot_arm_kinematics" params="namespace model">
-		<link name="world"/>
-		<joint name="$(arg namespace)joint_w" type="fixed">
-			<parent link="world"/>
-			<child link="$(arg namespace)base_link"/>
+	<xacro:macro name="denso_robot_arm_kinematics" params="namespace model parent *origin">
+		<joint name="${namespace}joint_w" type="fixed">
+			<xacro:insert_block name="origin" />
+			<parent link="${parent}" />
+			<child link="${namespace}base_link" />
 		</joint>
-		<link name="$(arg namespace)base_link">
+		<link name="${namespace}base_link">
 			<visual>
 				<origin rpy="0 0 0" xyz="0 0 0"/>
@@ -26,5 +26,5 @@
 			</inertial>
 		</link>
-		<link name="$(arg namespace)J1">
+		<link name="${namespace}J1">
 			<visual>
 				<origin rpy="0 0 0" xyz="0 0 0"/>
@@ -45,13 +45,13 @@
 			</inertial>
 		</link>
-		<joint name="$(arg namespace)joint_1" type="revolute">
-			<parent link="$(arg namespace)base_link"/>
-			<child link="$(arg namespace)J1"/>
+		<joint name="${namespace}joint_1" type="revolute">
+			<parent link="${namespace}base_link"/>
+			<child link="${namespace}J1"/>
 			<origin rpy="0.000000 0.000000 0.000000" xyz="0.000000 0.000000 0.000000"/>
 			<axis xyz="-0.000000 -0.000000 1.000000"/>
-			<limit effort="1" lower="-2.61799387799149" upper="2.61799387799149" velocity="1.62490153360672"/>
+			<limit effort="1" lower="-2.61799387799149" upper="2.61799387799149" velocity="${radians(23.1)}"/>
 			<dynamics damping="0" friction="0"/>
 		</joint>
-		<link name="$(arg namespace)J2">
+		<link name="${namespace}J2">
 			<visual>
 				<origin rpy="0 0 0" xyz="0 0 0"/>
@@ -72,13 +72,13 @@
 			</inertial>
 		</link>
-		<joint name="$(arg namespace)joint_2" type="revolute">
-			<parent link="$(arg namespace)J1"/>
-			<child link="$(arg namespace)J2"/>
+		<joint name="${namespace}joint_2" type="revolute">
+			<parent link="${namespace}J1"/>
+			<child link="${namespace}J2"/>
 			<origin rpy="0.000000 0.000000 0.000000" xyz="0.000000 0.000000 0.180000"/>
 			<axis xyz="-0.000000 1.000000 -0.000000"/>
-			<limit effort="1" lower="-1.0471975511966" upper="1.74532925199433" velocity="0.759226951263793"/>
+			<limit effort="1" lower="-1.0471975511966" upper="1.74532925199433" velocity="${radians(22.47)}"/>
 			<dynamics damping="0" friction="0"/>
 		</joint>
-		<link name="$(arg namespace)J3">
+		<link name="${namespace}J3">
 			<visual>
 				<origin rpy="0 0 0" xyz="0 0 0"/>
@@ -99,13 +99,13 @@
 			</inertial>
 		</link>
-		<joint name="$(arg namespace)joint_3" type="revolute">
-			<parent link="$(arg namespace)J2"/>
-			<child link="$(arg namespace)J3"/>
+		<joint name="${namespace}joint_3" type="revolute">
+			<parent link="${namespace}J2"/>
+			<child link="${namespace}J3"/>
 			<origin rpy="0.000000 0.000000 0.000000" xyz="0.000000 0.000000 0.165000"/>
 			<axis xyz="-0.000000 1.000000 -0.000000"/>
-			<limit effort="1" lower="0.314159265358979" upper="2.44346095279206" velocity="1.66187633381022"/>
+			<limit effort="1" lower="0.314159265358979" upper="2.44346095279206" velocity="${radians(41.58)}"/>
 			<dynamics damping="0" friction="0"/>
 		</joint>
-		<link name="$(arg namespace)J4">
+		<link name="${namespace}J4">
 			<visual>
 				<origin rpy="0 0 0" xyz="0 0 0"/>
@@ -126,13 +126,13 @@
 			</inertial>
 		</link>
-		<joint name="$(arg namespace)joint_4" type="revolute">
-			<parent link="$(arg namespace)J3"/>
-			<child link="$(arg namespace)J4"/>
+		<joint name="${namespace}joint_4" type="revolute">
+			<parent link="${namespace}J3"/>
+			<child link="${namespace}J4"/>
 			<origin rpy="0.000000 0.000000 0.000000" xyz="-0.012000 0.020000 -0.345000"/>
 			<axis xyz="-0.000000 -0.000000 1.000000"/>
-			<limit effort="1" lower="-2.96705972839036" upper="2.96705972839036" velocity="2.5534166956677"/>
+			<limit effort="1" lower="-2.96705972839036" upper="2.96705972839036" velocity="${radians(42.35)}"/>
 			<dynamics damping="0" friction="0"/>
 		</joint>
-		<link name="$(arg namespace)J5">
+		<link name="${namespace}J5">
 			<visual>
 				<origin rpy="0 0 0" xyz="0 0 0"/>
@@ -153,13 +153,13 @@
 			</inertial>
 		</link>
-		<joint name="$(arg namespace)joint_5" type="revolute">
-			<parent link="$(arg namespace)J4"/>
-			<child link="$(arg namespace)J5"/>
+		<joint name="${namespace}joint_5" type="revolute">
+			<parent link="${namespace}J4"/>
+			<child link="${namespace}J5"/>
 			<origin rpy="0.000000 0.000000 0.000000" xyz="0.000000 -0.020000 0.522500"/>
 			<axis xyz="-0.000000 1.000000 -0.000000"/>
-			<limit effort="1" lower="-1.65806278939461" upper="2.35619449019234" velocity="2.66948109092533"/>
+			<limit effort="1" lower="-1.65806278939461" upper="2.35619449019234" velocity="${radians(42.35)}"/>
 			<dynamics damping="0" friction="0"/>
 		</joint>
-		<link name="$(arg namespace)J6">
+		<link name="${namespace}J6">
 			<visual>
 				<origin rpy="0 0 0" xyz="0 0 0"/>
@@ -180,11 +180,17 @@
 			</inertial>
 		</link>
-		<joint name="$(arg namespace)joint_6" type="revolute">
-			<parent link="$(arg namespace)J5"/>
-			<child link="$(arg namespace)J6"/>
+		<joint name="${namespace}joint_6" type="revolute">
+			<parent link="${namespace}J5"/>
+			<child link="${namespace}J6"/>
 			<origin rpy="0.000000 0.000000 0.000000" xyz="0.000000 -0.044500 0.042000"/>
 			<axis xyz="-0.000000 -0.000000 1.000000"/>
-			<limit effort="1" lower="-2.96705972839036" upper="2.96705972839036" velocity="3.83012504350156"/>
+			<limit effort="1" lower="-2.96705972839036" upper="2.96705972839036" velocity="${radians(63.56)}"/>
 			<dynamics damping="0" friction="0"/>
+		</joint>
+		<link name="${namespace}flange"/>
+		<joint name="${namespace}J6-flange" type="fixed">
+			<parent link="${namespace}J6"/>
+			<child link="${namespace}flange"/>
+			<origin rpy="0 0 0" xyz="0 0 0"/>
 		</joint>
 	</xacro:macro>

File: denso_robot_descriptions/robots/cobotta/urdf/denso_robot_macro.xacro (robot description, xacro)
@@ -12,11 +12,13 @@
     model
     namespace
+    parent
+    *origin
     transmission_hw_interface:=hardware_interface/PositionJointInterface
     sim:=false
+    gz_cam:=false
     ip_address
     send_format
     recv_format
-    verbose:=false"
-  >
+    verbose:=false">
     <!-- Robot data required by the denso driver -->
     <xacro:arg name="ip_address" default="192.168.0.1"/>
@@ -39,10 +41,17 @@
     <!-- ros2 control include -->
     <xacro:include filename="$(find denso_robot_descriptions)/robots/$(arg model)/urdf/denso_robot.ros2_control.xacro" />
+    <!-- For other tools, modify the filename parameter to the path of your tool's xacro file. -->
+    <!-- The line with tag xacro:tool passes the parameters defined in your tool's xacro file -->
+    <!-- (see gz_cam.xacro as an example implementation) -->
+    <xacro:if value="$(arg gz_cam)">
+      <xacro:include filename="$(find denso_robot_gazebo)/sensors/gz_cam/urdf/gz_cam.xacro" />
+    </xacro:if>
     <!-- ros2 control instance -->
     <xacro:denso_robot_ros2_control
-      name="GazeboSystem" namespace="$(arg namespace)"
+      name="Cobotta"
+      namespace="${namespace}"
       sim="$(arg sim)"
       model="$(arg model)"
-      ip_address="$(arg ip_address)"
+      ip_address="${ip_address}"
       robot_name="$(arg robot_name)"
       robot_joints="$(arg robot_joints)"
@@ -59,13 +68,13 @@
       recv_format="$(arg recv_format)" />
     <!-- Add URDF transmission elements (for ros_control) -->
-    <xacro:denso_robot_arm_transmission namespace="$(arg namespace)" hw_interface="$(arg transmission_hw_interface)" />
+    <xacro:denso_robot_arm_transmission namespace="${namespace}" hw_interface="$(arg transmission_hw_interface)" />
     <!-- Placeholder for ros2_control transmission which don't yet exist -->
-    <!-- links -  main serial chain -->
-    <xacro:denso_robot_arm_kinematics namespace="$(arg namespace)" model="$(arg model)" />
-    <gazebo>
-	    <plugin filename="gz_ros2_control-system" name="gz_ros2_control::GazeboSimROS2ControlPlugin">
-      		<parameters>$(find denso_robot_moveit_config)/robots/$(arg model)/config/denso_robot_controllers.yaml</parameters>
-    	</plugin>
-  	</gazebo>
+    <!-- links - main serial chain -->
+    <xacro:denso_robot_arm_kinematics namespace="${namespace}" model="$(arg model)" parent="${parent}">
+      <xacro:insert_block name="origin" />
+    </xacro:denso_robot_arm_kinematics>
+    <xacro:if value="$(arg gz_cam)">
+      <xacro:gz_cam namespace="${namespace}" />
+    </xacro:if>
   </xacro:macro>
 </robot>

File: denso_robot_moveit_config/robots/cobotta/srdf/denso_robot_macro.srdf.xacro (robot description, xacro)
@@ -5,5 +5,5 @@
     A URDF file must exist for this robot as well, where the joints and the links that are referenced are defined
 -->
-  <xacro:macro name="denso_robot_srdf" params="name namespace">
+  <xacro:macro name="denso_robot_srdf" params="namespace">
     <!--GROUPS - Representation of a set of joints and links. This can be useful for specifying DOF to plan for, defining arms, end effectors, etc-->
     <!--LINKS - When a link is specified, the parent joint of that link (if it exists) is automatically included-->
@@ -12,11 +12,11 @@
     <!--SUBGROUPS - Groups can also be formed by referencing to already defined group names-->
     <group name="${namespace}arm">
-		<joint name="$(arg namespace)joint_1"/>
-		<joint name="$(arg namespace)joint_2"/>
-		<joint name="$(arg namespace)joint_3"/>
-		<joint name="$(arg namespace)joint_4"/>
-		<joint name="$(arg namespace)joint_5"/>
-		<joint name="$(arg namespace)joint_6"/>
-	</group>
+      <joint name="${namespace}joint_1"/>
+      <joint name="${namespace}joint_2"/>
+      <joint name="${namespace}joint_3"/>
+      <joint name="${namespace}joint_4"/>
+      <joint name="${namespace}joint_5"/>
+      <joint name="${namespace}joint_6"/>
+    </group>
     <!--GROUP STATES - Purpose - Define a named state for a particular group, in terms of joint values. This is useful to define states like 'folded arms'-->
     <!--END EFFECTOR - Purpose - Represent information about an end effector.-->
@@ -24,12 +24,12 @@
     <virtual_joint name="${namespace}fixed_base" type="fixed" parent_frame="world" child_link="${namespace}base_link" />
     <!--DISABLE COLLISIONS - By default it is assumed that any link of the robot could potentially come into collision with any other link in the robot. This tag disables collision checking between a specified pair of links. -->
-	<disable_collisions link1="$(arg namespace)J6" link2="$(arg namespace)J3" reason="Never"/>
-	<disable_collisions link1="$(arg namespace)J6" link2="$(arg namespace)J5" reason="Adjacent"/>
-	<disable_collisions link1="$(arg namespace)J1" link2="$(arg namespace)J2" reason="Adjacent"/>
-	<disable_collisions link1="$(arg namespace)J1" link2="$(arg namespace)base_link" reason="Adjacent"/>
-	<disable_collisions link1="$(arg namespace)J2" link2="$(arg namespace)J3" reason="Adjacent"/>
-	<disable_collisions link1="$(arg namespace)J3" link2="$(arg namespace)J4" reason="Adjacent"/>
-	<disable_collisions link1="$(arg namespace)J3" link2="$(arg namespace)J5" reason="Never"/>
-	<disable_collisions link1="$(arg namespace)J4" link2="$(arg namespace)J5" reason="Adjacent"/>
+    <disable_collisions link1="${namespace}J6" link2="${namespace}J3" reason="Never"/>
+    <disable_collisions link1="${namespace}J6" link2="${namespace}J5" reason="Adjacent"/>
+    <disable_collisions link1="${namespace}J1" link2="${namespace}J2" reason="Adjacent"/>
+    <disable_collisions link1="${namespace}J1" link2="${namespace}base_link" reason="Adjacent"/>
+    <disable_collisions link1="${namespace}J2" link2="${namespace}J3" reason="Adjacent"/>
+    <disable_collisions link1="${namespace}J3" link2="${namespace}J4" reason="Adjacent"/>
+    <disable_collisions link1="${namespace}J3" link2="${namespace}J5" reason="Never"/>
+    <disable_collisions link1="${namespace}J4" link2="${namespace}J5" reason="Adjacent"/>
   </xacro:macro>
 </robot>
