Commit message: feat(cobotta): add cobotta support and fix kinematics/inertial data

File: denso_robot_descriptions/robots/cobotta/urdf/denso_robot_kinematics.xacro (robot description, xacro)
@@ -1,191 +1,269 @@
 <?xml version='1.0' encoding='UTF-8'?>
 <robot xmlns:xacro="http://www.ros.org/wiki/xacro">
-	<xacro:macro name="denso_robot_arm_kinematics" params="namespace model">
-		<link name="world"/>
-		<joint name="$(arg namespace)joint_w" type="fixed">
-			<parent link="world"/>
-			<child link="$(arg namespace)base_link"/>
-		</joint>
-		<link name="$(arg namespace)base_link">
-			<visual>
-				<origin rpy="0 0 0" xyz="0 0 0"/>
-				<geometry>
-					<mesh filename="file:///$(find denso_robot_descriptions)/robots/$(arg model)/meshes/base_link.dae" scale="1 1 1"/>
-				</geometry>
-			</visual>
-			<collision>
-				<origin rpy="0 0 0" xyz="0 0 0"/>
-				<geometry>
-					<mesh filename="file:///$(find denso_robot_descriptions)/robots/$(arg model)/meshes/base_link.dae" scale="1 1 1"/>
-				</geometry>
-			</collision>
-			<inertial>
-				<mass value="1"/>
-				<origin rpy="0.000000 0.000000 0.000000" xyz="0.000000 0.000000 0.000000"/>
-				<inertia ixx="1" ixy="0" ixz="0" iyy="1" iyz="0" izz="1"/>
-			</inertial>
-		</link>
-		<link name="$(arg namespace)J1">
-			<visual>
-				<origin rpy="0 0 0" xyz="0 0 0"/>
-				<geometry>
-					<mesh filename="file:///$(find denso_robot_descriptions)/robots/$(arg model)/meshes/J1.dae" scale="1 1 1"/>
-				</geometry>
-			</visual>
-			<collision>
-				<origin rpy="0 0 0" xyz="0 0 0"/>
-				<geometry>
-					<mesh filename="file:///$(find denso_robot_descriptions)/robots/$(arg model)/meshes/J1.dae" scale="1 1 1"/>
-				</geometry>
-			</collision>
-			<inertial>
-				<mass value="1"/>
-				<origin rpy="0.000000 0.000000 0.000000" xyz="0.000000 0.000000 0.000000"/>
-				<inertia ixx="1" ixy="0" ixz="0" iyy="1" iyz="0" izz="1"/>
-			</inertial>
-		</link>
-		<joint name="$(arg namespace)joint_1" type="revolute">
-			<parent link="$(arg namespace)base_link"/>
-			<child link="$(arg namespace)J1"/>
-			<origin rpy="0.000000 0.000000 0.000000" xyz="0.000000 0.000000 0.000000"/>
-			<axis xyz="-0.000000 -0.000000 1.000000"/>
-			<limit effort="1" lower="-2.61799387799149" upper="2.61799387799149" velocity="1.62490153360672"/>
-			<dynamics damping="0" friction="0"/>
-		</joint>
-		<link name="$(arg namespace)J2">
-			<visual>
-				<origin rpy="0 0 0" xyz="0 0 0"/>
-				<geometry>
-					<mesh filename="file:///$(find denso_robot_descriptions)/robots/$(arg model)/meshes/J2.dae" scale="1 1 1"/>
-				</geometry>
-			</visual>
-			<collision>
-				<origin rpy="0 0 0" xyz="0 0 0"/>
-				<geometry>
-					<mesh filename="file:///$(find denso_robot_descriptions)/robots/$(arg model)/meshes/J2.dae" scale="1 1 1"/>
-				</geometry>
-			</collision>
-			<inertial>
-				<mass value="1"/>
-				<origin rpy="0.000000 0.000000 0.000000" xyz="0.000000 0.000000 0.000000"/>
-				<inertia ixx="1" ixy="0" ixz="0" iyy="1" iyz="0" izz="1"/>
-			</inertial>
-		</link>
-		<joint name="$(arg namespace)joint_2" type="revolute">
-			<parent link="$(arg namespace)J1"/>
-			<child link="$(arg namespace)J2"/>
-			<origin rpy="0.000000 0.000000 0.000000" xyz="0.000000 0.000000 0.180000"/>
-			<axis xyz="-0.000000 1.000000 -0.000000"/>
-			<limit effort="1" lower="-1.0471975511966" upper="1.74532925199433" velocity="0.759226951263793"/>
-			<dynamics damping="0" friction="0"/>
-		</joint>
-		<link name="$(arg namespace)J3">
-			<visual>
-				<origin rpy="0 0 0" xyz="0 0 0"/>
-				<geometry>
-					<mesh filename="file:///$(find denso_robot_descriptions)/robots/$(arg model)/meshes/J3.dae" scale="1 1 1"/>
-				</geometry>
-			</visual>
-			<collision>
-				<origin rpy="0 0 0" xyz="0 0 0"/>
-				<geometry>
-					<mesh filename="file:///$(find denso_robot_descriptions)/robots/$(arg model)/meshes/J3.dae" scale="1 1 1"/>
-				</geometry>
-			</collision>
-			<inertial>
-				<mass value="1"/>
-				<origin rpy="0.000000 0.000000 0.000000" xyz="0.000000 0.000000 0.000000"/>
-				<inertia ixx="1" ixy="0" ixz="0" iyy="1" iyz="0" izz="1"/>
-			</inertial>
-		</link>
-		<joint name="$(arg namespace)joint_3" type="revolute">
-			<parent link="$(arg namespace)J2"/>
-			<child link="$(arg namespace)J3"/>
-			<origin rpy="0.000000 0.000000 0.000000" xyz="0.000000 0.000000 0.165000"/>
-			<axis xyz="-0.000000 1.000000 -0.000000"/>
-			<limit effort="1" lower="0.314159265358979" upper="2.44346095279206" velocity="1.66187633381022"/>
-			<dynamics damping="0" friction="0"/>
-		</joint>
-		<link name="$(arg namespace)J4">
-			<visual>
-				<origin rpy="0 0 0" xyz="0 0 0"/>
-				<geometry>
-					<mesh filename="file:///$(find denso_robot_descriptions)/robots/$(arg model)/meshes/J4.dae" scale="1 1 1"/>
-				</geometry>
-			</visual>
-			<collision>
-				<origin rpy="0 0 0" xyz="0 0 0"/>
-				<geometry>
-					<mesh filename="file:///$(find denso_robot_descriptions)/robots/$(arg model)/meshes/J4.dae" scale="1 1 1"/>
-				</geometry>
-			</collision>
-			<inertial>
-				<mass value="1"/>
-				<origin rpy="0.000000 0.000000 0.000000" xyz="0.000000 0.000000 0.000000"/>
-				<inertia ixx="1" ixy="0" ixz="0" iyy="1" iyz="0" izz="1"/>
-			</inertial>
-		</link>
-		<joint name="$(arg namespace)joint_4" type="revolute">
-			<parent link="$(arg namespace)J3"/>
-			<child link="$(arg namespace)J4"/>
-			<origin rpy="0.000000 0.000000 0.000000" xyz="-0.012000 0.020000 -0.345000"/>
-			<axis xyz="-0.000000 -0.000000 1.000000"/>
-			<limit effort="1" lower="-2.96705972839036" upper="2.96705972839036" velocity="2.5534166956677"/>
-			<dynamics damping="0" friction="0"/>
-		</joint>
-		<link name="$(arg namespace)J5">
-			<visual>
-				<origin rpy="0 0 0" xyz="0 0 0"/>
-				<geometry>
-					<mesh filename="file:///$(find denso_robot_descriptions)/robots/$(arg model)/meshes/J5.dae" scale="1 1 1"/>
-				</geometry>
-			</visual>
-			<collision>
-				<origin rpy="0 0 0" xyz="0 0 0"/>
-				<geometry>
-					<mesh filename="file:///$(find denso_robot_descriptions)/robots/$(arg model)/meshes/J5.dae" scale="1 1 1"/>
-				</geometry>
-			</collision>
-			<inertial>
-				<mass value="1"/>
-				<origin rpy="0.000000 0.000000 0.000000" xyz="0.000000 0.000000 0.000000"/>
-				<inertia ixx="1" ixy="0" ixz="0" iyy="1" iyz="0" izz="1"/>
-			</inertial>
-		</link>
-		<joint name="$(arg namespace)joint_5" type="revolute">
-			<parent link="$(arg namespace)J4"/>
-			<child link="$(arg namespace)J5"/>
-			<origin rpy="0.000000 0.000000 0.000000" xyz="0.000000 -0.020000 0.522500"/>
-			<axis xyz="-0.000000 1.000000 -0.000000"/>
-			<limit effort="1" lower="-1.65806278939461" upper="2.35619449019234" velocity="2.66948109092533"/>
-			<dynamics damping="0" friction="0"/>
-		</joint>
-		<link name="$(arg namespace)J6">
-			<visual>
-				<origin rpy="0 0 0" xyz="0 0 0"/>
-				<geometry>
-					<mesh filename="file:///$(find denso_robot_descriptions)/robots/$(arg model)/meshes/J6.dae" scale="1 1 1"/>
-				</geometry>
-			</visual>
-			<collision>
-				<origin rpy="0 0 0" xyz="0 0 0"/>
-				<geometry>
-					<mesh filename="file:///$(find denso_robot_descriptions)/robots/$(arg model)/meshes/J6.dae" scale="1 1 1"/>
-				</geometry>
-			</collision>
-			<inertial>
-				<mass value="1"/>
-				<origin rpy="0.000000 0.000000 0.000000" xyz="0.000000 0.000000 0.000000"/>
-				<inertia ixx="1" ixy="0" ixz="0" iyy="1" iyz="0" izz="1"/>
-			</inertial>
-		</link>
-		<joint name="$(arg namespace)joint_6" type="revolute">
-			<parent link="$(arg namespace)J5"/>
-			<child link="$(arg namespace)J6"/>
-			<origin rpy="0.000000 0.000000 0.000000" xyz="0.000000 -0.044500 0.042000"/>
-			<axis xyz="-0.000000 -0.000000 1.000000"/>
-			<limit effort="1" lower="-2.96705972839036" upper="2.96705972839036" velocity="3.83012504350156"/>
-			<dynamics damping="0" friction="0"/>
-		</joint>
-	</xacro:macro>
+  <xacro:macro name="denso_robot_arm_kinematics" params="namespace model parent *origin">
+    <joint name="${namespace}joint_w" type="fixed">
+      <xacro:insert_block name="origin" />
+      <parent link="${parent}" />
+      <child link="${namespace}base_link" />
+    </joint>
+    <link name="${namespace}base_link">
+      <visual>
+        <origin rpy="0 0 0" xyz="0 0 0" />
+        <geometry>
+          <mesh
+            filename="file:///$(find denso_robot_descriptions)/robots/$(arg model)/meshes/base_link.dae"
+            scale="1 1 1" />
+        </geometry>
+      </visual>
+      <collision>
+        <origin rpy="0 0 0" xyz="0 0 0" />
+        <geometry>
+          <mesh
+            filename="file:///$(find denso_robot_descriptions)/robots/$(arg model)/meshes/base_link.dae"
+            scale="1 1 1" />
+        </geometry>
+      </collision>
+      <inertial>
+        <mass value="1.685" />
+        <origin rpy="0.000000 0.000000 0.000000" xyz="-2.13096893e-02 2.22019729e-06 4.40110144e-02" />
+        <inertia ixx="3.18266625e-06" ixy="0" ixz="0" iyy="4.31224522e-06" iyz="0"
+          izz="4.84185879e-06" />
+      </inertial>
+    </link>
+    <link name="${namespace}J1">
+      <visual>
+        <origin rpy="0 0 0" xyz="0 0 0" />
+        <geometry>
+          <mesh
+            filename="file:///$(find denso_robot_descriptions)/robots/$(arg model)/meshes/J1.dae"
+            scale="1 1 1" />
+        </geometry>
+      </visual>
+      <collision>
+        <origin rpy="0 0 0" xyz="0 0 0" />
+        <geometry>
+          <mesh
+            filename="file:///$(find denso_robot_descriptions)/robots/$(arg model)/meshes/J1.dae"
+            scale="1 1 1" />
+        </geometry>
+      </collision>
+      <inertial>
+        <mass value="0.710" />
+        <origin rpy="0.000000 0.000000 0.000000" xyz="5.97644313e-08 7.16199291e-03 1.58026984e-01" />
+        <inertia ixx="1.03970662e-06" ixy="0" ixz="0" iyy="9.08490662e-07" iyz="0"
+          izz="7.81158752e-07" />
+      </inertial>
+    </link>
+    <joint name="${namespace}joint_1" type="revolute">
+      <parent link="${namespace}base_link" />
+      <child link="${namespace}J1" />
+      <origin rpy="0.000000 0.000000 0.000000" xyz="0.000000 0.000000 0.000000" />
+      <axis xyz="-0.000000 -0.000000 1.000000" />
+      <!-- Initially, a negative effort value acting as a sentinel indicating "no limit" (treated as
+      infinity) was used,
+			but this was changed following the error on line 175 of
+			https://github.com/gazebosim/gz-physics/blob/ign-physics5/dartsim/src/JointFeatures.cc -->
+      <limit effort="1e6" lower="${radians(-150)}" upper="${radians(150)}"
+        velocity="${radians(23.1)}" />
+      <dynamics damping="0" friction="0" />
+    </joint>
+    <link name="${namespace}J2">
+      <visual>
+        <origin rpy="0 0 0" xyz="0 0 0" />
+        <geometry>
+          <mesh
+            filename="file:///$(find denso_robot_descriptions)/robots/$(arg model)/meshes/J2.dae"
+            scale="1 1 1" />
+        </geometry>
+      </visual>
+      <collision>
+        <origin rpy="0 0 0" xyz="0 0 0" />
+        <geometry>
+          <mesh
+            filename="file:///$(find denso_robot_descriptions)/robots/$(arg model)/meshes/J2.dae"
+            scale="1 1 1" />
+        </geometry>
+      </collision>
+      <inertial>
+        <mass value="0.712" />
+        <origin rpy="0.000000 0.000000 0.000000" xyz="-0.0127344 0.08946026 0.07820109" />
+        <inertia ixx="3.31627797e-06" ixy="0" ixz="0" iyy="3.46094967e-06" iyz="0"
+          izz="4.75952442e-07" />
+      </inertial>
+    </link>
+    <joint name="${namespace}joint_2" type="revolute">
+      <parent link="${namespace}J1" />
+      <child link="${namespace}J2" />
+      <origin rpy="0.000000 0.000000 0.000000" xyz="0.000000 0.000000 0.180000" />
+      <axis xyz="-0.000000 1.000000 -0.000000" />
+      <!-- Initially, a negative effort value acting as a sentinel indicating "no limit" (treated as
+      infinity) was used,
+			but this was changed following the error on line 175 of
+			https://github.com/gazebosim/gz-physics/blob/ign-physics5/dartsim/src/JointFeatures.cc -->
+      <limit effort="1e6" lower="${radians(-60)}" upper="${radians(100)}"
+        velocity="${radians(22.47)}" />
+      <dynamics damping="0" friction="0" />
+    </joint>
+    <link name="${namespace}J3">
+      <visual>
+        <origin rpy="0 0 0" xyz="0 0 0" />
+        <geometry>
+          <mesh
+            filename="file:///$(find denso_robot_descriptions)/robots/$(arg model)/meshes/J3.dae"
+            scale="1 1 1" />
+        </geometry>
+      </visual>
+      <collision>
+        <origin rpy="0 0 0" xyz="0 0 0" />
+        <geometry>
+          <mesh
+            filename="file:///$(find denso_robot_descriptions)/robots/$(arg model)/meshes/J3.dae"
+            scale="1 1 1" />
+        </geometry>
+      </collision>
+      <inertial>
+        <mass value="0.411" />
+        <origin rpy="0.000000 0.000000 0.000000" xyz="-0.00530934 0.02317424 0.02748904" />
+        <inertia ixx="5.44102812e-07" ixy="0" ixz="0" iyy="5.36692738e-07" iyz="0"
+          izz="2.36621010e-07" />
+      </inertial>
+    </link>
+    <joint name="${namespace}joint_3" type="revolute">
+      <parent link="${namespace}J2" />
+      <child link="${namespace}J3" />
+      <origin rpy="0.000000 0.000000 0.000000" xyz="0.000000 0.000000 0.165000" />
+      <axis xyz="-0.000000 1.000000 -0.000000" />
+      <!-- Initially, a negative effort value acting as a sentinel indicating "no limit" (treated as
+      infinity) was used,
+			but this was changed following the error on line 175 of
+			https://github.com/gazebosim/gz-physics/blob/ign-physics5/dartsim/src/JointFeatures.cc -->
+      <limit effort="1e6" lower="${radians(18)}" upper="${radians(140)}"
+        velocity="${radians(41.58)}" />
+      <dynamics damping="0" friction="0" />
+    </joint>
+    <link name="${namespace}J4">
+      <visual>
+        <origin rpy="0 0 0" xyz="0 0 0" />
+        <geometry>
+          <mesh
+            filename="file:///$(find denso_robot_descriptions)/robots/$(arg model)/meshes/J4.dae"
+            scale="1 1 1" />
+        </geometry>
+      </visual>
+      <collision>
+        <origin rpy="0 0 0" xyz="0 0 0" />
+        <geometry>
+          <mesh
+            filename="file:///$(find denso_robot_descriptions)/robots/$(arg model)/meshes/J4.dae"
+            scale="1 1 1" />
+        </geometry>
+      </collision>
+      <inertial>
+        <mass value="0.305" />
+        <origin rpy="0.000000 0.000000 0.000000" xyz="-3.09596454e-06 -1.84459215e-03 4.87930791e-01" />
+        <inertia ixx="3.70943790e-07" ixy="0" ixz="0" iyy="3.63684800e-07" iyz="0"
+          izz="1.29385899e-07" />
+      </inertial>
+    </link>
+    <joint name="${namespace}joint_4" type="revolute">
+      <parent link="${namespace}J3" />
+      <child link="${namespace}J4" />
+      <origin rpy="0.000000 0.000000 0.000000" xyz="-0.012000 0.020000 -0.345000" />
+      <axis xyz="-0.000000 -0.000000 1.000000" />
+      <!-- Initially, a negative effort value acting as a sentinel indicating "no limit" (treated as
+      infinity) was used,
+			but this was changed following the error on line 175 of
+			https://github.com/gazebosim/gz-physics/blob/ign-physics5/dartsim/src/JointFeatures.cc -->
+      <limit effort="1e6" lower="${radians(-170)}" upper="${radians(170)}"
+        velocity="${radians(42.35)}" />
+      <dynamics damping="0" friction="0" />
+    </joint>
+    <link name="${namespace}J5">
+      <visual>
+        <origin rpy="0 0 0" xyz="0 0 0" />
+        <geometry>
+          <mesh
+            filename="file:///$(find denso_robot_descriptions)/robots/$(arg model)/meshes/J5.dae"
+            scale="1 1 1" />
+        </geometry>
+      </visual>
+      <collision>
+        <origin rpy="0 0 0" xyz="0 0 0" />
+        <geometry>
+          <mesh
+            filename="file:///$(find denso_robot_descriptions)/robots/$(arg model)/meshes/J5.dae"
+            scale="1 1 1" />
+        </geometry>
+      </collision>
+      <inertial>
+        <mass value="0.171" />
+        <origin rpy="0.000000 0.000000 0.000000" xyz="-6.03044393e-06 -4.07093619e-02 8.17389682e-03" />
+        <inertia ixx="8.95222593e-08" ixy="0" ixz="0" iyy="8.16419651e-08" iyz="0"
+          izz="7.42211107e-08" />
+      </inertial>
+    </link>
+    <joint name="${namespace}joint_5" type="revolute">
+      <parent link="${namespace}J4" />
+      <child link="${namespace}J5" />
+      <origin rpy="0.000000 0.000000 0.000000" xyz="0.000000 -0.020000 0.522500" />
+      <axis xyz="-0.000000 1.000000 -0.000000" />
+      <!-- Initially, a negative effort value acting as a sentinel indicating "no limit" (treated as
+      infinity) was used,
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