Commit message: feat(cobotta): add cobotta support and fix kinematics/inertial data

File: denso_robot_descriptions/robots/cobotta/urdf/denso_robot_macro.xacro (robot description, xacro)
@@ -1,4 +1,4 @@
 <?xml version="1.0"?>
-<robot xmlns:xacro="http://wiki.ros.org/xacro">
+<robot xmlns:xacro="http://www.ros.org/wiki/xacro">
   <!--
     Base Denso robot xacro macro.
@@ -9,40 +9,54 @@
     Author DENSO WAVE INCORPORATED
   -->
-  <xacro:macro name="denso_robot" params="
-    model
-    namespace
-    transmission_hw_interface:=hardware_interface/PositionJointInterface
-    sim:=false
-    ip_address
-    send_format
-    recv_format
-    verbose:=false"
-  >
+  <xacro:macro name="denso_robot" params="model
+                                          namespace
+                                          parent
+                                          *origin
+                                          transmission_hw_interface:=hardware_interface/PositionJointInterface
+                                          sim:=false
+                                          gz_cam:=false
+                                          ip_address
+                                          send_format
+                                          recv_format
+                                          verbose:=false">
     <!-- Robot data required by the denso driver -->
-    <xacro:arg name="ip_address" default="192.168.0.1"/>
-    <xacro:arg name="robot_name" default="CVR038A1-NV6-NN"/> <!-- "robot_name" param must be consistent with the @TYPE_NAME variable of the real robot !! -->
-    <xacro:arg name="robot_joints" default="6"/> <!-- number of total joints in the kinematic chain -->
-    <xacro:arg name="joint_1" default="1"/> <!-- 0 = prismatic , 1 = revolute -->
-    <xacro:arg name="joint_2" default="1"/> <!-- 0 = prismatic , 1 = revolute -->
-    <xacro:arg name="joint_3" default="1"/> <!-- 0 = prismatic , 1 = revolute -->
-    <xacro:arg name="joint_4" default="1"/> <!-- 0 = prismatic , 1 = revolute -->
-    <xacro:arg name="joint_5" default="1"/> <!-- 0 = prismatic , 1 = revolute -->
-    <xacro:arg name="joint_6" default="1"/> <!-- 0 = prismatic , 1 = revolute -->
-    <xacro:arg name="controller_type" default="8"/> <!-- 8 = RC8 , 9 = RC9 -->
-    <xacro:arg name="arm_group" default="0"/>
-    <xacro:arg name="send_format" default="288"/>
-    <xacro:arg name="recv_format" default="292"/>
-    <xacro:arg name="verbose" default="false"/>
-    <xacro:include filename="$(find denso_robot_descriptions)/robots/$(arg model)/urdf/denso_robot_transmissions.xacro" />
+    <xacro:arg name="ip_address" default="" />
+    <xacro:arg name="robot_name" default="CVR038A1-NV6-NN" /> <!-- "robot_name" param must be
+    consistent with the @TYPE_NAME variable of the real robot !! -->
+    <xacro:arg name="robot_joints" default="6" /> <!-- number of total joints in the kinematic chain -->
+    <xacro:arg name="joint_1" default="1" /> <!-- 0 = prismatic , 1 = revolute -->
+    <xacro:arg name="joint_2" default="1" /> <!-- 0 = prismatic , 1 = revolute -->
+    <xacro:arg name="joint_3" default="1" /> <!-- 0 = prismatic , 1 = revolute -->
+    <xacro:arg name="joint_4" default="1" /> <!-- 0 = prismatic , 1 = revolute -->
+    <xacro:arg name="joint_5" default="1" /> <!-- 0 = prismatic , 1 = revolute -->
+    <xacro:arg name="joint_6" default="1" /> <!-- 0 = prismatic , 1 = revolute -->
+    <xacro:arg name="controller_type" default="8" /> <!-- 8 = RC8 , 9 = RC9 -->
+    <xacro:arg name="arm_group" default="0" />
+    <xacro:arg name="send_format" default="288" />
+    <xacro:arg name="recv_format" default="292" />
+    <xacro:arg name="verbose" default="false" />
+    <!-- initial position for simulations-->
+    <xacro:arg name="initial_positions_file"
+      default="$(find denso_robot_moveit_config)/robots/$(arg model)/config/initial_positions.yaml" />
+    <xacro:include
+      filename="$(find denso_robot_descriptions)/robots/$(arg model)/urdf/denso_robot_transmissions.xacro" />
     <!-- robot kinematics include -->
-    <xacro:include filename="$(find denso_robot_descriptions)/robots/$(arg model)/urdf/denso_robot_kinematics.xacro" />
+    <xacro:include
+      filename="$(find denso_robot_descriptions)/robots/$(arg model)/urdf/denso_robot_kinematics.xacro" />
     <!-- ros2 control include -->
-    <xacro:include filename="$(find denso_robot_descriptions)/robots/$(arg model)/urdf/denso_robot.ros2_control.xacro" />
+    <xacro:include
+      filename="$(find denso_robot_descriptions)/robots/$(arg model)/urdf/denso_robot.ros2_control.xacro" />
+    <!-- For other tools, modify the filename parameter to the path of your tool's xacro file. -->
+    <!-- The line with tag xacro:tool passes the parameters defined in your tool's xacro file -->
+    <!-- (see gz_cam.xacro as an example implementation) -->
+    <xacro:if value="$(arg gz_cam)">
+      <xacro:include filename="$(find denso_robot_gazebo)/sensors/gz_cam/urdf/gz_cam.xacro" />
+    </xacro:if>
     <!-- ros2 control instance -->
-    <xacro:denso_robot_ros2_control
-      name="GazeboSystem" namespace="$(arg namespace)"
+    <xacro:denso_robot_ros2_control name="Cobotta"
+      namespace="${namespace}"
       sim="$(arg sim)"
       model="$(arg model)"
-      ip_address="$(arg ip_address)"
+      ip_address="${ip_address}"
       robot_name="$(arg robot_name)"
       robot_joints="$(arg robot_joints)"
@@ -57,15 +71,18 @@
       verbose="$(arg verbose)"
       send_format="$(arg send_format)"
-      recv_format="$(arg recv_format)" />
+      recv_format="$(arg recv_format)"
+      initial_positions_file="$(arg initial_positions_file)" />
     <!-- Add URDF transmission elements (for ros_control) -->
-    <xacro:denso_robot_arm_transmission namespace="$(arg namespace)" hw_interface="$(arg transmission_hw_interface)" />
+    <xacro:denso_robot_arm_transmission namespace="${namespace}"
+      hw_interface="$(arg transmission_hw_interface)" />
     <!-- Placeholder for ros2_control transmission which don't yet exist -->
     <!-- links -  main serial chain -->
-    <xacro:denso_robot_arm_kinematics namespace="$(arg namespace)" model="$(arg model)" />
-    <gazebo>
-	    <plugin filename="gz_ros2_control-system" name="gz_ros2_control::GazeboSimROS2ControlPlugin">
-      		<parameters>$(find denso_robot_moveit_config)/robots/$(arg model)/config/denso_robot_controllers.yaml</parameters>
-    	</plugin>
-  	</gazebo>
+    <xacro:denso_robot_arm_kinematics namespace="${namespace}" model="$(arg model)"
+      parent="${parent}">
+      <xacro:insert_block name="origin" />
+    </xacro:denso_robot_arm_kinematics>
+    <xacro:if value="$(arg gz_cam)">
+      <xacro:gz_cam namespace="${namespace}" />
+    </xacro:if>
   </xacro:macro>
 </robot>

File: denso_robot_moveit_config/robots/cobotta/srdf/denso_robot_macro.srdf.xacro (robot description, xacro)
@@ -1,9 +1,9 @@
-<?xml version="1.0" encoding="UTF-8"?>
-<robot xmlns:xacro="http://wiki.ros.org/xacro">
+<?xml version="1.0"?>
+<robot xmlns:xacro="http://www.ros.org/wiki/xacro">
 <!--This does not replace URDF, and is not an extension of URDF.
     This is a format for representing semantic information about the robot structure.
     A URDF file must exist for this robot as well, where the joints and the links that are referenced are defined
 -->
-  <xacro:macro name="denso_robot_srdf" params="name namespace">
+  <xacro:macro name="denso_robot_srdf" params="namespace">
     <!--GROUPS - Representation of a set of joints and links. This can be useful for specifying DOF to plan for, defining arms, end effectors, etc-->
     <!--LINKS - When a link is specified, the parent joint of that link (if it exists) is automatically included-->
@@ -12,24 +12,39 @@
     <!--SUBGROUPS - Groups can also be formed by referencing to already defined group names-->
     <group name="${namespace}arm">
-		<joint name="$(arg namespace)joint_1"/>
-		<joint name="$(arg namespace)joint_2"/>
-		<joint name="$(arg namespace)joint_3"/>
-		<joint name="$(arg namespace)joint_4"/>
-		<joint name="$(arg namespace)joint_5"/>
-		<joint name="$(arg namespace)joint_6"/>
-	</group>
+      <chain base_link="${namespace}base_link" tip_link="${namespace}tool0" />
+    </group>
+    <group name="${namespace}end_effector">
+        <link name="${namespace}tool0"/>
+    </group>
     <!--GROUP STATES - Purpose - Define a named state for a particular group, in terms of joint values. This is useful to define states like 'folded arms'-->
+    <group_state name="${namespace}home" group="${namespace}arm">
+      <joint name="${namespace}joint_1" value="0"/>
+      <joint name="${namespace}joint_2" value="-0.5"/>
+      <joint name="${namespace}joint_3" value="1.2"/>
+      <joint name="${namespace}joint_4" value="0"/>
+      <joint name="${namespace}joint_5" value="1.5"/>
+      <joint name="${namespace}joint_6" value="0"/>
+    </group_state>
     <!--END EFFECTOR - Purpose - Represent information about an end effector.-->
+    <end_effector name="${namespace}eff" parent_link="${namespace}tool0" group="${namespace}end_effector" parent_group="${namespace}arm"/>
     <!--VIRTUAL JOINT - Purpose - this element defines a virtual joint between a robot link and an external frame of reference (considered fixed with respect to the robot)-->
     <virtual_joint name="${namespace}fixed_base" type="fixed" parent_frame="world" child_link="${namespace}base_link" />
     <!--DISABLE COLLISIONS - By default it is assumed that any link of the robot could potentially come into collision with any other link in the robot. This tag disables collision checking between a specified pair of links. -->
-	<disable_collisions link1="$(arg namespace)J6" link2="$(arg namespace)J3" reason="Never"/>
-	<disable_collisions link1="$(arg namespace)J6" link2="$(arg namespace)J5" reason="Adjacent"/>
-	<disable_collisions link1="$(arg namespace)J1" link2="$(arg namespace)J2" reason="Adjacent"/>
-	<disable_collisions link1="$(arg namespace)J1" link2="$(arg namespace)base_link" reason="Adjacent"/>
-	<disable_collisions link1="$(arg namespace)J2" link2="$(arg namespace)J3" reason="Adjacent"/>
-	<disable_collisions link1="$(arg namespace)J3" link2="$(arg namespace)J4" reason="Adjacent"/>
-	<disable_collisions link1="$(arg namespace)J3" link2="$(arg namespace)J5" reason="Never"/>
-	<disable_collisions link1="$(arg namespace)J4" link2="$(arg namespace)J5" reason="Adjacent"/>
+	  <disable_collisions link1="J1" link2="J2" reason="Adjacent"/>
+    <disable_collisions link1="J1" link2="J3" reason="Never"/>
+    <disable_collisions link1="J1" link2="J4" reason="Never"/>
+    <disable_collisions link1="J1" link2="base_link" reason="Adjacent"/>
+    <disable_collisions link1="J2" link2="J3" reason="Adjacent"/>
+    <disable_collisions link1="J2" link2="J4" reason="Never"/>
+    <disable_collisions link1="J2" link2="J5" reason="Never"/>
+    <disable_collisions link1="J2" link2="J6" reason="Never"/>
+    <disable_collisions link1="J2" link2="base_link" reason="Never"/>
+    <disable_collisions link1="J3" link2="J4" reason="Adjacent"/>
+    <disable_collisions link1="J3" link2="J5" reason="Never"/>
+    <disable_collisions link1="J3" link2="J6" reason="Never"/>
+    <disable_collisions link1="J3" link2="base_link" reason="Never"/>
+    <disable_collisions link1="J4" link2="J5" reason="Adjacent"/>
+    <disable_collisions link1="J4" link2="J6" reason="Never"/>
+    <disable_collisions link1="J5" link2="J6" reason="Adjacent"/>
   </xacro:macro>
 </robot>
