Commit message: fix(vs060): revert downgrade and restore latest description
Updates the VS060 URDF and MoveIt configuration back to the latest version, effectively undoing the restore applied in the commit e57a9b06f7040b104574736f75bf81dd3767fd68 for this specific robot. Cobotta and HSR models remain in their restored legacy state.

File: denso_robot_descriptions/robots/vs060/urdf/denso_robot_macro.xacro (robot description, xacro)
@@ -12,4 +12,6 @@
     model
     namespace
+    parent
+    *origin
     transmission_hw_interface:=hardware_interface/PositionJointInterface
     sim:=false
@@ -48,5 +50,5 @@
     <!-- ros2 control instance -->
     <xacro:denso_robot_ros2_control
-      name="GazeboSystem" namespace="$(arg namespace)"
+      name="GazeboSystem" namespace="${namespace}"
       sim="$(arg sim)"
       model="$(arg model)"
@@ -66,16 +68,13 @@
       recv_format="$(arg recv_format)" />
     <!-- Add URDF transmission elements (for ros_control) -->
-    <xacro:denso_robot_arm_transmission namespace="$(arg namespace)" hw_interface="$(arg transmission_hw_interface)" />
+    <xacro:denso_robot_arm_transmission namespace="${namespace}" hw_interface="$(arg transmission_hw_interface)" />
     <!-- Placeholder for ros2_control transmission which don't yet exist -->
     <!-- links -  main serial chain -->
-    <xacro:denso_robot_arm_kinematics namespace="$(arg namespace)" model="$(arg model)" />
+    <xacro:denso_robot_arm_kinematics namespace="${namespace}" model="$(arg model)" parent="${parent}" >
+      <xacro:insert_block name="origin" />
+    </xacro:denso_robot_arm_kinematics>
     <xacro:if value="$(arg basic_camera)">
-      <xacro:tool namespace="$(arg namespace)" />
+      <xacro:basic_camera namespace="${namespace}" end_effector="J6" />
     </xacro:if>
-    <gazebo>
-	    <plugin filename="gz_ros2_control-system" name="gz_ros2_control::GazeboSimROS2ControlPlugin">
-      		<parameters>$(find denso_robot_moveit_config)/robots/$(arg model)/config/denso_robot_controllers.yaml</parameters>
-    	</plugin>
-  	</gazebo>
   </xacro:macro>
 </robot>

File: denso_robot_moveit_config/robots/vs060/srdf/denso_robot_macro.srdf.xacro (robot description, xacro)
@@ -5,5 +5,5 @@
     A URDF file must exist for this robot as well, where the joints and the links that are referenced are defined
 -->
-  <xacro:macro name="denso_robot_srdf" params="name namespace">
+  <xacro:macro name="denso_robot_srdf" params="namespace">
     <!--GROUPS - Representation of a set of joints and links. This can be useful for specifying DOF to plan for, defining arms, end effectors, etc-->
     <!--LINKS - When a link is specified, the parent joint of that link (if it exists) is automatically included-->
@@ -12,10 +12,10 @@
     <!--SUBGROUPS - Groups can also be formed by referencing to already defined group names-->
     <group name="${namespace}arm">
-		<joint name="$(arg namespace)joint_1"/>
-		<joint name="$(arg namespace)joint_2"/>
-		<joint name="$(arg namespace)joint_3"/>
-		<joint name="$(arg namespace)joint_4"/>
-		<joint name="$(arg namespace)joint_5"/>
-		<joint name="$(arg namespace)joint_6"/>
+		<joint name="${namespace}joint_1"/>
+		<joint name="${namespace}joint_2"/>
+		<joint name="${namespace}joint_3"/>
+		<joint name="${namespace}joint_4"/>
+		<joint name="${namespace}joint_5"/>
+		<joint name="${namespace}joint_6"/>
 	</group>
     <!--GROUP STATES - Purpose - Define a named state for a particular group, in terms of joint values. This is useful to define states like 'folded arms'-->
@@ -24,12 +24,12 @@
     <virtual_joint name="${namespace}fixed_base" type="fixed" parent_frame="world" child_link="${namespace}base_link" />
     <!--DISABLE COLLISIONS - By default it is assumed that any link of the robot could potentially come into collision with any other link in the robot. This tag disables collision checking between a specified pair of links. -->
-	<disable_collisions link1="$(arg namespace)J6" link2="$(arg namespace)J3" reason="Never"/>
-	<disable_collisions link1="$(arg namespace)J6" link2="$(arg namespace)J5" reason="Adjacent"/>
-	<disable_collisions link1="$(arg namespace)J1" link2="$(arg namespace)J2" reason="Adjacent"/>
-	<disable_collisions link1="$(arg namespace)J1" link2="$(arg namespace)base_link" reason="Adjacent"/>
-	<disable_collisions link1="$(arg namespace)J2" link2="$(arg namespace)J3" reason="Adjacent"/>
-	<disable_collisions link1="$(arg namespace)J3" link2="$(arg namespace)J4" reason="Adjacent"/>
-	<disable_collisions link1="$(arg namespace)J3" link2="$(arg namespace)J5" reason="Never"/>
-	<disable_collisions link1="$(arg namespace)J4" link2="$(arg namespace)J5" reason="Adjacent"/>
+	<disable_collisions link1="${namespace}J6" link2="${namespace}J3" reason="Never"/>
+	<disable_collisions link1="${namespace}J6" link2="${namespace}J5" reason="Adjacent"/>
+	<disable_collisions link1="${namespace}J1" link2="${namespace}J2" reason="Adjacent"/>
+	<disable_collisions link1="${namespace}J1" link2="${namespace}base_link" reason="Adjacent"/>
+	<disable_collisions link1="${namespace}J2" link2="${namespace}J3" reason="Adjacent"/>
+	<disable_collisions link1="${namespace}J3" link2="${namespace}J4" reason="Adjacent"/>
+	<disable_collisions link1="${namespace}J3" link2="${namespace}J5" reason="Never"/>
+	<disable_collisions link1="${namespace}J4" link2="${namespace}J5" reason="Adjacent"/>
   </xacro:macro>
 </robot>
