Commit message: feat(vs060): enable initial joint positions support in ros2_control
Adds the ability to configure initial joint positions for the VS060
robot via a YAML file, improving simulation startup behavior.

Changes:
- Adds `initial_positions_file` argument to the VS060 macro to load
  default positions.
- Passes the position map to the ros2_control xacro definition.
- Updates joint limits to inject `initial_value` parameters into the
  position state interfaces.

File: denso_robot_descriptions/robots/vs060/urdf/denso_robot_joint_limits.xacro (robot description, xacro)
@@ -1,5 +1,5 @@
 <?xml version='1.0' encoding='UTF-8'?>
 <robot xmlns:xacro="http://www.ros.org/wiki/xacro">
-	<xacro:macro name="denso_robot_control_limits" params="namespace">
+	<xacro:macro name="denso_robot_control_limits" params="namespace initial_positions">
 		<joint name="${namespace}joint_1">
 			<command_interface name="position">
@@ -11,5 +11,7 @@
 				<param name="max">0.392699081698724</param>
 			</command_interface>
-			<state_interface name="position"/>
+			<state_interface name="position">
+				<param name="initial_value">${initial_positions['joint_1']}</param>
+			</state_interface>
 			<state_interface name="velocity"/>
 			<state_interface name="effort"/>
@@ -24,5 +26,7 @@
 				<param name="max">0.261799387799149</param>
 			</command_interface>
-			<state_interface name="position"/>
+			<state_interface name="position">
+				<param name="initial_value">${initial_positions['joint_2']}</param>
+			</state_interface>
 			<state_interface name="velocity"/>
 			<state_interface name="effort"/>
@@ -37,5 +41,7 @@
 				<param name="max">0.285832571599111</param>
 			</command_interface>
-			<state_interface name="position"/>
+			<state_interface name="position">
+				<param name="initial_value">${initial_positions['joint_3']}</param>
+			</state_interface>
 			<state_interface name="velocity"/>
 			<state_interface name="effort"/>
@@ -50,5 +56,7 @@
 				<param name="max">0.392699081698724</param>
 			</command_interface>
-			<state_interface name="position"/>
+			<state_interface name="position">
+				<param name="initial_value">${initial_positions['joint_4']}</param>
+			</state_interface>
 			<state_interface name="velocity"/>
 			<state_interface name="effort"/>
@@ -63,5 +71,7 @@
 				<param name="max">0.302168853397778</param>
 			</command_interface>
-			<state_interface name="position"/>
+			<state_interface name="position">
+				<param name="initial_value">${initial_positions['joint_5']}</param>
+			</state_interface>
 			<state_interface name="velocity"/>
 			<state_interface name="effort"/>
@@ -76,5 +86,7 @@
 				<param name="max">0.628318530717959</param>
 			</command_interface>
-			<state_interface name="position"/>
+			<state_interface name="position">
+				<param name="initial_value">${initial_positions['joint_6']}</param>
+			</state_interface>
 			<state_interface name="velocity"/>
 			<state_interface name="effort"/>

File: denso_robot_descriptions/robots/vs060/urdf/denso_robot_macro.xacro (robot description, xacro)
@@ -37,4 +37,8 @@
     <xacro:arg name="recv_format" default="292"/>
     <xacro:arg name="verbose" default="false"/>
+    <!-- initial position for simulations-->
+    <xacro:arg name="initial_positions_file" default="$(find denso_robot_descriptions)/robots/$(arg model)/initial_positions.yaml"/>
+    <!-- convert to property to use substitution in function -->
+    <xacro:property name="initial_positions_file" default="$(arg initial_positions_file)"/>
     <xacro:include filename="$(find denso_robot_descriptions)/robots/$(arg model)/urdf/denso_robot_transmissions.xacro" />
     <!-- robot kinematics include -->
@@ -66,5 +70,6 @@
       verbose="$(arg verbose)"
       send_format="$(arg send_format)"
-      recv_format="$(arg recv_format)" />
+      recv_format="$(arg recv_format)"
+      initial_positions="${xacro.load_yaml(initial_positions_file)}" />
     <!-- Add URDF transmission elements (for ros_control) -->
     <xacro:denso_robot_arm_transmission namespace="${namespace}" hw_interface="$(arg transmission_hw_interface)" />
