Commit message: feat(vs060): add vs060 support and fix kinematics/inertial data
- denso_robot_bringup: add 'vs060' to the allowed model choices
- denso_robot.ros2_control.xacro: clean up macro parameter formatting,
  rename initial_positions to initial_positions_file, and load the
  YAML file directly inside denso_robot_joint_limits.xacro instead of
  passing pre-parsed data through the macro chain
- denso_robot_joint_limits.xacro: drop hardcoded position/velocity
  command_interface limits in favor of values loaded at runtime from
  the initial positions file
- denso_robot_kinematics.xacro: add correct inertial mass/origin/
  inertia values per link, convert joint limits to use radians(),
  raise effort limits to avoid gz-physics DART errors, and add
  flange/tool0 links and joints for end-effector attachment
- denso_robot_macro.xacro / denso_robot_transmissions.xacro: fix
  xacro namespace URL, rename basic_camera to gz_cam, point
  initial_positions_file default to denso_robot_moveit_config, and
  clean up whitespace/formatting
- joint_limits.yaml: correct max_velocity values (previously in rad/s
  scaled incorrectly, now matching actual joint velocity limits)
- denso_robot_macro.srdf.xacro: fix xacro namespace and XML
  declaration, replace explicit joint list with a base_link-to-tool0
  chain, add an end_effector group/definition, a home group state,
  and expand disable_collisions pairs for non-adjacent links

This change enables full support for the vs060 robot model across
description, control, and MoveIt configuration.

File: denso_robot_descriptions/robots/vs060/urdf/denso_robot.ros2_control.xacro (robot description, xacro)
@@ -1,27 +1,38 @@
 <?xml version="1.0"?>
 <robot xmlns:xacro="http://www.ros.org/wiki/xacro">
-  <xacro:macro name="denso_robot_ros2_control" params="name namespace
-	robot_name
-    sim:=false fake_sensor_commands:=false
-    ip_address
-    model
-    robot_joints joint_1 joint_2 joint_3 joint_4 joint_5 joint_6
-    arm_group
-    send_format recv_format
-	controller_type
-    verbose
-    initial_positions
-    ">
+  <xacro:macro name="denso_robot_ros2_control"
+               params="name
+                       namespace
+                       robot_name
+                       sim:=false
+                       fake_sensor_commands:=false
+                       ip_address
+                       model
+                       robot_joints
+                       joint_1
+                       joint_2
+                       joint_3
+                       joint_4
+                       joint_5
+                       joint_6
+                       arm_group
+                       send_format
+                       recv_format
+                       controller_type
+                       verbose
+                       initial_positions_file">
     <ros2_control name="${namespace}${name}" type="system">
-	<!-- joint limits include -->
-	<xacro:include filename="$(find denso_robot_descriptions)/robots/$(arg model)/urdf/denso_robot_joint_limits.xacro" />
+      <!-- joint limits include -->
+      <xacro:include
+        filename="$(find denso_robot_descriptions)/robots/$(arg model)/urdf/denso_robot_joint_limits.xacro" />
       <hardware>
         <xacro:if value="${sim}">
-      	  <plugin>gz_ros2_control/GazeboSimSystem</plugin>
+          <plugin>gz_ros2_control/GazeboSimSystem</plugin>
         </xacro:if>
         <xacro:unless value="${sim}">
           <plugin>denso_robot_control/DensoRobotHW</plugin>
           <param name="ip_address">${ip_address}</param>
-<!-- "robot_name" param must be consistent with the @TYPE_NAME variable of the real robot !!  -->
+          <!-- "robot_name" param must be consistent with the @TYPE_NAME variable of the real robot
+          !!  -->
           <param name="robot_name">${robot_name}</param>
           <param name="node_name">denso_robot_control</param>
@@ -41,5 +52,6 @@
         </xacro:unless>
       </hardware>
-      <xacro:denso_robot_control_limits namespace="${namespace}" initial_positions="${initial_positions}" />
+      <xacro:denso_robot_control_limits namespace="${namespace}"
+        initial_positions_file="${initial_positions_file}" />
     </ros2_control>
   </xacro:macro>

File: denso_robot_descriptions/robots/vs060/urdf/denso_robot_joint_limits.xacro (robot description, xacro)
@@ -1,95 +1,61 @@
 <?xml version='1.0' encoding='UTF-8'?>
 <robot xmlns:xacro="http://www.ros.org/wiki/xacro">
-	<xacro:macro name="denso_robot_control_limits" params="namespace initial_positions">
-		<joint name="${namespace}joint_1">
-			<command_interface name="position">
-				<param name="min">-2.967060</param>
-				<param name="max">2.967060</param>
-			</command_interface>
-			<command_interface name="velocity">
-				<param name="min">0</param>
-				<param name="max">0.392699081698724</param>
-			</command_interface>
-			<state_interface name="position">
-				<param name="initial_value">${initial_positions['joint_1']}</param>
-			</state_interface>
-			<state_interface name="velocity"/>
-			<state_interface name="effort"/>
-		</joint>
-		<joint name="${namespace}joint_2">
-			<command_interface name="position">
-				<param name="min">-2.094395</param>
-				<param name="max">2.094395</param>
-			</command_interface>
-			<command_interface name="velocity">
-				<param name="min">0</param>
-				<param name="max">0.261799387799149</param>
-			</command_interface>
-			<state_interface name="position">
-				<param name="initial_value">${initial_positions['joint_2']}</param>
-			</state_interface>
-			<state_interface name="velocity"/>
-			<state_interface name="effort"/>
-		</joint>
-		<joint name="${namespace}joint_3">
-			<command_interface name="position">
-				<param name="min">-2.181662</param>
-				<param name="max">2.705260</param>
-			</command_interface>
-			<command_interface name="velocity">
-				<param name="min">0</param>
-				<param name="max">0.285832571599111</param>
-			</command_interface>
-			<state_interface name="position">
-				<param name="initial_value">${initial_positions['joint_3']}</param>
-			</state_interface>
-			<state_interface name="velocity"/>
-			<state_interface name="effort"/>
-		</joint>
-		<joint name="${namespace}joint_4">
-			<command_interface name="position">
-				<param name="min">-4.712389</param>
-				<param name="max">4.712389</param>
-			</command_interface>
-			<command_interface name="velocity">
-				<param name="min">0</param>
-				<param name="max">0.392699081698724</param>
-			</command_interface>
-			<state_interface name="position">
-				<param name="initial_value">${initial_positions['joint_4']}</param>
-			</state_interface>
-			<state_interface name="velocity"/>
-			<state_interface name="effort"/>
-		</joint>
-		<joint name="${namespace}joint_5">
-			<command_interface name="position">
-				<param name="min">-2.094395</param>
-				<param name="max">2.094395</param>
-			</command_interface>
-			<command_interface name="velocity">
-				<param name="min">0</param>
-				<param name="max">0.302168853397778</param>
-			</command_interface>
-			<state_interface name="position">
-				<param name="initial_value">${initial_positions['joint_5']}</param>
-			</state_interface>
-			<state_interface name="velocity"/>
-			<state_interface name="effort"/>
-		</joint>
-		<joint name="${namespace}joint_6">
-			<command_interface name="position">
-				<param name="min">-6.283185</param>
-				<param name="max">6.283185</param>
-			</command_interface>
-			<command_interface name="velocity">
-				<param name="min">0</param>
-				<param name="max">0.628318530717959</param>
-			</command_interface>
-			<state_interface name="position">
-				<param name="initial_value">${initial_positions['joint_6']}</param>
-			</state_interface>
-			<state_interface name="velocity"/>
-			<state_interface name="effort"/>
-		</joint>
-	</xacro:macro>
+  <xacro:macro name="denso_robot_control_limits" params="namespace initial_positions_file">
+    <xacro:property name="initial_positions"
+      value="${xacro.load_yaml(initial_positions_file)['initial_positions']}" />
+    <joint name="${namespace}joint_1">
+      <command_interface name="position" />
+      <command_interface name="velocity" />
+      <state_interface name="position">
+        <param name="initial_value">${initial_positions['joint_1']}</param>
+      </state_interface>
+      <state_interface name="velocity" />
+      <state_interface name="effort" />
+    </joint>
+    <joint name="${namespace}joint_2">
+      <command_interface name="position" />
+      <command_interface name="velocity" />
+      <state_interface name="position">
+        <param name="initial_value">${initial_positions['joint_2']}</param>
+      </state_interface>
+      <state_interface name="velocity" />
+      <state_interface name="effort" />
+    </joint>
+    <joint name="${namespace}joint_3">
+      <command_interface name="position" />
+      <command_interface name="velocity" />
+      <state_interface name="position">
+        <param name="initial_value">${initial_positions['joint_3']}</param>
+      </state_interface>
+      <state_interface name="velocity" />
+      <state_interface name="effort" />
+    </joint>
+    <joint name="${namespace}joint_4">
+      <command_interface name="position" />
+      <command_interface name="velocity" />
+      <state_interface name="position">
+        <param name="initial_value">${initial_positions['joint_4']}</param>
+      </state_interface>
+      <state_interface name="velocity" />
+      <state_interface name="effort" />
+    </joint>
+    <joint name="${namespace}joint_5">
+      <command_interface name="position" />
+      <command_interface name="velocity" />
+      <state_interface name="position">
+        <param name="initial_value">${initial_positions['joint_5']}</param>
+      </state_interface>
+      <state_interface name="velocity" />
+      <state_interface name="effort" />
+    </joint>
+    <joint name="${namespace}joint_6">
+      <command_interface name="position" />
+      <command_interface name="velocity" />
+      <state_interface name="position">
+        <param name="initial_value">${initial_positions['joint_6']}</param>
+      </state_interface>
+      <state_interface name="velocity" />
+      <state_interface name="effort" />
+    </joint>
+  </xacro:macro>
 </robot>
