Commit message: feat(vs060): add vs060 support and fix kinematics/inertial data
- denso_robot_bringup: add 'vs060' to the allowed model choices
- denso_robot.ros2_control.xacro: clean up macro parameter formatting,
  rename initial_positions to initial_positions_file, and load the
  YAML file directly inside denso_robot_joint_limits.xacro instead of
  passing pre-parsed data through the macro chain
- denso_robot_joint_limits.xacro: drop hardcoded position/velocity
  command_interface limits in favor of values loaded at runtime from
  the initial positions file
- denso_robot_kinematics.xacro: add correct inertial mass/origin/
  inertia values per link, convert joint limits to use radians(),
  raise effort limits to avoid gz-physics DART errors, and add
  flange/tool0 links and joints for end-effector attachment
- denso_robot_macro.xacro / denso_robot_transmissions.xacro: fix
  xacro namespace URL, rename basic_camera to gz_cam, point
  initial_positions_file default to denso_robot_moveit_config, and
  clean up whitespace/formatting
- joint_limits.yaml: correct max_velocity values (previously in rad/s
  scaled incorrectly, now matching actual joint velocity limits)
- denso_robot_macro.srdf.xacro: fix xacro namespace and XML
  declaration, replace explicit joint list with a base_link-to-tool0
  chain, add an end_effector group/definition, a home group state,
  and expand disable_collisions pairs for non-adjacent links

This change enables full support for the vs060 robot model across
description, control, and MoveIt configuration.

File: denso_robot_descriptions/robots/vs060/urdf/denso_robot_kinematics.xacro (robot description, xacro)
@@ -1,189 +1,257 @@
 <?xml version='1.0' encoding='UTF-8'?>
 <robot xmlns:xacro="http://www.ros.org/wiki/xacro">
-	<xacro:macro name="denso_robot_arm_kinematics" params="namespace model parent *origin">
-		<joint name="${namespace}joint_w" type="fixed">
-			<xacro:insert_block name="origin" />
-			<parent link="${parent}"/>
-			<child link="${namespace}base_link"/>
-		</joint>
-		<link name="${namespace}base_link">
-			<visual>
-				<origin rpy="0 0 0" xyz="0 0 0"/>
-				<geometry>
-					<mesh filename="file:///$(find denso_robot_descriptions)/robots/$(arg model)/meshes/base_link.dae" scale="1 1 1"/>
-				</geometry>
-			</visual>
-			<collision>
-				<origin rpy="0 0 0" xyz="0 0 0"/>
-				<geometry>
-					<mesh filename="file:///$(find denso_robot_descriptions)/robots/$(arg model)/meshes/base_link.dae" scale="1 1 1"/>
-				</geometry>
-			</collision>
-			<inertial>
-				<mass value="1"/>
-				<origin rpy="0.000000 0.000000 0.000000" xyz="0.000000 0.000000 0.000000"/>
-				<inertia ixx="1" ixy="0" ixz="0" iyy="1" iyz="0" izz="1"/>
-			</inertial>
-		</link>
-		<link name="${namespace}J1">
-			<visual>
-				<origin rpy="0 0 0" xyz="0 0 0"/>
-				<geometry>
-					<mesh filename="file:///$(find denso_robot_descriptions)/robots/$(arg model)/meshes/J1.dae" scale="1 1 1"/>
-				</geometry>
-			</visual>
-			<collision>
-				<origin rpy="0 0 0" xyz="0 0 0"/>
-				<geometry>
-					<mesh filename="file:///$(find denso_robot_descriptions)/robots/$(arg model)/meshes/J1.dae" scale="1 1 1"/>
-				</geometry>
-			</collision>
-			<inertial>
-				<mass value="1"/>
-				<origin rpy="0.000000 0.000000 0.000000" xyz="0.000000 0.000000 0.000000"/>
-				<inertia ixx="1" ixy="0" ixz="0" iyy="1" iyz="0" izz="1"/>
-			</inertial>
-		</link>
-		<joint name="${namespace}joint_1" type="revolute">
-			<parent link="${namespace}base_link"/>
-			<child link="${namespace}J1"/>
-			<origin rpy="0.000000 0.000000 0.000000" xyz="0.000000 0.000000 0.181500"/>
-			<axis xyz="-0.000000 -0.000000 1.000000"/>
-			<limit effort="1000" lower="-2.96705972839036" upper="2.96705972839036" velocity="3.73064127613788"/>   <!-- effort value is arbitary for make gazebo simulation runs without gravity problems -->
-			<dynamics damping="0" friction="0"/>
-		</joint>
-		<link name="${namespace}J2">
-			<visual>
-				<origin rpy="0 0 0" xyz="0 0 0"/>
-				<geometry>
-					<mesh filename="file:///$(find denso_robot_descriptions)/robots/$(arg model)/meshes/J2.dae" scale="1 1 1"/>
-				</geometry>
-			</visual>
-			<collision>
-				<origin rpy="0 0 0" xyz="0 0 0"/>
-				<geometry>
-					<mesh filename="file:///$(find denso_robot_descriptions)/robots/$(arg model)/meshes/J2.dae" scale="1 1 1"/>
-				</geometry>
-			</collision>
-			<inertial>
-				<mass value="1"/>
-				<origin rpy="0.000000 0.000000 0.000000" xyz="0.000000 0.000000 0.000000"/>
-				<inertia ixx="1" ixy="0" ixz="0" iyy="1" iyz="0" izz="1"/>
-			</inertial>
-		</link>
-		<joint name="${namespace}joint_2" type="revolute">
-			<parent link="${namespace}J1"/>
-			<child link="${namespace}J2"/>
-			<origin rpy="0.000000 0.000000 0.000000" xyz="0.000000 0.000000 0.163500"/>
-			<axis xyz="-0.000000 1.000000 -0.000000"/>
-			<limit effort="1000" lower="-2.0943951023932" upper="2.0943951023932" velocity="2.48709418409192"/> <!-- effort value is arbitary for make gazebo simulation runs without gravity problems -->
-		</joint>
-		<link name="${namespace}J3">
-			<visual>
-				<origin rpy="0 0 0" xyz="0 0 0"/>
-				<geometry>
-					<mesh filename="file:///$(find denso_robot_descriptions)/robots/$(arg model)/meshes/J3.dae" scale="1 1 1"/>
-				</geometry>
-			</visual>
-			<collision>
-				<origin rpy="0 0 0" xyz="0 0 0"/>
-				<geometry>
-					<mesh filename="file:///$(find denso_robot_descriptions)/robots/$(arg model)/meshes/J3.dae" scale="1 1 1"/>
-				</geometry>
-			</collision>
-			<inertial>
-				<mass value="1"/>
-				<origin rpy="0.000000 0.000000 0.000000" xyz="0.000000 0.000000 0.000000"/>
-				<inertia ixx="1" ixy="0" ixz="0" iyy="1" iyz="0" izz="1"/>
-			</inertial>
-		</link>
-		<joint name="${namespace}joint_3" type="revolute">
-			<parent link="${namespace}J2"/>
-			<child link="${namespace}J3"/>
-			<origin rpy="0.000000 0.000000 0.000000" xyz="0.000000 0.000000 0.305000"/>
-			<axis xyz="-0.000000 1.000000 -0.000000"/>
-			<limit effort="1000" lower="-2.18166156499291" upper="2.70526034059121" velocity="2.71540943019156"/> <!-- effort value is arbitary for make gazebo simulation runs without gravity problems -->
-			<dynamics damping="0" friction="0"/>
-		</joint>
-		<link name="${namespace}J4">
-			<visual>
-				<origin rpy="0 0 0" xyz="0 0 0"/>
-				<geometry>
-					<mesh filename="file:///$(find denso_robot_descriptions)/robots/$(arg model)/meshes/J4.dae" scale="1 1 1"/>
-				</geometry>
-			</visual>
-			<collision>
-				<origin rpy="0 0 0" xyz="0 0 0"/>
-				<geometry>
-					<mesh filename="file:///$(find denso_robot_descriptions)/robots/$(arg model)/meshes/J4.dae" scale="1 1 1"/>
-				</geometry>
-			</collision>
-			<inertial>
-				<mass value="1"/>
-				<origin rpy="0.000000 0.000000 0.000000" xyz="0.000000 0.000000 0.000000"/>
-				<inertia ixx="1" ixy="0" ixz="0" iyy="1" iyz="0" izz="1"/>
-			</inertial>
-		</link>
-		<joint name="${namespace}joint_4" type="revolute">
-			<parent link="${namespace}J3"/>
-			<child link="${namespace}J4"/>
-			<origin rpy="0.000000 0.000000 0.000000" xyz="-0.010000 0.000000 0.164500"/>
-			<axis xyz="-0.000000 -0.000000 1.000000"/>
-			<limit effort="1000" lower="-4.71238898038469" upper="4.71238898038469" velocity="3.73064127613788"/> <!-- effort value is arbitary for make gazebo simulation runs without gravity problems -->
-		</joint>
-		<link name="${namespace}J5">
-			<visual>
-				<origin rpy="0 0 0" xyz="0 0 0"/>
-				<geometry>
-					<mesh filename="file:///$(find denso_robot_descriptions)/robots/$(arg model)/meshes/J5.dae" scale="1 1 1"/>
-				</geometry>
-			</visual>
-			<collision>
-				<origin rpy="0 0 0" xyz="0 0 0"/>
-				<geometry>
-					<mesh filename="file:///$(find denso_robot_descriptions)/robots/$(arg model)/meshes/J5.dae" scale="1 1 1"/>
-				</geometry>
-			</collision>
-			<inertial>
-				<mass value="1"/>
-				<origin rpy="0.000000 0.000000 0.000000" xyz="0.000000 0.000000 0.000000"/>
-				<inertia ixx="1" ixy="0" ixz="0" iyy="1" iyz="0" izz="1"/>
-			</inertial>
-		</link>
-		<joint name="${namespace}joint_5" type="revolute">
-			<parent link="${namespace}J4"/>
-			<child link="${namespace}J5"/>
-			<origin rpy="0.000000 0.000000 0.000000" xyz="0.000000 0.000000 0.135500"/>
-			<axis xyz="-0.000000 1.000000 -0.000000"/>
-			<limit effort="1000" lower="-2.0943951023932" upper="2.0943951023932" velocity="2.87060410727889"/> <!-- effort value is arbitary for make gazebo simulation runs without gravity problems -->
-			<dynamics damping="0" friction="0"/>
-		</joint>
-		<link name="${namespace}J6">
-			<visual>
-				<origin rpy="0 0 0" xyz="0 0 0"/>
-				<geometry>
-					<mesh filename="file:///$(find denso_robot_descriptions)/robots/$(arg model)/meshes/J6.dae" scale="1 1 1"/>
-				</geometry>
-			</visual>
-			<collision>
-				<origin rpy="0 0 0" xyz="0 0 0"/>
-				<geometry>
-					<mesh filename="file:///$(find denso_robot_descriptions)/robots/$(arg model)/meshes/J6.dae" scale="1 1 1"/>
-				</geometry>
-			</collision>
-			<inertial>
-				<mass value="1"/>
-				<origin rpy="0.000000 0.000000 0.000000" xyz="0.000000 0.000000 0.000000"/>
-				<inertia ixx="1" ixy="0" ixz="0" iyy="1" iyz="0" izz="1"/>
-			</inertial>
-		</link>
-		<joint name="${namespace}joint_6" type="revolute">
-			<parent link="${namespace}J5"/>
-			<child link="${namespace}J6"/>
-			<origin rpy="0.000000 0.000000 0.000000" xyz="0.000000 0.000000 0.070000"/>
-			<axis xyz="-0.000000 -0.000000 1.000000"/>
-			<limit effort="1000" lower="-6.28318530717959" upper="6.28318530717959" velocity="5.96902604182061"/> <!-- effort value is arbitary for make gazebo simulation runs without gravity problems -->
-			<dynamics damping="0" friction="0"/>
-		</joint>
-	</xacro:macro>
+  <xacro:macro name="denso_robot_arm_kinematics" params="namespace model parent *origin">
+    <joint name="${namespace}joint_w" type="fixed">
+      <xacro:insert_block name="origin" />
+      <parent link="${parent}" />
+      <child link="${namespace}base_link" />
+    </joint>
+    <link name="${namespace}base_link">
+      <visual>
+        <origin rpy="0 0 0" xyz="0 0 0" />
+        <geometry>
+          <mesh
+            filename="file:///$(find denso_robot_descriptions)/robots/$(arg model)/meshes/base_link.dae"
+            scale="1 1 1" />
+        </geometry>
+      </visual>
+      <collision>
+        <origin rpy="0 0 0" xyz="0 0 0" />
+        <geometry>
+          <mesh
+            filename="file:///$(find denso_robot_descriptions)/robots/$(arg model)/meshes/base_link.dae"
+            scale="1 1 1" />
+        </geometry>
+      </collision>
+      <inertial>
+        <mass value="10.461" />
+        <origin rpy="0.000000 0.000000 0.000000" xyz="-0.03869715 -0.00013435 0.09015562" />
+        <inertia ixx="2.56287484e-05" ixy="0" ixz="0" iyy="4.04428633e-05" iyz="0"
+          izz="3.52691555e-05" />
+      </inertial>
+    </link>
+    <link name="${namespace}J1">
+      <visual>
+        <origin rpy="0 0 0" xyz="0 0 0" />
+        <geometry>
+          <mesh
+            filename="file:///$(find denso_robot_descriptions)/robots/$(arg model)/meshes/J1.dae"
+            scale="1 1 1" />
+        </geometry>
+      </visual>
+      <collision>
+        <origin rpy="0 0 0" xyz="0 0 0" />
+        <geometry>
+          <mesh
+            filename="file:///$(find denso_robot_descriptions)/robots/$(arg model)/meshes/J1.dae"
+            scale="1 1 1" />
+        </geometry>
+      </collision>
+      <inertial>
+        <mass value="4.857" />
+        <origin rpy="0.000000 0.000000 0.000000" xyz="0.00876456 -0.00129251 0.0831962" />
+        <inertia ixx="2.03436156e-05" ixy="0" ixz="0" iyy="1.43098790e-05" iyz="0"
+          izz="1.33404841e-05" />
+      </inertial>
+    </link>
+    <joint name="${namespace}joint_1" type="revolute">
+      <parent link="${namespace}base_link" />
+      <child link="${namespace}J1" />
+      <origin rpy="0.000000 0.000000 0.000000" xyz="0.000000 0.000000 0.181500" />
+      <axis xyz="-0.000000 -0.000000 1.000000" />
+      <!-- Initially, a negative effort value acting as a sentinel indicating "no limit" (treated as
+      infinity) was used,
+			but this was changed following the error on line 175 of
+			https://github.com/gazebosim/gz-physics/blob/ign-physics5/dartsim/src/JointFeatures.cc -->
+      <limit effort="1e6" lower="${radians(-170)}" upper="${radians(170)}"
+        velocity="${radians(425)}" />
+      <dynamics damping="0" friction="0" />
+    </joint>
+    <link name="${namespace}J2">
+      <visual>
+        <origin rpy="0 0 0" xyz="0 0 0" />
+        <geometry>
+          <mesh
+            filename="file:///$(find denso_robot_descriptions)/robots/$(arg model)/meshes/J2.dae"
+            scale="1 1 1" />
+        </geometry>
+      </visual>
+      <collision>
+        <origin rpy="0 0 0" xyz="0 0 0" />
+        <geometry>
+          <mesh
+            filename="file:///$(find denso_robot_descriptions)/robots/$(arg model)/meshes/J2.dae"
+            scale="1 1 1" />
+        </geometry>
+      </collision>
+      <inertial>
+        <mass value="6.830" />
+        <origin rpy="0.000000 0.000000 0.000000" xyz="-0.01430033 -0.00011275 0.10801241" />
+        <inertia ixx="5.11887760e-05" ixy="0" ixz="0" iyy="4.79804708e-05" iyz="0"
+          izz="1.07669409e-05" />
+      </inertial>
+    </link>
+    <joint name="${namespace}joint_2" type="revolute">
+      <parent link="${namespace}J1" />
+      <child link="${namespace}J2" />
+      <origin rpy="0.000000 0.000000 0.000000" xyz="0.000000 0.000000 0.163500" />
+      <axis xyz="-0.000000 1.000000 -0.000000" />
+      <!-- Initially, a negative effort value acting as a sentinel indicating "no limit" (treated as
+      infinity) was used,
+			but this was changed following the error on line 175 of
+			https://github.com/gazebosim/gz-physics/blob/ign-physics5/dartsim/src/JointFeatures.cc -->
+      <limit effort="1e6" lower="${radians(-120)}" upper="${radians(120)}"
+        velocity="${radians(283.33)}" />
+      <dynamics damping="0" friction="0" />
+    </joint>
+    <link name="${namespace}J3">
+      <visual>
+        <origin rpy="0 0 0" xyz="0 0 0" />
+        <geometry>
+          <mesh
+            filename="file:///$(find denso_robot_descriptions)/robots/$(arg model)/meshes/J3.dae"
+            scale="1 1 1" />
+        </geometry>
+      </visual>
+      <collision>
+        <origin rpy="0 0 0" xyz="0 0 0" />
+        <geometry>
+          <mesh
+            filename="file:///$(find denso_robot_descriptions)/robots/$(arg model)/meshes/J3.dae"
+            scale="1 1 1" />
+        </geometry>
+      </collision>
+      <inertial>
+        <mass value="3.352" />
+        <origin rpy="0.000000 0.000000 0.000000" xyz="-0.00423762 0.0017248 0.05850176" />
+        <inertia ixx="8.35358498e-06" ixy="0" ixz="0" iyy="8.39350395e-06" iyz="0"
+          izz="2.68861407e-06" />
+      </inertial>
+    </link>
+    <joint name="${namespace}joint_3" type="revolute">
+      <parent link="${namespace}J2" />
+      <child link="${namespace}J3" />
+      <origin rpy="0.000000 0.000000 0.000000" xyz="0.000000 0.000000 0.305000" />
+      <axis xyz="-0.000000 1.000000 -0.000000" />
+      <!-- Initially, a negative effort value acting as a sentinel indicating "no limit" (treated as
+      infinity) was used,
+			but this was changed following the error on line 175 of
+			https://github.com/gazebosim/gz-physics/blob/ign-physics5/dartsim/src/JointFeatures.cc -->
+      <limit effort="1e6" lower="${radians(-25)}" upper="${radians(155)}"
+        velocity="${radians(309.35)}" />
+      <dynamics damping="0" friction="0" />
+    </joint>
+    <link name="${namespace}J4">
+      <visual>
+        <origin rpy="0 0 0" xyz="0 0 0" />
+        <geometry>
+          <mesh
+            filename="file:///$(find denso_robot_descriptions)/robots/$(arg model)/meshes/J4.dae"
+            scale="1 1 1" />
+        </geometry>
+      </visual>
+      <collision>
+        <origin rpy="0 0 0" xyz="0 0 0" />
+        <geometry>
+          <mesh
+            filename="file:///$(find denso_robot_descriptions)/robots/$(arg model)/meshes/J4.dae"
+            scale="1 1 1" />
+        </geometry>
+      </collision>
+      <inertial>
+        <mass value="1.737" />
+        <origin rpy="0.000000 0.000000 0.000000" xyz="-0.00091641 0.00242194 0.06198817" />
+        <inertia ixx="2.99936270e-06" ixy="0" ixz="0" iyy="2.61340569e-06" iyz="0"
+          izz="1.50956216e-06" />
+      </inertial>
+    </link>
+    <joint name="${namespace}joint_4" type="revolute">
+      <parent link="${namespace}J3" />
+      <child link="${namespace}J4" />
+      <origin rpy="0.000000 0.000000 0.000000" xyz="-0.010000 0.000000 0.164500" />
+      <axis xyz="-0.000000 -0.000000 1.000000" />
+      <limit effort="6.66" lower="${radians(-270)}" upper="${radians(270)}"
+        velocity="${radians(425)}" />
+      <dynamics damping="0" friction="0" />
+    </joint>
+    <link name="${namespace}J5">
+      <visual>
+        <origin rpy="0 0 0" xyz="0 0 0" />
+        <geometry>
+          <mesh
+            filename="file:///$(find denso_robot_descriptions)/robots/$(arg model)/meshes/J5.dae"
+            scale="1 1 1" />
+        </geometry>
+      </visual>
+      <collision>
+        <origin rpy="0 0 0" xyz="0 0 0" />
+        <geometry>
+          <mesh
+            filename="file:///$(find denso_robot_descriptions)/robots/$(arg model)/meshes/J5.dae"
+            scale="1 1 1" />
+        </geometry>
+      </collision>
+      <inertial>
+        <mass value="0.721" />
+        <origin rpy="0.000000 0.000000 0.000000" xyz="0.00122859 -0.00178514 0.00591313" />
+        <inertia ixx="4.40135596e-07" ixy="0" ixz="0" iyy="5.27048557e-07" iyz="0"
+          izz="2.67901836e-07" />
+      </inertial>
+    </link>
+    <joint name="${namespace}joint_5" type="revolute">
+      <parent link="${namespace}J4" />
+      <child link="${namespace}J5" />
+      <origin rpy="0.000000 0.000000 0.000000" xyz="0.000000 0.000000 0.135500" />
+      <axis xyz="-0.000000 1.000000 -0.000000" />
+      <limit effort="6.66" lower="${radians(-120)}" upper="${radians(120)}"
+        velocity="${radians(327.01)}" />
+      <dynamics damping="0" friction="0" />
+    </joint>
+    <link name="${namespace}J6">
+      <visual>
+        <origin rpy="0 0 0" xyz="0 0 0" />
+        <geometry>
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