Commit message: feat(vs060): add vs060 support and fix kinematics/inertial data
- denso_robot_bringup: add 'vs060' to the allowed model choices
- denso_robot.ros2_control.xacro: clean up macro parameter formatting,
  rename initial_positions to initial_positions_file, and load the
  YAML file directly inside denso_robot_joint_limits.xacro instead of
  passing pre-parsed data through the macro chain
- denso_robot_joint_limits.xacro: drop hardcoded position/velocity
  command_interface limits in favor of values loaded at runtime from
  the initial positions file
- denso_robot_kinematics.xacro: add correct inertial mass/origin/
  inertia values per link, convert joint limits to use radians(),
  raise effort limits to avoid gz-physics DART errors, and add
  flange/tool0 links and joints for end-effector attachment
- denso_robot_macro.xacro / denso_robot_transmissions.xacro: fix
  xacro namespace URL, rename basic_camera to gz_cam, point
  initial_positions_file default to denso_robot_moveit_config, and
  clean up whitespace/formatting
- joint_limits.yaml: correct max_velocity values (previously in rad/s
  scaled incorrectly, now matching actual joint velocity limits)
- denso_robot_macro.srdf.xacro: fix xacro namespace and XML
  declaration, replace explicit joint list with a base_link-to-tool0
  chain, add an end_effector group/definition, a home group state,
  and expand disable_collisions pairs for non-adjacent links

This change enables full support for the vs060 robot model across
description, control, and MoveIt configuration.

File: denso_robot_descriptions/robots/vs060/urdf/denso_robot_macro.xacro (robot description, xacro)
@@ -1,4 +1,4 @@
 <?xml version="1.0"?>
-<robot xmlns:xacro="http://wiki.ros.org/xacro">
+<robot xmlns:xacro="http://www.ros.org/wiki/xacro">
   <!--
     Base Denso robot xacro macro.
@@ -9,53 +9,54 @@
     Author DENSO WAVE INCORPORATED
   -->
-  <xacro:macro name="denso_robot" params="
-    model
-    namespace
-    parent
-    *origin
-    transmission_hw_interface:=hardware_interface/PositionJointInterface
-    sim:=false
-    basic_camera:=false
-    ip_address
-    send_format
-    recv_format
-    verbose:=false"
-  >
+  <xacro:macro name="denso_robot" params="model
+                                          namespace
+                                          parent
+                                          *origin
+                                          transmission_hw_interface:=hardware_interface/PositionJointInterface
+                                          sim:=false
+                                          gz_cam:=false
+                                          ip_address
+                                          send_format
+                                          recv_format
+                                          verbose:=false">
     <!-- Robot data required by the denso driver -->
-    <xacro:arg name="ip_address" default="192.168.0.1"/>
-    <xacro:arg name="robot_name" default="VS060A3-AV6-NNN-NNN A"/> <!-- "robot_name" param must be consistent with the @TYPE_NAME variable of the real robot !! -->
-    <xacro:arg name="robot_joints" default="6"/> <!-- number of total joints in the kinematic chain -->
-    <xacro:arg name="joint_1" default="1"/> <!-- 0 = prismatic , 1 = revolute -->
-    <xacro:arg name="joint_2" default="1"/> <!-- 0 = prismatic , 1 = revolute -->
-    <xacro:arg name="joint_3" default="1"/> <!-- 0 = prismatic , 1 = revolute -->
-    <xacro:arg name="joint_4" default="1"/> <!-- 0 = prismatic , 1 = revolute -->
-    <xacro:arg name="joint_5" default="1"/> <!-- 0 = prismatic , 1 = revolute -->
-    <xacro:arg name="joint_6" default="1"/> <!-- 0 = prismatic , 1 = revolute -->
-    <xacro:arg name="controller_type" default="8"/> <!-- 8 = RC8 , 9 = RC9 -->
-    <xacro:arg name="arm_group" default="0"/>
-    <xacro:arg name="send_format" default="288"/>
-    <xacro:arg name="recv_format" default="292"/>
-    <xacro:arg name="verbose" default="false"/>
+    <xacro:arg name="ip_address" default="" />
+    <xacro:arg name="robot_name" default="VS060A3-AV6-NNN-NNN A" /> <!-- "robot_name" param must be
+    consistent with the @TYPE_NAME variable of the real robot !! -->
+    <xacro:arg name="robot_joints" default="6" /> <!-- number of total joints in the kinematic chain -->
+    <xacro:arg name="joint_1" default="1" /> <!-- 0 = prismatic , 1 = revolute -->
+    <xacro:arg name="joint_2" default="1" /> <!-- 0 = prismatic , 1 = revolute -->
+    <xacro:arg name="joint_3" default="1" /> <!-- 0 = prismatic , 1 = revolute -->
+    <xacro:arg name="joint_4" default="1" /> <!-- 0 = prismatic , 1 = revolute -->
+    <xacro:arg name="joint_5" default="1" /> <!-- 0 = prismatic , 1 = revolute -->
+    <xacro:arg name="joint_6" default="1" /> <!-- 0 = prismatic , 1 = revolute -->
+    <xacro:arg name="controller_type" default="8" /> <!-- 8 = RC8 , 9 = RC9 -->
+    <xacro:arg name="arm_group" default="0" />
+    <xacro:arg name="send_format" default="288" />
+    <xacro:arg name="recv_format" default="292" />
+    <xacro:arg name="verbose" default="false" />
     <!-- initial position for simulations-->
-    <xacro:arg name="initial_positions_file" default="$(find denso_robot_descriptions)/robots/$(arg model)/initial_positions.yaml"/>
-    <!-- convert to property to use substitution in function -->
-    <xacro:property name="initial_positions_file" default="$(arg initial_positions_file)"/>
-    <xacro:include filename="$(find denso_robot_descriptions)/robots/$(arg model)/urdf/denso_robot_transmissions.xacro" />
+    <xacro:arg name="initial_positions_file"
+      default="$(find denso_robot_moveit_config)/robots/$(arg model)/config/initial_positions.yaml" />
+    <xacro:include
+      filename="$(find denso_robot_descriptions)/robots/$(arg model)/urdf/denso_robot_transmissions.xacro" />
     <!-- robot kinematics include -->
-    <xacro:include filename="$(find denso_robot_descriptions)/robots/$(arg model)/urdf/denso_robot_kinematics.xacro" />
+    <xacro:include
+      filename="$(find denso_robot_descriptions)/robots/$(arg model)/urdf/denso_robot_kinematics.xacro" />
     <!-- ros2 control include -->
-    <xacro:include filename="$(find denso_robot_descriptions)/robots/$(arg model)/urdf/denso_robot.ros2_control.xacro" />
+    <xacro:include
+      filename="$(find denso_robot_descriptions)/robots/$(arg model)/urdf/denso_robot.ros2_control.xacro" />
     <!-- For other tools, modify the filename parameter to the path of your tool's xacro file. -->
     <!-- The line with tag xacro:tool passes the parameters defined in your tool's xacro file -->
-    <!-- (see basic_camera.xacro as an example implementation) -->
-    <xacro:if value="$(arg basic_camera)">
-      <xacro:include filename="$(find denso_robot_gazebo)/sensors/basic_camera/urdf/basic_camera.xacro" />
+    <!-- (see gz_cam.xacro as an example implementation) -->
+    <xacro:if value="$(arg gz_cam)">
+      <xacro:include filename="$(find denso_robot_gazebo)/sensors/gz_cam/urdf/gz_cam.xacro" />
     </xacro:if>
     <!-- ros2 control instance -->
-    <xacro:denso_robot_ros2_control
-      name="GazeboSystem" namespace="${namespace}"
+    <xacro:denso_robot_ros2_control name="VS060"
+      namespace="${namespace}"
       sim="$(arg sim)"
       model="$(arg model)"
-      ip_address="$(arg ip_address)"
+      ip_address="${ip_address}"
       robot_name="$(arg robot_name)"
       robot_joints="$(arg robot_joints)"
@@ -71,14 +72,16 @@
       send_format="$(arg send_format)"
       recv_format="$(arg recv_format)"
-      initial_positions="${xacro.load_yaml(initial_positions_file)}" />
+      initial_positions_file="$(arg initial_positions_file)" />
     <!-- Add URDF transmission elements (for ros_control) -->
-    <xacro:denso_robot_arm_transmission namespace="${namespace}" hw_interface="$(arg transmission_hw_interface)" />
+    <xacro:denso_robot_arm_transmission namespace="${namespace}"
+      hw_interface="$(arg transmission_hw_interface)" />
     <!-- Placeholder for ros2_control transmission which don't yet exist -->
     <!-- links -  main serial chain -->
-    <xacro:denso_robot_arm_kinematics namespace="${namespace}" model="$(arg model)" parent="${parent}" >
+    <xacro:denso_robot_arm_kinematics namespace="${namespace}" model="$(arg model)"
+      parent="${parent}">
       <xacro:insert_block name="origin" />
     </xacro:denso_robot_arm_kinematics>
-    <xacro:if value="$(arg basic_camera)">
-      <xacro:basic_camera namespace="${namespace}" end_effector="J6" />
+    <xacro:if value="$(arg gz_cam)">
+      <xacro:gz_cam namespace="${namespace}" />
     </xacro:if>
   </xacro:macro>

File: denso_robot_moveit_config/robots/vs060/srdf/denso_robot_macro.srdf.xacro (robot description, xacro)
@@ -1,4 +1,4 @@
-<?xml version="1.0" encoding="UTF-8"?>
-<robot xmlns:xacro="http://wiki.ros.org/xacro">
+<?xml version="1.0"?>
+<robot xmlns:xacro="http://www.ros.org/wiki/xacro">
 <!--This does not replace URDF, and is not an extension of URDF.
     This is a format for representing semantic information about the robot structure.
@@ -12,24 +12,37 @@
     <!--SUBGROUPS - Groups can also be formed by referencing to already defined group names-->
     <group name="${namespace}arm">
-		<joint name="${namespace}joint_1"/>
-		<joint name="${namespace}joint_2"/>
-		<joint name="${namespace}joint_3"/>
-		<joint name="${namespace}joint_4"/>
-		<joint name="${namespace}joint_5"/>
-		<joint name="${namespace}joint_6"/>
-	</group>
+      <chain base_link="${namespace}base_link" tip_link="${namespace}tool0" />
+    </group>
+    <group name="${namespace}end_effector">
+        <link name="${namespace}tool0"/>
+    </group>
     <!--GROUP STATES - Purpose - Define a named state for a particular group, in terms of joint values. This is useful to define states like 'folded arms'-->
+    <group_state name="${namespace}home" group="${namespace}arm">
+      <joint name="${namespace}joint_1" value="0"/>
+      <joint name="${namespace}joint_2" value="-0.5"/>
+      <joint name="${namespace}joint_3" value="1.2"/>
+      <joint name="${namespace}joint_4" value="0"/>
+      <joint name="${namespace}joint_5" value="1.5"/>
+      <joint name="${namespace}joint_6" value="0"/>
+    </group_state>
     <!--END EFFECTOR - Purpose - Represent information about an end effector.-->
+    <end_effector name="${namespace}eff" parent_link="${namespace}tool0" group="${namespace}end_effector" parent_group="${namespace}arm"/>
     <!--VIRTUAL JOINT - Purpose - this element defines a virtual joint between a robot link and an external frame of reference (considered fixed with respect to the robot)-->
     <virtual_joint name="${namespace}fixed_base" type="fixed" parent_frame="world" child_link="${namespace}base_link" />
     <!--DISABLE COLLISIONS - By default it is assumed that any link of the robot could potentially come into collision with any other link in the robot. This tag disables collision checking between a specified pair of links. -->
-	<disable_collisions link1="${namespace}J6" link2="${namespace}J3" reason="Never"/>
-	<disable_collisions link1="${namespace}J6" link2="${namespace}J5" reason="Adjacent"/>
-	<disable_collisions link1="${namespace}J1" link2="${namespace}J2" reason="Adjacent"/>
-	<disable_collisions link1="${namespace}J1" link2="${namespace}base_link" reason="Adjacent"/>
-	<disable_collisions link1="${namespace}J2" link2="${namespace}J3" reason="Adjacent"/>
-	<disable_collisions link1="${namespace}J3" link2="${namespace}J4" reason="Adjacent"/>
-	<disable_collisions link1="${namespace}J3" link2="${namespace}J5" reason="Never"/>
-	<disable_collisions link1="${namespace}J4" link2="${namespace}J5" reason="Adjacent"/>
+	  <disable_collisions link1="${namespace}J1" link2="${namespace}J2" reason="Adjacent"/>
+	  <disable_collisions link1="${namespace}J1" link2="${namespace}J3" reason="Never"/>
+    <disable_collisions link1="${namespace}J1" link2="${namespace}base_link" reason="Adjacent"/>
+    <disable_collisions link1="${namespace}J2" link2="${namespace}J3" reason="Adjacent"/>
+    <disable_collisions link1="${namespace}J2" link2="${namespace}J4" reason="Never"/>
+    <disable_collisions link1="${namespace}J2" link2="${namespace}J5" reason="Never"/>
+    <disable_collisions link1="${namespace}J2" link2="${namespace}J6" reason="Never"/>
+    <disable_collisions link1="${namespace}J2" link2="${namespace}base_link" reason="Never"/>
+    <disable_collisions link1="${namespace}J3" link2="${namespace}J4" reason="Adjacent"/>
+    <disable_collisions link1="${namespace}J3" link2="${namespace}J5" reason="Never"/>
+    <disable_collisions link1="${namespace}J3" link2="${namespace}J6" reason="Never"/>
+    <disable_collisions link1="${namespace}J4" link2="${namespace}J5" reason="Adjacent"/>
+    <disable_collisions link1="${namespace}J4" link2="${namespace}J6" reason="Never"/>
+    <disable_collisions link1="${namespace}J5" link2="${namespace}J6" reason="Adjacent"/>
   </xacro:macro>
 </robot>
