Commit message: feat(bringup): parameterize robot base origin pose (xyz, rpy)
Exposes 'xyz' and 'rpy' arguments in both single and dual robot launch files, passing them directly to the URDF xacro. This allows defining the robot's base position and orientation relative to the world frame at runtime, replacing previously hardcoded origin values.

File: denso_robot_descriptions/urdf/denso_robot.urdf.xacro (robot description, xacro)
@@ -15,4 +15,6 @@
    <xacro:arg name="send_format" default="288" />
    <xacro:arg name="recv_format" default="292" />
+   <xacro:arg name="xyz" default="0 0 0" />
+   <xacro:arg name="rpy" default="0 0 0" />
    <!-- Root link -->
    <link name="world"/>
@@ -29,5 +31,5 @@
      send_format="$(arg send_format)"
      recv_format="$(arg recv_format)" >
-     <origin xyz="0 0 0" rpy="0 0 0" />
+     <origin xyz="$(arg xyz)" rpy="$(arg rpy)" />
    </xacro:denso_robot>
    <gazebo>

File: denso_robot_descriptions/urdf/dual_denso_robot.urdf.xacro (robot description, xacro)
@@ -15,4 +15,8 @@
    <xacro:arg name="send_format" default="288" />
    <xacro:arg name="recv_format" default="292" />
+   <xacro:arg name="left_xyz" default="0 0.42 0" />
+   <xacro:arg name="left_rpy" default="0 0 ${-pi/2}" />
+   <xacro:arg name="right_xyz" default="0 -0.42 0" />
+   <xacro:arg name="right_rpy" default="0 0 ${pi/2}" />
    <!-- Root link -->
    <link name="world"/>
@@ -29,5 +33,5 @@
      send_format="$(arg send_format)"
      recv_format="$(arg recv_format)" >
-     <origin xyz="0 0.42 0" rpy="0 0 ${-pi/2}" />
+     <origin xyz="$(arg left_xyz)" rpy="$(arg left_rpy)" />
    </xacro:denso_robot>
    <!-- right arm -->
@@ -43,5 +47,5 @@
      send_format="$(arg send_format)"
      recv_format="$(arg recv_format)" >
-     <origin xyz="0 -0.42 0" rpy="0 0 ${pi/2}" />
+     <origin xyz="$(arg right_xyz)" rpy="$(arg right_rpy)" />
    </xacro:denso_robot>
    <gazebo>
