Commit message: feat: add dual-arm robot support in vs050 xacro/urdf description

File: denso_robot_descriptions/robots/vs050/urdf/denso_robot.ros2_control.xacro (robot description, xacro)
@@ -40,5 +40,5 @@
         </xacro:unless>
       </hardware>
-      <xacro:denso_robot_control_limits namespace="$(arg namespace)" />
+      <xacro:denso_robot_control_limits namespace="${namespace}" />
     </ros2_control>
   </xacro:macro>

File: denso_robot_descriptions/robots/vs050/urdf/denso_robot_joint_limits.xacro (robot description, xacro)
@@ -2,5 +2,5 @@
 <robot xmlns:xacro="http://www.ros.org/wiki/xacro">
 	<xacro:macro name="denso_robot_control_limits" params="namespace">
-		<joint name="$(arg namespace)joint_1">
+		<joint name="${namespace}joint_1">
 			<command_interface name="position">
 				<param name="min">-2.967060</param>
@@ -15,5 +15,5 @@
 			<state_interface name="effort"/>
 		</joint>
-		<joint name="$(arg namespace)joint_2">
+		<joint name="${namespace}joint_2">
 			<command_interface name="position">
 				<param name="min">-2.094395</param>
@@ -28,5 +28,5 @@
 			<state_interface name="effort"/>
 		</joint>
-		<joint name="$(arg namespace)joint_3">
+		<joint name="${namespace}joint_3">
 			<command_interface name="position">
 				<param name="min">${radians(-120)}</param>
@@ -41,5 +41,5 @@
 			<state_interface name="effort"/>
 		</joint>
-		<joint name="$(arg namespace)joint_4">
+		<joint name="${namespace}joint_4">
 			<command_interface name="position">
 				<param name="min">-4.712389</param>
@@ -54,5 +54,5 @@
 			<state_interface name="effort"/>
 		</joint>
-		<joint name="$(arg namespace)joint_5">
+		<joint name="${namespace}joint_5">
 			<command_interface name="position">
 				<param name="min">-2.094395</param>
@@ -67,5 +67,5 @@
 			<state_interface name="effort"/>
 		</joint>
-		<joint name="$(arg namespace)joint_6">
+		<joint name="${namespace}joint_6">
 			<command_interface name="position">
 				<param name="min">-6.283185</param>

File: denso_robot_descriptions/robots/vs050/urdf/denso_robot_kinematics.xacro (robot description, xacro)
@@ -1,11 +1,11 @@
 <?xml version='1.0' encoding='UTF-8'?>
 <robot xmlns:xacro="http://www.ros.org/wiki/xacro">
-	<xacro:macro name="denso_robot_arm_kinematics" params="namespace model">
-		<link name="world"/>
-		<joint name="$(arg namespace)joint_w" type="fixed">
-			<parent link="world"/>
-			<child link="$(arg namespace)base_link"/>
+	<xacro:macro name="denso_robot_arm_kinematics" params="namespace model parent *origin">
+		<joint name="${namespace}joint_w" type="fixed">
+			<xacro:insert_block name="origin" />
+			<parent link="${parent}"/>
+			<child link="${namespace}base_link"/>
 		</joint>
-		<link name="$(arg namespace)base_link">
+		<link name="${namespace}base_link">
 			<visual>
 				<origin rpy="0 0 0" xyz="0 0 0"/>
@@ -26,5 +26,5 @@
 			</inertial>
 		</link>
-		<link name="$(arg namespace)J1">
+		<link name="${namespace}J1">
 			<visual>
 				<origin rpy="0 0 0" xyz="0 0 0"/>
@@ -45,7 +45,7 @@
 			</inertial>
 		</link>
-		<joint name="$(arg namespace)joint_1" type="revolute">
-			<parent link="$(arg namespace)base_link"/>
-			<child link="$(arg namespace)J1"/>
+		<joint name="${namespace}joint_1" type="revolute">
+			<parent link="${namespace}base_link"/>
+			<child link="${namespace}J1"/>
 			<origin rpy="0.000000 0.000000 0.000000" xyz="0.000000 0.000000 0.181500"/>
 			<axis xyz="-0.000000 -0.000000 1.000000"/>
@@ -53,5 +53,5 @@
 			<dynamics damping="0" friction="0"/>
 		</joint>
-		<link name="$(arg namespace)J2">
+		<link name="${namespace}J2">
 			<visual>
 				<origin rpy="0 0 0" xyz="0 0 0"/>
@@ -72,7 +72,7 @@
 			</inertial>
 		</link>
-		<joint name="$(arg namespace)joint_2" type="revolute">
-			<parent link="$(arg namespace)J1"/>
-			<child link="$(arg namespace)J2"/>
+		<joint name="${namespace}joint_2" type="revolute">
+			<parent link="${namespace}J1"/>
+			<child link="${namespace}J2"/>
 			<origin rpy="0.000000 0.000000 0.000000" xyz="0.000000 0.000000 0.163500"/>
 			<axis xyz="-0.000000 1.000000 -0.000000"/>
@@ -80,5 +80,5 @@
 			<dynamics damping="0" friction="0"/>
 		</joint>
-		<link name="$(arg namespace)J3">
+		<link name="${namespace}J3">
 			<visual>
 				<origin rpy="0 0 0" xyz="0 0 0"/>
@@ -99,7 +99,7 @@
 			</inertial>
 		</link>
-		<joint name="$(arg namespace)joint_3" type="revolute">
-			<parent link="$(arg namespace)J2"/>
-			<child link="$(arg namespace)J3"/>
+		<joint name="${namespace}joint_3" type="revolute">
+			<parent link="${namespace}J2"/>
+			<child link="${namespace}J3"/>
 			<origin rpy="0.000000 0.000000 0.000000" xyz="0.000000 0.000000 0.250000"/>
 			<axis xyz="-0.000000 1.000000 -0.000000"/>
@@ -107,5 +107,5 @@
 			<dynamics damping="0" friction="0"/>
 		</joint>
-		<link name="$(arg namespace)J4">
+		<link name="${namespace}J4">
 			<visual>
 				<origin rpy="0 0 0" xyz="0 0 0"/>
@@ -126,7 +126,7 @@
 			</inertial>
 		</link>
-		<joint name="$(arg namespace)joint_4" type="revolute">
-			<parent link="$(arg namespace)J3"/>
-			<child link="$(arg namespace)J4"/>
+		<joint name="${namespace}joint_4" type="revolute">
+			<parent link="${namespace}J3"/>
+			<child link="${namespace}J4"/>
 			<origin rpy="0.000000 0.000000 0.000000" xyz="-0.010000 0.000000 0.119500"/>
 			<axis xyz="-0.000000 -0.000000 1.000000"/>
@@ -134,5 +134,5 @@
 			<dynamics damping="0" friction="0"/>
 		</joint>
-		<link name="$(arg namespace)J5">
+		<link name="${namespace}J5">
 			<visual>
 				<origin rpy="0 0 0" xyz="0 0 0"/>
@@ -153,7 +153,7 @@
 			</inertial>
 		</link>
-		<joint name="$(arg namespace)joint_5" type="revolute">
-			<parent link="$(arg namespace)J4"/>
-			<child link="$(arg namespace)J5"/>
+		<joint name="${namespace}joint_5" type="revolute">
+			<parent link="${namespace}J4"/>
+			<child link="${namespace}J5"/>
 			<origin rpy="0.000000 0.000000 0.000000" xyz="0.000000 0.000000 0.135500"/>
 			<axis xyz="-0.000000 1.000000 -0.000000"/>
@@ -161,5 +161,5 @@
 			<dynamics damping="0" friction="0"/>
 		</joint>
-		<link name="$(arg namespace)J6">
+		<link name="${namespace}J6">
 			<visual>
 				<origin rpy="0 0 0" xyz="0 0 0"/>
@@ -180,7 +180,7 @@
 			</inertial>
 		</link>
-		<joint name="$(arg namespace)joint_6" type="revolute">
-			<parent link="$(arg namespace)J5"/>
-			<child link="$(arg namespace)J6"/>
+		<joint name="${namespace}joint_6" type="revolute">
+			<parent link="${namespace}J5"/>
+			<child link="${namespace}J6"/>
 			<origin rpy="0.000000 0.000000 0.000000" xyz="0.000000 0.000000 0.070000"/>
 			<axis xyz="-0.000000 -0.000000 1.000000"/>

File: denso_robot_descriptions/robots/vs050/urdf/denso_robot_macro.xacro (robot description, xacro)
@@ -12,4 +12,6 @@
     model
     namespace
+    parent
+    *origin
     transmission_hw_interface:=hardware_interface/PositionJointInterface
     sim:=false
@@ -48,5 +50,5 @@
     <!-- ros2 control instance -->
     <xacro:denso_robot_ros2_control
-      name="GazeboSystem" namespace="$(arg namespace)"
+      name="GazeboSystem" namespace="${namespace}"
       sim="$(arg sim)"
       model="$(arg model)"
@@ -66,10 +68,12 @@
       recv_format="$(arg recv_format)" />
     <!-- Add URDF transmission elements (for ros_control) -->
-    <xacro:denso_robot_arm_transmission namespace="$(arg namespace)" hw_interface="$(arg transmission_hw_interface)" />
+    <xacro:denso_robot_arm_transmission namespace="${namespace}" hw_interface="$(arg transmission_hw_interface)" />
     <!-- Placeholder for ros2_control transmission which don't yet exist -->
     <!-- links -  main serial chain -->
-    <xacro:denso_robot_arm_kinematics namespace="$(arg namespace)" model="$(arg model)" />
+    <xacro:denso_robot_arm_kinematics namespace="${namespace}" model="$(arg model)" parent="${parent}" >
+      <xacro:insert_block name="origin" />
+    </xacro:denso_robot_arm_kinematics>
     <xacro:if value="$(arg basic_camera)">
-      <xacro:tool namespace="$(arg namespace)" />
+      <xacro:tool namespace="${namespace}" />
     </xacro:if>
     <gazebo>

File: denso_robot_descriptions/tools/basic_camera/urdf/basic_camera.xacro (robot description, xacro)
@@ -5,5 +5,5 @@
     <!-- if your tool has meshes, define the path to it in geometry tag. -->
     <!-- see the vs050 robot urdf implementation as an example. -->
-    <link name="$(arg namespace)basic_camera_link">
+    <link name="${namespace}basic_camera_link">
 		<inertial>
 			<mass value="1"/>
@@ -21,11 +21,11 @@
 		</visual>
 	</link>
-	<joint name="$(arg namespace)basic_camera_joint" type="fixed">
+	<joint name="${namespace}basic_camera_joint" type="fixed">
         <!-- here you define where your tool will connect. In this case, it's at joint 6. -->
-		<parent link="$(arg namespace)J6"/>
-		<child link="$(arg namespace)basic_camera_link"/>
+		<parent link="${namespace}J6"/>
+		<child link="${namespace}basic_camera_link"/>
 		<origin rpy="0 ${radians(-90)} 0" xyz="0 0 0.01"/>
 	</joint>
-    <gazebo reference="$(arg namespace)basic_camera_link">
+    <gazebo reference="${namespace}basic_camera_link">
       <sensor name="basic_camera" type="camera">
         <camera>

File: denso_robot_descriptions/urdf/dual_denso_robot.urdf.xacro (robot description, xacro)
@@ -6,5 +6,4 @@
    <xacro:include filename="$(find denso_robot_descriptions)/robots/$(arg model)/urdf/denso_robot_macro.xacro"/>
    <!-- parameters -->
-   <xacro:arg name="namespace" default="" />
    <xacro:arg name="transmission_hw_interface" default=""/>
    <!-- ros2_control related parameters -->
@@ -17,8 +16,8 @@
    <!-- Root link -->
    <link name="world"/>
-   <!-- arm -->
+   <!-- left arm -->
    <xacro:denso_robot
      model="$(arg model)"
-     namespace="$(arg namespace)"
+     namespace="left_"
      parent="world"
      transmission_hw_interface="$(arg transmission_hw_interface)"
@@ -29,5 +28,19 @@
      send_format="$(arg send_format)"
      recv_format="$(arg recv_format)" >
-     <origin xyz="0 0 0" rpy="0 0 0" />
+     <origin xyz="0 0.42 0" rpy="0 0 ${-pi/2}" />
+   </xacro:denso_robot>
+   <!-- right arm -->
+   <xacro:denso_robot
+     model="$(arg model)"
+     namespace="right_"
+     parent="world"
+     transmission_hw_interface="$(arg transmission_hw_interface)"
+     sim="$(arg sim)"
+     basic_camera="$(arg basic_camera)"
+     ip_address="$(arg ip_address)"
+     verbose="$(arg verbose)"
+     send_format="$(arg send_format)"
+     recv_format="$(arg recv_format)" >
+     <origin xyz="0 -0.42 0" rpy="0 0 ${pi/2}" />
    </xacro:denso_robot>
 </robot>

Commit message: feat(urdf): add support for initial joint positions in ros2_control
Introduces the ability to set initial joint positions for simulation
via a YAML configuration file.

Changes:
- Adds `initial_positions_file` argument to the main robot macro to
  load a YAML dictionary.
- Passes the `initial_positions` map down to the ros2_control xacro.
- Updates joint limits xacro to inject `initial_value` parameters into
  the position state interfaces.

This allows the robot to spawn in a specific configuration in
simulations (e.g., Mock Hardware), facilitating MoveIt 2 integration.

File: denso_robot_descriptions/robots/vs050/urdf/denso_robot.ros2_control.xacro (robot description, xacro)
@@ -11,4 +11,5 @@
 	controller_type
     verbose
+    initial_positions
     ">
     <ros2_control name="${namespace}${name}" type="system">
@@ -40,5 +41,5 @@
         </xacro:unless>
       </hardware>
-      <xacro:denso_robot_control_limits namespace="${namespace}" />
+      <xacro:denso_robot_control_limits namespace="${namespace}" initial_positions="${initial_positions}" />
     </ros2_control>
   </xacro:macro>

File: denso_robot_descriptions/robots/vs050/urdf/denso_robot_joint_limits.xacro (robot description, xacro)
@@ -1,5 +1,5 @@
 <?xml version='1.0' encoding='UTF-8'?>
 <robot xmlns:xacro="http://www.ros.org/wiki/xacro">
-	<xacro:macro name="denso_robot_control_limits" params="namespace">
+	<xacro:macro name="denso_robot_control_limits" params="namespace initial_positions">
 		<joint name="${namespace}joint_1">
 			<command_interface name="position">
@@ -11,5 +11,7 @@
 				<param name="max">0.392699081698724</param>
 			</command_interface>
-			<state_interface name="position"/>
+			<state_interface name="position">
+				<param name="initial_value">${initial_positions['joint_1']}</param>
+			</state_interface>
 			<state_interface name="velocity"/>
 			<state_interface name="effort"/>
@@ -24,5 +26,7 @@
 				<param name="max">0.261799387799149</param>
 			</command_interface>
-			<state_interface name="position"/>
+			<state_interface name="position">
+				<param name="initial_value">${initial_positions['joint_2']}</param>
+			</state_interface>
 			<state_interface name="velocity"/>
 			<state_interface name="effort"/>
@@ -37,5 +41,7 @@
 				<param name="max">0.285832571599111</param>
 			</command_interface>
-			<state_interface name="position"/>
+			<state_interface name="position">
+				<param name="initial_value">${initial_positions['joint_3']}</param>
+			</state_interface>
 			<state_interface name="velocity"/>
 			<state_interface name="effort"/>
@@ -50,5 +56,7 @@
 				<param name="max">0.392699081698724</param>
 			</command_interface>
-			<state_interface name="position"/>
+			<state_interface name="position">
+				<param name="initial_value">${initial_positions['joint_4']}</param>
+			</state_interface>
 			<state_interface name="velocity"/>
 			<state_interface name="effort"/>
@@ -63,5 +71,7 @@
 				<param name="max">0.302168853397778</param>
 			</command_interface>
-			<state_interface name="position"/>
+			<state_interface name="position">
+				<param name="initial_value">${initial_positions['joint_5']}</param>
+			</state_interface>
 			<state_interface name="velocity"/>
 			<state_interface name="effort"/>
@@ -76,5 +86,7 @@
 				<param name="max">0.628318530717959</param>
 			</command_interface>
-			<state_interface name="position"/>
+			<state_interface name="position">
+				<param name="initial_value">${initial_positions['joint_6']}</param>
+			</state_interface>
 			<state_interface name="velocity"/>
 			<state_interface name="effort"/>

File: denso_robot_descriptions/robots/vs050/urdf/denso_robot_macro.xacro (robot description, xacro)
@@ -37,4 +37,8 @@
     <xacro:arg name="recv_format" default="292"/>
     <xacro:arg name="verbose" default="false"/>
+    <!-- initial position for simulations-->
+    <xacro:arg name="initial_positions_file" default="$(find denso_robot_descriptions)/robots/$(arg model)/initial_positions.yaml"/>
+    <!-- convert to property to use substitution in function -->
+    <xacro:property name="initial_positions_file" default="$(arg initial_positions_file)"/>
     <xacro:include filename="$(find denso_robot_descriptions)/robots/$(arg model)/urdf/denso_robot_transmissions.xacro" />
     <!-- robot kinematics include -->
@@ -66,5 +70,6 @@
       verbose="$(arg verbose)"
       send_format="$(arg send_format)"
-      recv_format="$(arg recv_format)" />
+      recv_format="$(arg recv_format)"
+      initial_positions="${xacro.load_yaml(initial_positions_file)}" />
     <!-- Add URDF transmission elements (for ros_control) -->
     <xacro:denso_robot_arm_transmission namespace="${namespace}" hw_interface="$(arg transmission_hw_interface)" />
