Commit message: style(urdf): format xacro files and fix xml namespaces
- Improve readability by vertically aligning macro parameters, fixing indentation, and standardizing blank lines across the vs050 URDF files.
- Correct the `xmlns:xacro` URLs from `http://wiki.ros.org/xacro` to `http://www.ros.org/wiki/xacro`.
- Update the `ros2_control` system name from "GazeboSystem" to "VS050" in the main robot macro.

File: denso_robot_descriptions/robots/vs050/urdf/denso_robot.ros2_control.xacro (robot description, xacro)
@@ -1,19 +1,28 @@
 <?xml version="1.0"?>
 <robot xmlns:xacro="http://www.ros.org/wiki/xacro">
-  <xacro:macro name="denso_robot_ros2_control" params="name namespace
-	robot_name
-    sim:=false fake_sensor_commands:=false
-    ip_address
-    model
-    robot_joints joint_1 joint_2 joint_3 joint_4 joint_5 joint_6
-    arm_group
-    send_format recv_format
-	controller_type
-    verbose
-    initial_positions
-    ">
+  <xacro:macro name="denso_robot_ros2_control"
+               params="name
+                       namespace
+                       robot_name
+                       sim:=false
+                       fake_sensor_commands:=false
+                       ip_address
+                       model
+                       robot_joints
+                       joint_1
+                       joint_2
+                       joint_3
+                       joint_4
+                       joint_5
+                       joint_6
+                       arm_group
+                       send_format
+                       recv_format
+                       controller_type
+                       verbose
+                       initial_positions">
     <ros2_control name="${namespace}${name}" type="system">
-	<!-- joint limits include -->
-	<xacro:include filename="$(find denso_robot_descriptions)/robots/$(arg model)/urdf/denso_robot_joint_limits.xacro" />
+	  <!-- joint limits include -->
+	  <xacro:include filename="$(find denso_robot_descriptions)/robots/$(arg model)/urdf/denso_robot_joint_limits.xacro" />
       <hardware>
         <xacro:if value="${sim}">
@@ -23,5 +32,5 @@
           <plugin>denso_robot_control/DensoRobotHW</plugin>
           <param name="ip_address">${ip_address}</param>
-<!-- "robot_name" param must be consistent with the @TYPE_NAME variable of the real robot !!  -->
+          <!-- "robot_name" param must be consistent with the @TYPE_NAME variable of the real robot !!  -->
           <param name="robot_name">${robot_name}</param>
           <param name="node_name">denso_robot_control</param>

File: denso_robot_descriptions/robots/vs050/urdf/denso_robot_macro.xacro (robot description, xacro)
@@ -1,4 +1,4 @@
 <?xml version="1.0"?>
-<robot xmlns:xacro="http://wiki.ros.org/xacro">
+<robot xmlns:xacro="http://www.ros.org/wiki/xacro">
   <!--
     Base Denso robot xacro macro.
@@ -9,77 +9,75 @@
     Author DENSO WAVE INCORPORATED
   -->
-  <xacro:macro name="denso_robot" params="
-    model
-    namespace
-    parent
-    *origin
-    transmission_hw_interface:=hardware_interface/PositionJointInterface
-    sim:=false
-    basic_camera:=false
-    ip_address
-    send_format
-    recv_format
-    verbose:=false"
-  >
-    <!-- Robot data required by the denso driver -->
-    <xacro:arg name="ip_address" default=""/>
-    <xacro:arg name="robot_name" default="VS050A3-AV6-NNN-NNN A"/> <!-- "robot_name" param must be consistent with the @TYPE_NAME variable of the real robot !! -->
-    <xacro:arg name="robot_joints" default="6"/> <!-- number of total joints in the kinematic chain -->
-    <xacro:arg name="joint_1" default="1"/> <!-- 0 = prismatic , 1 = revolute -->
-    <xacro:arg name="joint_2" default="1"/> <!-- 0 = prismatic , 1 = revolute -->
-    <xacro:arg name="joint_3" default="1"/> <!-- 0 = prismatic , 1 = revolute -->
-    <xacro:arg name="joint_4" default="1"/> <!-- 0 = prismatic , 1 = revolute -->
-    <xacro:arg name="joint_5" default="1"/> <!-- 0 = prismatic , 1 = revolute -->
-    <xacro:arg name="joint_6" default="1"/> <!-- 0 = prismatic , 1 = revolute -->
-    <xacro:arg name="controller_type" default="8"/> <!-- 8 = RC8 , 9 = RC9 -->
-    <xacro:arg name="arm_group" default="0"/>
-    <xacro:arg name="send_format" default="288"/>
-    <xacro:arg name="recv_format" default="292"/>
-    <xacro:arg name="verbose" default="false"/>
-    <!-- initial position for simulations-->
-    <xacro:arg name="initial_positions_file" default="$(find denso_robot_descriptions)/robots/$(arg model)/initial_positions.yaml"/>
-    <!-- convert to property to use substitution in function -->
-    <xacro:property name="initial_positions_file" default="$(arg initial_positions_file)"/>
-    <xacro:include filename="$(find denso_robot_descriptions)/robots/$(arg model)/urdf/denso_robot_transmissions.xacro" />
-    <!-- robot kinematics include -->
-    <xacro:include filename="$(find denso_robot_descriptions)/robots/$(arg model)/urdf/denso_robot_kinematics.xacro" />
-    <!-- ros2 control include -->
-    <xacro:include filename="$(find denso_robot_descriptions)/robots/$(arg model)/urdf/denso_robot.ros2_control.xacro" />
-    <!-- For other tools, modify the filename parameter to the path of your tool's xacro file. -->
-    <!-- The line with tag xacro:tool passes the parameters defined in your tool's xacro file -->
-    <!-- (see basic_camera.xacro as an example implementation) -->
-    <xacro:if value="$(arg basic_camera)">
-      <xacro:include filename="$(find denso_robot_gazebo)/sensors/basic_camera/urdf/basic_camera.xacro" />
-    </xacro:if>
-    <!-- ros2 control instance -->
-    <xacro:denso_robot_ros2_control
-      name="GazeboSystem" namespace="${namespace}"
-      sim="$(arg sim)"
-      model="$(arg model)"
-      ip_address="${ip_address}"
-      robot_name="$(arg robot_name)"
-      robot_joints="$(arg robot_joints)"
-      joint_1="$(arg joint_1)"
-      joint_2="$(arg joint_2)"
-      joint_3="$(arg joint_3)"
-      joint_4="$(arg joint_4)"
-      joint_5="$(arg joint_5)"
-      joint_6="$(arg joint_6)"
-      arm_group="$(arg arm_group)"
-      controller_type="$(arg controller_type)"
-      verbose="$(arg verbose)"
-      send_format="$(arg send_format)"
-      recv_format="$(arg recv_format)"
-      initial_positions="${xacro.load_yaml(initial_positions_file)}" />
-    <!-- Add URDF transmission elements (for ros_control) -->
-    <xacro:denso_robot_arm_transmission namespace="${namespace}" hw_interface="$(arg transmission_hw_interface)" />
-    <!-- Placeholder for ros2_control transmission which don't yet exist -->
-    <!-- links -  main serial chain -->
-    <xacro:denso_robot_arm_kinematics namespace="${namespace}" model="$(arg model)" parent="${parent}" >
-      <xacro:insert_block name="origin" />
-    </xacro:denso_robot_arm_kinematics>
-    <xacro:if value="$(arg basic_camera)">
-      <xacro:basic_camera namespace="${namespace}" end_effector="J6" />
-    </xacro:if>
+  <xacro:macro name="denso_robot" params="model
+                                          namespace
+                                          parent
+                                          *origin
+                                          transmission_hw_interface:=hardware_interface/PositionJointInterface
+                                          sim:=false
+                                          basic_camera:=false
+                                          ip_address
+                                          send_format
+                                          recv_format
+                                          verbose:=false">
+  <!-- Robot data required by the denso driver -->
+  <xacro:arg name="ip_address" default=""/>
+  <xacro:arg name="robot_name" default="VS050A3-AV6-NNN-NNN A"/> <!-- "robot_name" param must be consistent with the @TYPE_NAME variable of the real robot !! -->
+  <xacro:arg name="robot_joints" default="6"/> <!-- number of total joints in the kinematic chain -->
+  <xacro:arg name="joint_1" default="1"/> <!-- 0 = prismatic , 1 = revolute -->
+  <xacro:arg name="joint_2" default="1"/> <!-- 0 = prismatic , 1 = revolute -->
+  <xacro:arg name="joint_3" default="1"/> <!-- 0 = prismatic , 1 = revolute -->
+  <xacro:arg name="joint_4" default="1"/> <!-- 0 = prismatic , 1 = revolute -->
+  <xacro:arg name="joint_5" default="1"/> <!-- 0 = prismatic , 1 = revolute -->
+  <xacro:arg name="joint_6" default="1"/> <!-- 0 = prismatic , 1 = revolute -->
+  <xacro:arg name="controller_type" default="8"/> <!-- 8 = RC8 , 9 = RC9 -->
+  <xacro:arg name="arm_group" default="0"/>
+  <xacro:arg name="send_format" default="288"/>
+  <xacro:arg name="recv_format" default="292"/>
+  <xacro:arg name="verbose" default="false"/>
+  <!-- initial position for simulations-->
+  <xacro:arg name="initial_positions_file" default="$(find denso_robot_descriptions)/robots/$(arg model)/initial_positions.yaml" />
+  <!-- convert to property to use substitution in function -->
+  <xacro:property name="initial_positions_file" default="$(arg initial_positions_file)" />
+  <xacro:include filename="$(find denso_robot_descriptions)/robots/$(arg model)/urdf/denso_robot_transmissions.xacro" />
+  <!-- robot kinematics include -->
+  <xacro:include filename="$(find denso_robot_descriptions)/robots/$(arg model)/urdf/denso_robot_kinematics.xacro" />
+  <!-- ros2 control include -->
+  <xacro:include filename="$(find denso_robot_descriptions)/robots/$(arg model)/urdf/denso_robot.ros2_control.xacro" />
+  <!-- For other tools, modify the filename parameter to the path of your tool's xacro file. -->
+  <!-- The line with tag xacro:tool passes the parameters defined in your tool's xacro file -->
+  <!-- (see basic_camera.xacro as an example implementation) -->
+  <xacro:if value="$(arg basic_camera)">
+    <xacro:include filename="$(find denso_robot_gazebo)/sensors/basic_camera/urdf/basic_camera.xacro" />
+  </xacro:if>
+  <!-- ros2 control instance -->
+  <xacro:denso_robot_ros2_control name="VS050"
+                                  namespace="${namespace}"
+                                  sim="$(arg sim)"
+                                  model="$(arg model)"
+                                  ip_address="${ip_address}"
+                                  robot_name="$(arg robot_name)"
+                                  robot_joints="$(arg robot_joints)"
+                                  joint_1="$(arg joint_1)"
+                                  joint_2="$(arg joint_2)"
+                                  joint_3="$(arg joint_3)"
+                                  joint_4="$(arg joint_4)"
+                                  joint_5="$(arg joint_5)"
+                                  joint_6="$(arg joint_6)"
+                                  arm_group="$(arg arm_group)"
+                                  controller_type="$(arg controller_type)"
+                                  verbose="$(arg verbose)"
+                                  send_format="$(arg send_format)"
+                                  recv_format="$(arg recv_format)"
+                                  initial_positions="${xacro.load_yaml(initial_positions_file)}" />
+  <!-- Add URDF transmission elements (for ros_control) -->
+  <xacro:denso_robot_arm_transmission namespace="${namespace}" hw_interface="$(arg transmission_hw_interface)" />
+  <!-- Placeholder for ros2_control transmission which don't yet exist -->
+  <!-- links -  main serial chain -->
+  <xacro:denso_robot_arm_kinematics namespace="${namespace}" model="$(arg model)" parent="${parent}">
+    <xacro:insert_block name="origin" />
+  </xacro:denso_robot_arm_kinematics>
+  <xacro:if value="$(arg basic_camera)">
+    <xacro:basic_camera namespace="${namespace}" end_effector="J6" />
+  </xacro:if>
   </xacro:macro>
 </robot>

File: denso_robot_descriptions/robots/vs050/urdf/denso_robot_transmissions.xacro (robot description, xacro)
@@ -1,4 +1,4 @@
 <?xml version="1.0"?>
-<robot xmlns:xacro="http://wiki.ros.org/xacro">
+<robot xmlns:xacro="http://www.ros.org/wiki/xacro">
   <!--
     NOTE the macro defined in this file is NOT part of the public API of this

File: denso_robot_descriptions/urdf/denso_robot.urdf.xacro (robot description, xacro)
@@ -1,40 +1,41 @@
 <?xml version="1.0"?>
-<robot xmlns:xacro="http://wiki.ros.org/xacro" name="$(arg model)">
-   <!-- robot name parameter -->
-   <xacro:arg name="model" default="denso_robot"/>
-   <!-- import main macro -->
-   <xacro:include filename="$(find denso_robot_descriptions)/robots/$(arg model)/urdf/denso_robot_macro.xacro"/>
-   <!-- parameters -->
-   <xacro:arg name="namespace" default="" />
-   <xacro:arg name="transmission_hw_interface" default=""/>
-   <!-- ros2_control related parameters -->
-   <xacro:arg name="verbose" default="false" />
-   <xacro:arg name="sim" default="false" />
-   <xacro:arg name="basic_camera" default="false" />
-   <xacro:arg name="ip_address" default="192.168.0.1" />
-   <xacro:arg name="send_format" default="288" />
-   <xacro:arg name="recv_format" default="292" />
-   <xacro:arg name="xyz" default="0 0 0" />
-   <xacro:arg name="rpy" default="0 0 0" />
-   <!-- Root link -->
-   <link name="world"/>
-   <!-- arm -->
-   <xacro:denso_robot
-     model="$(arg model)"
-     namespace="$(arg namespace)"
-     parent="world"
-     transmission_hw_interface="$(arg transmission_hw_interface)"
-     sim="$(arg sim)"
-     basic_camera="$(arg basic_camera)"
-     ip_address="$(arg ip_address)"
-     verbose="$(arg verbose)"
-     send_format="$(arg send_format)"
-     recv_format="$(arg recv_format)" >
-     <origin xyz="$(arg xyz)" rpy="$(arg rpy)" />
-   </xacro:denso_robot>
-   <gazebo>
-	   <plugin filename="gz_ros2_control-system" name="gz_ros2_control::GazeboSimROS2ControlPlugin">
-      <parameters>$(find denso_robot_moveit_config)/robots/$(arg model)/config/denso_robot_controllers.yaml</parameters>
-     </plugin>
-   </gazebo>
+<robot xmlns:xacro="http://www.ros.org/wiki/xacro" name="$(arg model)">
+  <!-- robot name parameter -->
+  <xacro:arg name="model" default="denso_robot" />
+  <!-- import main macro -->
+  <xacro:include filename="$(find denso_robot_descriptions)/robots/$(arg model)/urdf/denso_robot_macro.xacro" />
+  <!-- parameters -->
+  <xacro:arg name="namespace" default="" />
+  <xacro:arg name="transmission_hw_interface" default="" />
+  <!-- ros2_control related parameters -->
+  <xacro:arg name="verbose" default="false" />
+  <xacro:arg name="sim" default="false" />
+  <xacro:arg name="basic_camera" default="false" />
+  <xacro:arg name="ip_address" default="192.168.0.1" />
+  <xacro:arg name="send_format" default="288" />
+  <xacro:arg name="recv_format" default="292" />
+  <xacro:arg name="xyz" default="0 0 0" />
+  <xacro:arg name="rpy" default="0 0 0" />
+  <!-- Root link -->
+  <link name="world" />
+  <!-- arm -->
+  <xacro:denso_robot model="$(arg model)"
+                     namespace="$(arg namespace)"
+                     parent="world"
+                     transmission_hw_interface="$(arg transmission_hw_interface)"
+                     sim="$(arg sim)"
+                     basic_camera="$(arg basic_camera)"
+                     ip_address="$(arg ip_address)"
+                     verbose="$(arg verbose)"
+                     send_format="$(arg send_format)"
+                     recv_format="$(arg recv_format)" >
+    <origin xyz="$(arg xyz)" rpy="$(arg rpy)" />
+  </xacro:denso_robot>
+  <gazebo>
+    <plugin filename="gz_ros2_control-system" name="gz_ros2_control::GazeboSimROS2ControlPlugin">
+      <parameters>
+        $(find denso_robot_moveit_config)/robots/$(arg model)/config/denso_robot_controllers.yaml
+      </parameters>
+    </plugin>
+  </gazebo>
 </robot>
