Commit message: feat(vs050): overhaul MoveIt configuration and URDF kinematics
- Add standard `flange` and `tool0` links to the URDF and integrate them into the SRDF as a dedicated `end_effector` group.
- Define a predefined `home` group state and generate a comprehensive collision checking matrix in the SRDF.
- Enable Pilz cartesian limits in the bringup launch pipeline via the MoveItConfigsBuilder.
- Relocate `initial_positions.yaml` to the moveit_config package and streamline how xacro loads initial values into ros2_control interfaces.
- Refine physical and MoveIt joint limits, applying velocity/acceleration scaling factors and exact radian conversions.

File: denso_robot_descriptions/robots/vs050/urdf/denso_robot.ros2_control.xacro (robot description, xacro)
@@ -21,5 +21,5 @@
                        controller_type
                        verbose
-                       initial_positions">
+                       initial_positions_file">
     <ros2_control name="${namespace}${name}" type="system">
 	  <!-- joint limits include -->
@@ -50,5 +50,5 @@
         </xacro:unless>
       </hardware>
-      <xacro:denso_robot_control_limits namespace="${namespace}" initial_positions="${initial_positions}" />
+      <xacro:denso_robot_control_limits namespace="${namespace}" initial_positions_file="${initial_positions_file}" />
     </ros2_control>
   </xacro:macro>

File: denso_robot_descriptions/robots/vs050/urdf/denso_robot_joint_limits.xacro (robot description, xacro)
@@ -1,95 +1,48 @@
 <?xml version='1.0' encoding='UTF-8'?>
 <robot xmlns:xacro="http://www.ros.org/wiki/xacro">
-	<xacro:macro name="denso_robot_control_limits" params="namespace initial_positions">
-		<joint name="${namespace}joint_1">
-			<command_interface name="position">
-				<param name="min">-2.967060</param>
-				<param name="max">2.967060</param>
-			</command_interface>
-			<command_interface name="velocity">
-				<param name="min">0</param>
-				<param name="max">0.392699081698724</param>
-			</command_interface>
-			<state_interface name="position">
-				<param name="initial_value">${initial_positions['joint_1']}</param>
-			</state_interface>
-			<state_interface name="velocity"/>
-			<state_interface name="effort"/>
-		</joint>
-		<joint name="${namespace}joint_2">
-			<command_interface name="position">
-				<param name="min">-2.094395</param>
-				<param name="max">2.094395</param>
-			</command_interface>
-			<command_interface name="velocity">
-				<param name="min">0</param>
-				<param name="max">0.261799387799149</param>
-			</command_interface>
-			<state_interface name="position">
-				<param name="initial_value">${initial_positions['joint_2']}</param>
-			</state_interface>
-			<state_interface name="velocity"/>
-			<state_interface name="effort"/>
-		</joint>
-		<joint name="${namespace}joint_3">
-			<command_interface name="position">
-				<param name="min">${radians(-120)}</param>
-				<param name="max">${radians(151)}</param>
-			</command_interface>
-			<command_interface name="velocity">
-				<param name="min">0</param>
-				<param name="max">0.285832571599111</param>
-			</command_interface>
-			<state_interface name="position">
-				<param name="initial_value">${initial_positions['joint_3']}</param>
-			</state_interface>
-			<state_interface name="velocity"/>
-			<state_interface name="effort"/>
-		</joint>
-		<joint name="${namespace}joint_4">
-			<command_interface name="position">
-				<param name="min">-4.712389</param>
-				<param name="max">4.712389</param>
-			</command_interface>
-			<command_interface name="velocity">
-				<param name="min">0</param>
-				<param name="max">0.392699081698724</param>
-			</command_interface>
-			<state_interface name="position">
-				<param name="initial_value">${initial_positions['joint_4']}</param>
-			</state_interface>
-			<state_interface name="velocity"/>
-			<state_interface name="effort"/>
-		</joint>
-		<joint name="${namespace}joint_5">
-			<command_interface name="position">
-				<param name="min">-2.094395</param>
-				<param name="max">2.094395</param>
-			</command_interface>
-			<command_interface name="velocity">
-				<param name="min">0</param>
-				<param name="max">0.302168853397778</param>
-			</command_interface>
-			<state_interface name="position">
-				<param name="initial_value">${initial_positions['joint_5']}</param>
-			</state_interface>
-			<state_interface name="velocity"/>
-			<state_interface name="effort"/>
-		</joint>
-		<joint name="${namespace}joint_6">
-			<command_interface name="position">
-				<param name="min">-6.283185</param>
-				<param name="max">6.283185</param>
-			</command_interface>
-			<command_interface name="velocity">
-				<param name="min">0</param>
-				<param name="max">0.628318530717959</param>
-			</command_interface>
-			<state_interface name="position">
-				<param name="initial_value">${initial_positions['joint_6']}</param>
-			</state_interface>
-			<state_interface name="velocity"/>
-			<state_interface name="effort"/>
-		</joint>
+	<xacro:macro name="denso_robot_control_limits" params="namespace initial_positions_file">
+    <xacro:property name="initial_positions" value="${xacro.load_yaml(initial_positions_file)['initial_positions']}" />
+	  <joint name="joint_1">
+      <command_interface name="position" />
+      <state_interface name="position">
+        <param name="initial_value">${initial_positions['joint_1']}</param>
+      </state_interface>
+      <state_interface name="velocity" />
+    </joint>
+    <joint name="joint_2">
+      <command_interface name="position" />
+      <state_interface name="position">
+        <param name="initial_value">${initial_positions['joint_2']}</param>
+      </state_interface>
+      <state_interface name="velocity" />
+    </joint>
+    <joint name="joint_3">
+      <command_interface name="position" />
+      <state_interface name="position">
+        <param name="initial_value">${initial_positions['joint_3']}</param>
+      </state_interface>
+      <state_interface name="velocity" />
+    </joint>
+    <joint name="joint_4">
+      <command_interface name="position" />
+      <state_interface name="position">
+        <param name="initial_value">${initial_positions['joint_4']}</param>
+      </state_interface>
+      <state_interface name="velocity" />
+    </joint>
+    <joint name="joint_5">
+      <command_interface name="position" />
+      <state_interface name="position">
+        <param name="initial_value">${initial_positions['joint_5']}</param>
+      </state_interface>
+      <state_interface name="velocity" />
+    </joint>
+    <joint name="joint_6">
+      <command_interface name="position" />
+      <state_interface name="position">
+        <param name="initial_value">${initial_positions['joint_6']}</param>
+      </state_interface>
+      <state_interface name="velocity" />
+    </joint>
 	</xacro:macro>
 </robot>

File: denso_robot_descriptions/robots/vs050/urdf/denso_robot_kinematics.xacro (robot description, xacro)
@@ -3,188 +3,203 @@
 	<xacro:macro name="denso_robot_arm_kinematics" params="namespace model parent *origin">
 		<joint name="${namespace}joint_w" type="fixed">
-			<xacro:insert_block name="origin" />
-			<parent link="${parent}"/>
-			<child link="${namespace}base_link"/>
+			<xacro:insert_block name="origin"  />
+			<parent link="${parent}" />
+			<child link="${namespace}base_link" />
 		</joint>
 		<link name="${namespace}base_link">
 			<visual>
-				<origin rpy="0 0 0" xyz="0 0 0"/>
-				<geometry>
-					<mesh filename="file:///$(find denso_robot_descriptions)/robots/$(arg model)/meshes/base_link.dae" scale="1 1 1"/>
-				</geometry>
-			</visual>
-			<collision>
-				<origin rpy="0 0 0" xyz="0 0 0"/>
-				<geometry>
-					<mesh filename="file:///$(find denso_robot_descriptions)/robots/$(arg model)/meshes/base_link.dae" scale="1 1 1"/>
-				</geometry>
-			</collision>
-			<inertial>
-				<mass value="1"/>
-				<origin rpy="0.000000 0.000000 0.000000" xyz="0.000000 0.000000 0.000000"/>
-				<inertia ixx="1" ixy="0" ixz="0" iyy="1" iyz="0" izz="1"/>
+				<origin rpy="0 0 0" xyz="0 0 0" />
+				<geometry>
+					<mesh filename="file:///$(find denso_robot_descriptions)/robots/$(arg model)/meshes/base_link.dae" scale="1 1 1" />
+				</geometry>
+			</visual>
+			<collision>
+				<origin rpy="0 0 0" xyz="0 0 0" />
+				<geometry>
+					<mesh filename="file:///$(find denso_robot_descriptions)/robots/$(arg model)/meshes/base_link.dae" scale="1 1 1" />
+				</geometry>
+			</collision>
+			<inertial>
+				<mass value="1" />
+				<origin rpy="0.000000 0.000000 0.000000" xyz="0.000000 0.000000 0.000000" />
+				<inertia ixx="1" ixy="0" ixz="0" iyy="1" iyz="0" izz="1" />
 			</inertial>
 		</link>
 		<link name="${namespace}J1">
 			<visual>
-				<origin rpy="0 0 0" xyz="0 0 0"/>
-				<geometry>
-					<mesh filename="file:///$(find denso_robot_descriptions)/robots/$(arg model)/meshes/J1.dae" scale="1 1 1"/>
-				</geometry>
-			</visual>
-			<collision>
-				<origin rpy="0 0 0" xyz="0 0 0"/>
-				<geometry>
-					<mesh filename="file:///$(find denso_robot_descriptions)/robots/$(arg model)/meshes/J1.dae" scale="1 1 1"/>
-				</geometry>
-			</collision>
-			<inertial>
-				<mass value="1"/>
-				<origin rpy="0.000000 0.000000 0.000000" xyz="0.000000 0.000000 0.000000"/>
-				<inertia ixx="1" ixy="0" ixz="0" iyy="1" iyz="0" izz="1"/>
+				<origin rpy="0 0 0" xyz="0 0 0" />
+				<geometry>
+					<mesh filename="file:///$(find denso_robot_descriptions)/robots/$(arg model)/meshes/J1.dae" scale="1 1 1" />
+				</geometry>
+			</visual>
+			<collision>
+				<origin rpy="0 0 0" xyz="0 0 0" />
+				<geometry>
+					<mesh filename="file:///$(find denso_robot_descriptions)/robots/$(arg model)/meshes/J1.dae" scale="1 1 1" />
+				</geometry>
+			</collision>
+			<inertial>
+				<mass value="1" />
+				<origin rpy="0.000000 0.000000 0.000000" xyz="0.000000 0.000000 0.000000" />
+				<inertia ixx="1" ixy="0" ixz="0" iyy="1" iyz="0" izz="1" />
 			</inertial>
 		</link>
 		<joint name="${namespace}joint_1" type="revolute">
-			<parent link="${namespace}base_link"/>
-			<child link="${namespace}J1"/>
-			<origin rpy="0.000000 0.000000 0.000000" xyz="0.000000 0.000000 0.181500"/>
-			<axis xyz="-0.000000 -0.000000 1.000000"/>
-			<limit effort="1000" lower="-2.96705972839036" upper="2.96705972839036" velocity="3.73064127613788"/> <!-- effort value is arbitary for make gazebo simulation runs without gravity problems -->
-			<dynamics damping="0" friction="0"/>
+			<parent link="${namespace}base_link" />
+			<child link="${namespace}J1" />
+			<origin rpy="0.000000 0.000000 0.000000" xyz="0.000000 0.000000 0.181500" />
+			<axis xyz="-0.000000 -0.000000 1.000000" />
+      <!-- effort value is arbitary for make gazebo simulation runs without gravity problems -->
+			<limit effort="1000" lower="${radians(-170)}" upper="${radians(170)}" velocity="${radians(425)}" />
+			<dynamics damping="0" friction="0" />
 		</joint>
 		<link name="${namespace}J2">
 			<visual>
-				<origin rpy="0 0 0" xyz="0 0 0"/>
-				<geometry>
-					<mesh filename="file:///$(find denso_robot_descriptions)/robots/$(arg model)/meshes/J2.dae" scale="1 1 1"/>
-				</geometry>
-			</visual>
-			<collision>
-				<origin rpy="0 0 0" xyz="0 0 0"/>
-				<geometry>
-					<mesh filename="file:///$(find denso_robot_descriptions)/robots/$(arg model)/meshes/J2.dae" scale="1 1 1"/>
-				</geometry>
-			</collision>
-			<inertial>
-				<mass value="1"/>
-				<origin rpy="0.000000 0.000000 0.000000" xyz="0.000000 0.000000 0.000000"/>
-				<inertia ixx="1" ixy="0" ixz="0" iyy="1" iyz="0" izz="1"/>
+				<origin rpy="0 0 0" xyz="0 0 0" />
+				<geometry>
+					<mesh filename="file:///$(find denso_robot_descriptions)/robots/$(arg model)/meshes/J2.dae" scale="1 1 1" />
+				</geometry>
+			</visual>
+			<collision>
+				<origin rpy="0 0 0" xyz="0 0 0" />
+				<geometry>
+					<mesh filename="file:///$(find denso_robot_descriptions)/robots/$(arg model)/meshes/J2.dae" scale="1 1 1" />
+				</geometry>
+			</collision>
+			<inertial>
+				<mass value="1" />
+				<origin rpy="0.000000 0.000000 0.000000" xyz="0.000000 0.000000 0.000000" />
+				<inertia ixx="1" ixy="0" ixz="0" iyy="1" iyz="0" izz="1" />
 			</inertial>
 		</link>
 		<joint name="${namespace}joint_2" type="revolute">
-			<parent link="${namespace}J1"/>
-			<child link="${namespace}J2"/>
-			<origin rpy="0.000000 0.000000 0.000000" xyz="0.000000 0.000000 0.163500"/>
-			<axis xyz="-0.000000 1.000000 -0.000000"/>
-			<limit effort="1000" lower="-2.0943951023932" upper="2.0943951023932" velocity="2.48709418409192"/> <!-- effort value is arbitary for make gazebo simulation runs without gravity problems -->
-			<dynamics damping="0" friction="0"/>
+			<parent link="${namespace}J1" />
+			<child link="${namespace}J2" />
+			<origin rpy="0.000000 0.000000 0.000000" xyz="0.000000 0.000000 0.163500" />
+			<axis xyz="-0.000000 1.000000 -0.000000" />
+      <!-- effort value is arbitary for make gazebo simulation runs without gravity problems -->
+			<limit effort="1000" lower="${radians(-120)}" upper="${radians(120)}" velocity="${radians(340)}" />
+			<dynamics damping="0" friction="0" />
 		</joint>
 		<link name="${namespace}J3">
 			<visual>
-				<origin rpy="0 0 0" xyz="0 0 0"/>
-				<geometry>
-					<mesh filename="file:///$(find denso_robot_descriptions)/robots/$(arg model)/meshes/J3.dae" scale="1 1 1"/>
-				</geometry>
-			</visual>
-			<collision>
-				<origin rpy="0 0 0" xyz="0 0 0"/>
-				<geometry>
-					<mesh filename="file:///$(find denso_robot_descriptions)/robots/$(arg model)/meshes/J3.dae" scale="1 1 1"/>
-				</geometry>
-			</collision>
-			<inertial>
-				<mass value="1"/>
-				<origin rpy="0.000000 0.000000 0.000000" xyz="0.000000 0.000000 0.000000"/>
-				<inertia ixx="1" ixy="0" ixz="0" iyy="1" iyz="0" izz="1"/>
+				<origin rpy="0 0 0" xyz="0 0 0" />
+				<geometry>
+					<mesh filename="file:///$(find denso_robot_descriptions)/robots/$(arg model)/meshes/J3.dae" scale="1 1 1" />
+				</geometry>
+			</visual>
+			<collision>
+				<origin rpy="0 0 0" xyz="0 0 0" />
+				<geometry>
+					<mesh filename="file:///$(find denso_robot_descriptions)/robots/$(arg model)/meshes/J3.dae" scale="1 1 1" />
+				</geometry>
+			</collision>
+			<inertial>
+				<mass value="1" />
+				<origin rpy="0.000000 0.000000 0.000000" xyz="0.000000 0.000000 0.000000" />
+				<inertia ixx="1" ixy="0" ixz="0" iyy="1" iyz="0" izz="1" />
 			</inertial>
 		</link>
 		<joint name="${namespace}joint_3" type="revolute">
-			<parent link="${namespace}J2"/>
-			<child link="${namespace}J3"/>
-			<origin rpy="0.000000 0.000000 0.000000" xyz="0.000000 0.000000 0.250000"/>
-			<axis xyz="-0.000000 1.000000 -0.000000"/>
-			<limit effort="1000" lower="-2.18166156499291" upper="2.70526034059121" velocity="2.71540943019156"/> <!-- effort value is arbitary for make gazebo simulation runs without gravity problems -->
-			<dynamics damping="0" friction="0"/>
+			<parent link="${namespace}J2" />
+			<child link="${namespace}J3" />
+			<origin rpy="0.000000 0.000000 0.000000" xyz="0.000000 0.000000 0.250000" />
+			<axis xyz="-0.000000 1.000000 -0.000000" />
+      <!-- effort value is arbitary for make gazebo simulation runs without gravity problems -->
+			<limit effort="1000" lower="${radians(-120)}" upper="${radians(151)}" velocity="${radians(385.72)}" />
+			<dynamics damping="0" friction="0" />
 		</joint>
 		<link name="${namespace}J4">
 			<visual>
-				<origin rpy="0 0 0" xyz="0 0 0"/>
-				<geometry>
-					<mesh filename="file:///$(find denso_robot_descriptions)/robots/$(arg model)/meshes/J4.dae" scale="1 1 1"/>
-				</geometry>
-			</visual>
-			<collision>
-				<origin rpy="0 0 0" xyz="0 0 0"/>
-				<geometry>
-					<mesh filename="file:///$(find denso_robot_descriptions)/robots/$(arg model)/meshes/J4.dae" scale="1 1 1"/>
-				</geometry>
-			</collision>
-			<inertial>
-				<mass value="1"/>
-				<origin rpy="0.000000 0.000000 0.000000" xyz="0.000000 0.000000 0.000000"/>
-				<inertia ixx="1" ixy="0" ixz="0" iyy="1" iyz="0" izz="1"/>
+				<origin rpy="0 0 0" xyz="0 0 0" />
+				<geometry>
+					<mesh filename="file:///$(find denso_robot_descriptions)/robots/$(arg model)/meshes/J4.dae" scale="1 1 1" />
+				</geometry>
+			</visual>
+			<collision>
+				<origin rpy="0 0 0" xyz="0 0 0" />
+				<geometry>
+					<mesh filename="file:///$(find denso_robot_descriptions)/robots/$(arg model)/meshes/J4.dae" scale="1 1 1" />
+				</geometry>
+			</collision>
+			<inertial>
+				<mass value="1" />
+				<origin rpy="0.000000 0.000000 0.000000" xyz="0.000000 0.000000 0.000000" />
+				<inertia ixx="1" ixy="0" ixz="0" iyy="1" iyz="0" izz="1" />
 			</inertial>
 		</link>
 		<joint name="${namespace}joint_4" type="revolute">
-			<parent link="${namespace}J3"/>
-			<child link="${namespace}J4"/>
-			<origin rpy="0.000000 0.000000 0.000000" xyz="-0.010000 0.000000 0.119500"/>
-			<axis xyz="-0.000000 -0.000000 1.000000"/>
-			<limit effort="1000" lower="-4.71238898038469" upper="4.71238898038469" velocity="3.73064127613788"/> <!-- effort value is arbitary for make gazebo simulation runs without gravity problems -->
-			<dynamics damping="0" friction="0"/>
+			<parent link="${namespace}J3" />
+			<child link="${namespace}J4" />
+			<origin rpy="0.000000 0.000000 0.000000" xyz="-0.010000 0.000000 0.119500" />
+			<axis xyz="-0.000000 -0.000000 1.000000" />
+			<limit effort="6.66" lower="${radians(-270)}" upper="${radians(270)}" velocity="${radians(425)}" />
+			<dynamics damping="0" friction="0" />
 		</joint>
 		<link name="${namespace}J5">
 			<visual>
-				<origin rpy="0 0 0" xyz="0 0 0"/>
-				<geometry>
-					<mesh filename="file:///$(find denso_robot_descriptions)/robots/$(arg model)/meshes/J5.dae" scale="1 1 1"/>
-				</geometry>
-			</visual>
-			<collision>
-				<origin rpy="0 0 0" xyz="0 0 0"/>
-				<geometry>
-					<mesh filename="file:///$(find denso_robot_descriptions)/robots/$(arg model)/meshes/J5.dae" scale="1 1 1"/>
-				</geometry>
-			</collision>
-			<inertial>
-				<mass value="1"/>
-				<origin rpy="0.000000 0.000000 0.000000" xyz="0.000000 0.000000 0.000000"/>
-				<inertia ixx="1" ixy="0" ixz="0" iyy="1" iyz="0" izz="1"/>
+				<origin rpy="0 0 0" xyz="0 0 0" />
+				<geometry>
+					<mesh filename="file:///$(find denso_robot_descriptions)/robots/$(arg model)/meshes/J5.dae" scale="1 1 1" />
+				</geometry>
+			</visual>
+			<collision>
+				<origin rpy="0 0 0" xyz="0 0 0" />
+				<geometry>
+					<mesh filename="file:///$(find denso_robot_descriptions)/robots/$(arg model)/meshes/J5.dae" scale="1 1 1" />
+				</geometry>
+			</collision>
+			<inertial>
+				<mass value="1" />
+				<origin rpy="0.000000 0.000000 0.000000" xyz="0.000000 0.000000 0.000000" />
+				<inertia ixx="1" ixy="0" ixz="0" iyy="1" iyz="0" izz="1" />
 			</inertial>
 		</link>
 		<joint name="${namespace}joint_5" type="revolute">
-			<parent link="${namespace}J4"/>
-			<child link="${namespace}J5"/>
-			<origin rpy="0.000000 0.000000 0.000000" xyz="0.000000 0.000000 0.135500"/>
-			<axis xyz="-0.000000 1.000000 -0.000000"/>
-			<limit effort="1000" lower="-2.0943951023932" upper="2.0943951023932" velocity="2.87060410727889"/> <!-- effort value is arbitary for make gazebo simulation runs without gravity problems -->
-			<dynamics damping="0" friction="0"/>
+			<parent link="${namespace}J4" />
+			<child link="${namespace}J5" />
+			<origin rpy="0.000000 0.000000 0.000000" xyz="0.000000 0.000000 0.135500" />
+			<axis xyz="-0.000000 1.000000 -0.000000" />
+			<limit effort="6.66" lower="${radians(-120)}" upper="${radians(120)}" velocity="${radians(327.01)}" />
+			<dynamics damping="0" friction="0" />
 		</joint>
 		<link name="${namespace}J6">
 			<visual>
-				<origin rpy="0 0 0" xyz="0 0 0"/>
-				<geometry>
-					<mesh filename="file:///$(find denso_robot_descriptions)/robots/$(arg model)/meshes/J6.dae" scale="1 1 1"/>
-				</geometry>
-			</visual>
-			<collision>
-				<origin rpy="0 0 0" xyz="0 0 0"/>
-				<geometry>
-					<mesh filename="file:///$(find denso_robot_descriptions)/robots/$(arg model)/meshes/J6.dae" scale="1 1 1"/>
-				</geometry>
-			</collision>
-			<inertial>
-				<mass value="1"/>
-				<origin rpy="0.000000 0.000000 0.000000" xyz="0.000000 0.000000 0.000000"/>
-				<inertia ixx="1" ixy="0" ixz="0" iyy="1" iyz="0" izz="1"/>
+				<origin rpy="0 0 0" xyz="0 0 0" />
+				<geometry>
+					<mesh filename="file:///$(find denso_robot_descriptions)/robots/$(arg model)/meshes/J6.dae" scale="1 1 1" />
+				</geometry>
+			</visual>
+			<collision>
+				<origin rpy="0 0 0" xyz="0 0 0" />
+				<geometry>
+					<mesh filename="file:///$(find denso_robot_descriptions)/robots/$(arg model)/meshes/J6.dae" scale="1 1 1" />
+				</geometry>
+			</collision>
+			<inertial>
+				<mass value="1" />
+				<origin rpy="0.000000 0.000000 0.000000" xyz="0.000000 0.000000 0.000000" />
+				<inertia ixx="1" ixy="0" ixz="0" iyy="1" iyz="0" izz="1" />
 			</inertial>
 		</link>
 		<joint name="${namespace}joint_6" type="revolute">
-			<parent link="${namespace}J5"/>
-			<child link="${namespace}J6"/>
-			<origin rpy="0.000000 0.000000 0.000000" xyz="0.000000 0.000000 0.070000"/>
-			<axis xyz="-0.000000 -0.000000 1.000000"/>
-			<limit effort="1000" lower="-6.28318530717959" upper="6.28318530717959" velocity="5.96902604182061"/> <!-- effort value is arbitary for make gazebo simulation runs without gravity problems -->
-			<dynamics damping="0" friction="0"/>
+			<parent link="${namespace}J5" />
+			<child link="${namespace}J6" />
+			<origin rpy="0.000000 0.000000 0.000000" xyz="0.000000 0.000000 0.070000" />
+			<axis xyz="-0.000000 -0.000000 1.000000" />
+			<limit effort="3.13" lower="${radians(-360)}" upper="${radians(360)}" velocity="${radians(680)}" />
+			<dynamics damping="0" friction="0" />
+		</joint>
+		<link name="flange"/>
+		<joint name="J6-flange" type="fixed">
+		<parent link="J6"/>
+		<child link="flange"/>
+		<origin rpy="0 0 0" xyz="0 0 0"/>
+		</joint>
+		<link name="tool0"/>
+		<joint name="J6-tool0" type="fixed">
+		<parent link="J6"/>
+		<child link="tool0"/>
+		<origin rpy="${radians(pi)} ${radians(-pi/2)} 0" xyz="0 0 0"/>
 		</joint>
 	</xacro:macro>
