Commit message: feat(vs050): overhaul MoveIt configuration and URDF kinematics
- Add standard `flange` and `tool0` links to the URDF and integrate them into the SRDF as a dedicated `end_effector` group.
- Define a predefined `home` group state and generate a comprehensive collision checking matrix in the SRDF.
- Enable Pilz cartesian limits in the bringup launch pipeline via the MoveItConfigsBuilder.
- Relocate `initial_positions.yaml` to the moveit_config package and streamline how xacro loads initial values into ros2_control interfaces.
- Refine physical and MoveIt joint limits, applying velocity/acceleration scaling factors and exact radian conversions.

File: denso_robot_descriptions/robots/vs050/urdf/denso_robot_macro.xacro (robot description, xacro)
@@ -36,7 +36,5 @@
   <xacro:arg name="verbose" default="false"/>
   <!-- initial position for simulations-->
-  <xacro:arg name="initial_positions_file" default="$(find denso_robot_descriptions)/robots/$(arg model)/initial_positions.yaml" />
-  <!-- convert to property to use substitution in function -->
-  <xacro:property name="initial_positions_file" default="$(arg initial_positions_file)" />
+  <xacro:arg name="initial_positions_file" default="$(find denso_robot_moveit_config)/robots/$(arg model)/config/initial_positions.yaml" />
   <xacro:include filename="$(find denso_robot_descriptions)/robots/$(arg model)/urdf/denso_robot_transmissions.xacro" />
   <!-- robot kinematics include -->
@@ -69,5 +67,5 @@
                                   send_format="$(arg send_format)"
                                   recv_format="$(arg recv_format)"
-                                  initial_positions="${xacro.load_yaml(initial_positions_file)}" />
+                                  initial_positions_file="$(arg initial_positions_file)" />
   <!-- Add URDF transmission elements (for ros_control) -->
   <xacro:denso_robot_arm_transmission namespace="${namespace}" hw_interface="$(arg transmission_hw_interface)" />

File: denso_robot_moveit_config/robots/vs050/srdf/denso_robot_macro.srdf.xacro (robot description, xacro)
@@ -1,4 +1,4 @@
-<?xml version="1.0" encoding="UTF-8"?>
-<robot xmlns:xacro="http://wiki.ros.org/xacro">
+<?xml version="1.0"?>
+<robot xmlns:xacro="http://www.ros.org/wiki/xacro">
 <!--This does not replace URDF, and is not an extension of URDF.
     This is a format for representing semantic information about the robot structure.
@@ -12,24 +12,45 @@
     <!--SUBGROUPS - Groups can also be formed by referencing to already defined group names-->
     <group name="${namespace}arm">
-		<joint name="${namespace}joint_1"/>
-		<joint name="${namespace}joint_2"/>
-		<joint name="${namespace}joint_3"/>
-		<joint name="${namespace}joint_4"/>
-		<joint name="${namespace}joint_5"/>
-		<joint name="${namespace}joint_6"/>
-	</group>
+      <joint name="${namespace}fixed_base"/>
+      <joint name="${namespace}joint_w"/>
+      <joint name="${namespace}joint_1"/>
+      <joint name="${namespace}joint_2"/>
+      <joint name="${namespace}joint_3"/>
+      <joint name="${namespace}joint_4"/>
+      <joint name="${namespace}joint_5"/>
+      <joint name="${namespace}joint_6"/>
+      <joint name="${namespace}J6-tool0"/>
+    </group>
+    <group name="${namespace}end_effector">
+        <link name="${namespace}tool0"/>
+    </group>
     <!--GROUP STATES - Purpose - Define a named state for a particular group, in terms of joint values. This is useful to define states like 'folded arms'-->
+    <group_state name="${namespace}home" group="${namespace}arm">
+      <joint name="${namespace}joint_1" value="0"/>
+      <joint name="${namespace}joint_2" value="-0.5"/>
+      <joint name="${namespace}joint_3" value="1.2"/>
+      <joint name="${namespace}joint_4" value="0"/>
+      <joint name="${namespace}joint_5" value="1.5"/>
+      <joint name="${namespace}joint_6" value="0"/>
+    </group_state>
     <!--END EFFECTOR - Purpose - Represent information about an end effector.-->
+    <end_effector name="${namespace}eff" parent_link="${namespace}tool0" group="${namespace}end_effector" parent_group="${namespace}arm"/>
     <!--VIRTUAL JOINT - Purpose - this element defines a virtual joint between a robot link and an external frame of reference (considered fixed with respect to the robot)-->
     <virtual_joint name="${namespace}fixed_base" type="fixed" parent_frame="world" child_link="${namespace}base_link" />
     <!--DISABLE COLLISIONS - By default it is assumed that any link of the robot could potentially come into collision with any other link in the robot. This tag disables collision checking between a specified pair of links. -->
-	<disable_collisions link1="${namespace}J6" link2="${namespace}J3" reason="Never"/>
-	<disable_collisions link1="${namespace}J6" link2="${namespace}J5" reason="Adjacent"/>
-	<disable_collisions link1="${namespace}J1" link2="${namespace}J2" reason="Adjacent"/>
-	<disable_collisions link1="${namespace}J1" link2="${namespace}base_link" reason="Adjacent"/>
-	<disable_collisions link1="${namespace}J2" link2="${namespace}J3" reason="Adjacent"/>
-	<disable_collisions link1="${namespace}J3" link2="${namespace}J4" reason="Adjacent"/>
-	<disable_collisions link1="${namespace}J3" link2="${namespace}J5" reason="Never"/>
-	<disable_collisions link1="${namespace}J4" link2="${namespace}J5" reason="Adjacent"/>
+	  <disable_collisions link1="${namespace}J1" link2="${namespace}J2" reason="Adjacent"/>
+    <disable_collisions link1="${namespace}J1" link2="${namespace}J3" reason="Never"/>
+    <disable_collisions link1="${namespace}J1" link2="${namespace}base_link" reason="Adjacent"/>
+    <disable_collisions link1="${namespace}J2" link2="${namespace}J3" reason="Adjacent"/>
+    <disable_collisions link1="${namespace}J2" link2="${namespace}J4" reason="Never"/>
+    <disable_collisions link1="${namespace}J2" link2="${namespace}J5" reason="Never"/>
+    <disable_collisions link1="${namespace}J2" link2="${namespace}J6" reason="Never"/>
+    <disable_collisions link1="${namespace}J2" link2="${namespace}base_link" reason="Never"/>
+    <disable_collisions link1="${namespace}J3" link2="${namespace}J4" reason="Adjacent"/>
+    <disable_collisions link1="${namespace}J3" link2="${namespace}J5" reason="Never"/>
+    <disable_collisions link1="${namespace}J3" link2="${namespace}J6" reason="Never"/>
+    <disable_collisions link1="${namespace}J4" link2="${namespace}J5" reason="Adjacent"/>
+    <disable_collisions link1="${namespace}J4" link2="${namespace}J6" reason="Never"/>
+    <disable_collisions link1="${namespace}J5" link2="${namespace}J6" reason="Adjacent"/>
   </xacro:macro>
 </robot>
