Commit message: fix(urdf): fix missing namespaces on joints/tool links and add vel/effort interfaces
Resolves namespace collisions for dual-arm setups by adding the `${namespace}` prefix to joint limits, flange, and tool0 links. Also exposes velocity command and effort state interfaces in ros2_control.

File: denso_robot_descriptions/robots/vs050/urdf/denso_robot_joint_limits.xacro (robot description, xacro)
@@ -3,45 +3,57 @@
 	<xacro:macro name="denso_robot_control_limits" params="namespace initial_positions_file">
     <xacro:property name="initial_positions" value="${xacro.load_yaml(initial_positions_file)['initial_positions']}" />
-	  <joint name="joint_1">
+	  <joint name="${namespace}joint_1">
       <command_interface name="position" />
+      <command_interface name="velocity" />
       <state_interface name="position">
         <param name="initial_value">${initial_positions['joint_1']}</param>
       </state_interface>
       <state_interface name="velocity" />
+      <state_interface name="effort"/>
     </joint>
-    <joint name="joint_2">
+    <joint name="${namespace}joint_2">
       <command_interface name="position" />
+      <command_interface name="velocity" />
       <state_interface name="position">
         <param name="initial_value">${initial_positions['joint_2']}</param>
       </state_interface>
       <state_interface name="velocity" />
+      <state_interface name="effort"/>
     </joint>
-    <joint name="joint_3">
+    <joint name="${namespace}joint_3">
       <command_interface name="position" />
+      <command_interface name="velocity" />
       <state_interface name="position">
         <param name="initial_value">${initial_positions['joint_3']}</param>
       </state_interface>
       <state_interface name="velocity" />
+      <state_interface name="effort"/>
     </joint>
-    <joint name="joint_4">
+    <joint name="${namespace}joint_4">
       <command_interface name="position" />
+      <command_interface name="velocity" />
       <state_interface name="position">
         <param name="initial_value">${initial_positions['joint_4']}</param>
       </state_interface>
       <state_interface name="velocity" />
+      <state_interface name="effort"/>
     </joint>
-    <joint name="joint_5">
+    <joint name="${namespace}joint_5">
       <command_interface name="position" />
+      <command_interface name="velocity" />
       <state_interface name="position">
         <param name="initial_value">${initial_positions['joint_5']}</param>
       </state_interface>
       <state_interface name="velocity" />
+      <state_interface name="effort"/>
     </joint>
-    <joint name="joint_6">
+    <joint name="${namespace}joint_6">
       <command_interface name="position" />
+      <command_interface name="velocity" />
       <state_interface name="position">
         <param name="initial_value">${initial_positions['joint_6']}</param>
       </state_interface>
       <state_interface name="velocity" />
+      <state_interface name="effort"/>
     </joint>
 	</xacro:macro>

File: denso_robot_descriptions/robots/vs050/urdf/denso_robot_kinematics.xacro (robot description, xacro)
@@ -191,14 +191,14 @@
 			<dynamics damping="0" friction="0" />
 		</joint>
-		<link name="flange"/>
-		<joint name="J6-flange" type="fixed">
-		<parent link="J6"/>
-		<child link="flange"/>
+		<link name="${namespace}flange"/>
+		<joint name="${namespace}J6-flange" type="fixed">
+		<parent link="${namespace}J6"/>
+		<child link="${namespace}flange"/>
 		<origin rpy="0 0 0" xyz="0 0 0"/>
 		</joint>
-		<link name="tool0"/>
-		<joint name="J6-tool0" type="fixed">
-		<parent link="J6"/>
-		<child link="tool0"/>
+		<link name="${namespace}tool0"/>
+		<joint name="${namespace}J6-tool0" type="fixed">
+		<parent link="${namespace}J6"/>
+		<child link="${namespace}tool0"/>
 		<origin rpy="${radians(pi)} ${radians(-pi/2)} 0" xyz="0 0 0"/>
 		</joint>
