Commit message: fix: problemas com comentários

File: denso_robot_descriptions/robots/vs050/urdf/denso_robot_macro.xacro (robot description, xacro)
@@ -39,7 +39,4 @@
     <!-- ros2 control include -->
     <xacro:include filename="$(find denso_robot_descriptions)/robots/$(arg model)/urdf/denso_robot.ros2_control.xacro" />
-    <!-- For other tools, modify the filename parameter to the path of your tool's xacro file.
-    The line with tag <xacro:tool ... \> passes the parameters defined in your tool's xacro file
-    (see basic_camera.xacro as an example implementation) -->
     <xacro:include filename="$(find denso_robot_descriptions)/tools/basic_camera/urdf/basic_camera.xacro" />
     <!-- ros2 control instance -->

File: denso_robot_descriptions/tools/basic_camera/urdf/basic_camera.xacro (robot description, xacro)
@@ -1,5 +1,4 @@
 <?xml version='1.0' encoding='UTF-8'?>
 <robot xmlns:xacro="http://www.ros.org/wiki/xacro">
-    <!-- here you define the parameters you want your xacro file to receive. -->
     <xacro:macro name="tool" params="namespace">
     <link name="$(arg namespace)basic_camera_link">
@@ -10,20 +9,15 @@
 		<collision>
 			<geometry>
-				<box size="0.01 0.01 0.01"/> <!-- if your tool has meshes, define the path to it here,
-                                                  example: tools/basic_camera/meshes/.
-                                                  See the vs050 robot urdf implementation as an example. -->
+				<box size="0.01 0.01 0.01"/>
 			</geometry>
 		</collision>
 		<visual>
 			<geometry>
-				<box size="0.01 0.01 0.01"/> <!-- if your tool has meshes, define the path to it here
-                                                  example: tools/basic_camera/meshes/.
-                                                  see the vs050 robot urdf implementation as an example. -->
+				<box size="0.01 0.01 0.01"/>
 			</geometry>
 		</visual>
 	</link>
 	<joint name="$(arg namespace)basic_camera_joint" type="fixed">
-		<parent link="$(arg namespace)J6"/> <!-- here you define where your tool will connect.
-                                                 In this case, it's at joint 6. -->
+		<parent link="$(arg namespace)J6"/>
 		<child link="$(arg namespace)basic_camera_link"/>
 		<origin rpy="0 ${radians(-90)} 0" xyz="0 0 0.01"/>

Commit message: refactor: rename basic_camera macro from "tool" to "basic_camera"

File: denso_robot_descriptions/robots/vs050/urdf/denso_robot_macro.xacro (robot description, xacro)
@@ -75,5 +75,5 @@
     </xacro:denso_robot_arm_kinematics>
     <xacro:if value="$(arg basic_camera)">
-      <xacro:tool namespace="${namespace}" />
+      <xacro:basic_camera namespace="${namespace}" />
     </xacro:if>
   </xacro:macro>

File: denso_robot_descriptions/tools/basic_camera/urdf/basic_camera.xacro (robot description, xacro)
@@ -2,5 +2,5 @@
 <robot xmlns:xacro="http://www.ros.org/wiki/xacro">
     <!-- here you define the parameters you want your xacro file to receive. -->
-    <xacro:macro name="tool" params="namespace">
+    <xacro:macro name="basic_camera" params="namespace">
     <!-- if your tool has meshes, define the path to it in geometry tag. -->
     <!-- see the vs050 robot urdf implementation as an example. -->

Commit message: refactor: replace basic_camera with gz_cam in launch and urdf files
Updates all references, launch arguments, topics, and xacro macros from `basic_camera` to `gz_cam` across the single/dual robot setups, and removes the deprecated basic_camera xacro file.

File: denso_robot_descriptions/robots/vs050/urdf/denso_robot_macro.xacro (robot description, xacro)
@@ -15,5 +15,5 @@
                                           transmission_hw_interface:=hardware_interface/PositionJointInterface
                                           sim:=false
-                                          basic_camera:=false
+                                          gz_cam:=false
                                           ip_address
                                           send_format
@@ -44,7 +44,7 @@
   <!-- For other tools, modify the filename parameter to the path of your tool's xacro file. -->
   <!-- The line with tag xacro:tool passes the parameters defined in your tool's xacro file -->
-  <!-- (see basic_camera.xacro as an example implementation) -->
-  <xacro:if value="$(arg basic_camera)">
-    <xacro:include filename="$(find denso_robot_gazebo)/sensors/basic_camera/urdf/basic_camera.xacro" />
+  <!-- (see gz_cam.xacro as an example implementation) -->
+  <xacro:if value="$(arg gz_cam)">
+    <xacro:include filename="$(find denso_robot_gazebo)/sensors/gz_cam/urdf/gz_cam.xacro" />
   </xacro:if>
   <!-- ros2 control instance -->
@@ -75,6 +75,6 @@
     <xacro:insert_block name="origin" />
   </xacro:denso_robot_arm_kinematics>
-  <xacro:if value="$(arg basic_camera)">
-    <xacro:basic_camera namespace="${namespace}" end_effector="J6" />
+  <xacro:if value="$(arg gz_cam)">
+    <xacro:gz_cam namespace="${namespace}" end_effector="J6" />
   </xacro:if>
   </xacro:macro>

File: denso_robot_descriptions/urdf/denso_robot.urdf.xacro (robot description, xacro)
@@ -11,5 +11,5 @@
   <xacro:arg name="verbose" default="false" />
   <xacro:arg name="sim" default="false" />
-  <xacro:arg name="basic_camera" default="false" />
+  <xacro:arg name="gz_cam" default="false" />
   <xacro:arg name="ip_address" default="192.168.0.1" />
   <xacro:arg name="send_format" default="288" />
@@ -25,5 +25,5 @@
                      transmission_hw_interface="$(arg transmission_hw_interface)"
                      sim="$(arg sim)"
-                     basic_camera="$(arg basic_camera)"
+                     gz_cam="$(arg gz_cam)"
                      ip_address="$(arg ip_address)"
                      verbose="$(arg verbose)"

File: denso_robot_descriptions/urdf/dual_denso_robot.urdf.xacro (robot description, xacro)
@@ -10,5 +10,5 @@
    <xacro:arg name="verbose" default="false" />
    <xacro:arg name="sim" default="false" />
-   <xacro:arg name="basic_camera" default="false" />
+   <xacro:arg name="gz_cam" default="false" />
    <xacro:arg name="left_ip_address" default="192.168.0.1" />
    <xacro:arg name="right_ip_address" default="192.168.0.2" />
@@ -28,5 +28,5 @@
      transmission_hw_interface="$(arg transmission_hw_interface)"
      sim="$(arg sim)"
-     basic_camera="$(arg basic_camera)"
+     gz_cam="$(arg gz_cam)"
      ip_address="$(arg left_ip_address)"
      verbose="$(arg verbose)"
@@ -42,5 +42,5 @@
      transmission_hw_interface="$(arg transmission_hw_interface)"
      sim="$(arg sim)"
-     basic_camera="$(arg basic_camera)"
+     gz_cam="$(arg gz_cam)"
      ip_address="$(arg right_ip_address)"
      verbose="$(arg verbose)"

File: denso_robot_gazebo/sensors/gz_cam/urdf/gz_cam.xacro (robot description, xacro)
@@ -2,8 +2,8 @@
 <robot xmlns:xacro="http://www.ros.org/wiki/xacro">
     <!-- here you define the parameters you want your xacro file to receive. -->
-    <xacro:macro name="basic_camera" params="namespace end_effector">
+    <xacro:macro name="gz_cam" params="namespace end_effector">
     <!-- if your tool has meshes, define the path to it in geometry tag. -->
     <!-- see the vs050 robot urdf implementation as an example. -->
-    <link name="${namespace}basic_camera_link">
+    <link name="${namespace}gz_cam_link">
 		<inertial>
 			<mass value="1"/>
@@ -21,12 +21,12 @@
 		</visual>
 	</link>
-	<joint name="${namespace}basic_camera_joint" type="fixed">
+	<joint name="${namespace}gz_cam_joint" type="fixed">
         <!-- here you define where your tool will connect. In this case, it's at joint 6. -->
 		<parent link="${namespace}${end_effector}"/>
-		<child link="${namespace}basic_camera_link"/>
+		<child link="${namespace}gz_cam_link"/>
 		<origin rpy="0 ${radians(-90)} 0" xyz="0 0 0.01"/>
 	</joint>
-    <gazebo reference="${namespace}basic_camera_link">
-      <sensor name="${namespace}basic_camera" type="camera">
+    <gazebo reference="${namespace}gz_cam_link">
+      <sensor name="${namespace}gz_cam" type="camera">
         <camera>
           <horizontal_fov>1.047</horizontal_fov>
@@ -43,5 +43,5 @@
         <update_rate>30</update_rate>
         <visualize>true</visualize>
-        <topic>${namespace}basic_camera</topic>
+        <topic>${namespace}gz_cam</topic>
       </sensor>
     </gazebo>

Commit message: refactor(urdf): attach gz_cam to flange link
- Update the `gz_cam.xacro` macro to mount the camera directly to the `${namespace}flange` link instead of dynamically passing the last joint.
- Remove the now redundant `end_effector` parameter from the camera macro definition and its instantiation in `denso_robot_macro.xacro`.
- This aligns the sensor attachment with standard ROS architecture practices.

File: denso_robot_descriptions/robots/vs050/urdf/denso_robot_macro.xacro (robot description, xacro)
@@ -76,5 +76,5 @@
   </xacro:denso_robot_arm_kinematics>
   <xacro:if value="$(arg gz_cam)">
-    <xacro:gz_cam namespace="${namespace}" end_effector="J6" />
+    <xacro:gz_cam namespace="${namespace}" />
   </xacro:if>
   </xacro:macro>

File: denso_robot_gazebo/sensors/gz_cam/urdf/gz_cam.xacro (robot description, xacro)
@@ -2,5 +2,5 @@
 <robot xmlns:xacro="http://www.ros.org/wiki/xacro">
     <!-- here you define the parameters you want your xacro file to receive. -->
-    <xacro:macro name="gz_cam" params="namespace end_effector">
+    <xacro:macro name="gz_cam" params="namespace">
     <!-- if your tool has meshes, define the path to it in geometry tag. -->
     <!-- see the vs050 robot urdf implementation as an example. -->
@@ -23,5 +23,5 @@
 	<joint name="${namespace}gz_cam_joint" type="fixed">
         <!-- here you define where your tool will connect. In this case, it's at joint 6. -->
-		<parent link="${namespace}${end_effector}"/>
+		<parent link="${namespace}flange"/>
 		<child link="${namespace}gz_cam_link"/>
 		<origin rpy="0 ${radians(-90)} 0" xyz="0 0 0.01"/>
