Commit message: fix: origin of vs050 joints

File: denso_robot_descriptions/robots/vs050/urdf/denso_robot_kinematics.xacro (robot description, xacro)
@@ -102,5 +102,5 @@
 			<parent link="$(arg namespace)J2"/>
 			<child link="$(arg namespace)J3"/>
-			<origin rpy="0.000000 0.000000 0.000000" xyz="0.000000 0.000000 0.305000"/>
+			<origin rpy="0.000000 0.000000 0.000000" xyz="0.000000 0.000000 0.250000"/>
 			<axis xyz="-0.000000 1.000000 -0.000000"/>
 			<limit effort="1" lower="-2.18166156499291" upper="2.70526034059121" velocity="2.71540943019156"/>
@@ -129,5 +129,5 @@
 			<parent link="$(arg namespace)J3"/>
 			<child link="$(arg namespace)J4"/>
-			<origin rpy="0.000000 0.000000 0.000000" xyz="-0.010000 0.000000 0.164500"/>
+			<origin rpy="0.000000 0.000000 0.000000" xyz="-0.010000 0.000000 0.119500"/>
 			<axis xyz="-0.000000 -0.000000 1.000000"/>
 			<limit effort="1" lower="-4.71238898038469" upper="4.71238898038469" velocity="3.73064127613788"/>

Commit message: fix: adjust effort values in vs050 and vs060 to gazebo fortress

File: denso_robot_descriptions/robots/vs050/urdf/denso_robot_kinematics.xacro (robot description, xacro)
@@ -50,5 +50,5 @@
 			<origin rpy="0.000000 0.000000 0.000000" xyz="0.000000 0.000000 0.181500"/>
 			<axis xyz="-0.000000 -0.000000 1.000000"/>
-			<limit effort="1" lower="-2.96705972839036" upper="2.96705972839036" velocity="3.73064127613788"/>
+			<limit effort="1000" lower="-2.96705972839036" upper="2.96705972839036" velocity="3.73064127613788"/> #effort value is arbitary for make gazebo simulation runs without gravity problems
 			<dynamics damping="0" friction="0"/>
 		</joint>
@@ -77,5 +77,5 @@
 			<origin rpy="0.000000 0.000000 0.000000" xyz="0.000000 0.000000 0.163500"/>
 			<axis xyz="-0.000000 1.000000 -0.000000"/>
-			<limit effort="1" lower="-2.0943951023932" upper="2.0943951023932" velocity="2.48709418409192"/>
+			<limit effort="1000" lower="-2.0943951023932" upper="2.0943951023932" velocity="2.48709418409192"/> #effort value is arbitary for make gazebo simulation runs without gravity problems
 			<dynamics damping="0" friction="0"/>
 		</joint>
@@ -104,5 +104,5 @@
 			<origin rpy="0.000000 0.000000 0.000000" xyz="0.000000 0.000000 0.250000"/>
 			<axis xyz="-0.000000 1.000000 -0.000000"/>
-			<limit effort="1" lower="-2.18166156499291" upper="2.70526034059121" velocity="2.71540943019156"/>
+			<limit effort="1000" lower="-2.18166156499291" upper="2.70526034059121" velocity="2.71540943019156"/> #effort value is arbitary for make gazebo simulation runs without gravity problems
 			<dynamics damping="0" friction="0"/>
 		</joint>
@@ -131,5 +131,5 @@
 			<origin rpy="0.000000 0.000000 0.000000" xyz="-0.010000 0.000000 0.119500"/>
 			<axis xyz="-0.000000 -0.000000 1.000000"/>
-			<limit effort="1" lower="-4.71238898038469" upper="4.71238898038469" velocity="3.73064127613788"/>
+			<limit effort="1000" lower="-4.71238898038469" upper="4.71238898038469" velocity="3.73064127613788"/> #effort value is arbitary for make gazebo simulation runs without gravity problems
 			<dynamics damping="0" friction="0"/>
 		</joint>
@@ -158,5 +158,5 @@
 			<origin rpy="0.000000 0.000000 0.000000" xyz="0.000000 0.000000 0.135500"/>
 			<axis xyz="-0.000000 1.000000 -0.000000"/>
-			<limit effort="1" lower="-2.0943951023932" upper="2.0943951023932" velocity="2.87060410727889"/>
+			<limit effort="1000" lower="-2.0943951023932" upper="2.0943951023932" velocity="2.87060410727889"/> #effort value is arbitary for make gazebo simulation runs without gravity problems
 			<dynamics damping="0" friction="0"/>
 		</joint>
@@ -185,5 +185,5 @@
 			<origin rpy="0.000000 0.000000 0.000000" xyz="0.000000 0.000000 0.070000"/>
 			<axis xyz="-0.000000 -0.000000 1.000000"/>
-			<limit effort="1" lower="-6.28318530717959" upper="6.28318530717959" velocity="5.96902604182061"/>
+			<limit effort="1000" lower="-6.28318530717959" upper="6.28318530717959" velocity="5.96902604182061"/> #effort value is arbitary for make gazebo simulation runs without gravity problems
 			<dynamics damping="0" friction="0"/>
 		</joint>

File: denso_robot_descriptions/robots/vs060/urdf/denso_robot_kinematics.xacro (robot description, xacro)
@@ -50,5 +50,5 @@
 			<origin rpy="0.000000 0.000000 0.000000" xyz="0.000000 0.000000 0.181500"/>
 			<axis xyz="-0.000000 -0.000000 1.000000"/>
-			<limit effort="1" lower="-2.96705972839036" upper="2.96705972839036" velocity="3.73064127613788"/>
+			<limit effort="1000" lower="-2.96705972839036" upper="2.96705972839036" velocity="3.73064127613788"/> #effort value is arbitary for make gazebo simulation runs without gravity problems
 			<dynamics damping="0" friction="0"/>
 		</joint>
@@ -77,5 +77,5 @@
 			<origin rpy="0.000000 0.000000 0.000000" xyz="0.000000 0.000000 0.163500"/>
 			<axis xyz="-0.000000 1.000000 -0.000000"/>
-			<limit effort="1" lower="-2.0943951023932" upper="2.0943951023932" velocity="2.48709418409192"/>
+			<limit effort="1000" lower="-2.0943951023932" upper="2.0943951023932" velocity="2.48709418409192"/> #effort value is arbitary for make gazebo simulation runs without gravity problems
 			<dynamics damping="0" friction="0"/>
 		</joint>
@@ -104,5 +104,5 @@
 			<origin rpy="0.000000 0.000000 0.000000" xyz="0.000000 0.000000 0.305000"/>
 			<axis xyz="-0.000000 1.000000 -0.000000"/>
-			<limit effort="1" lower="-2.18166156499291" upper="2.70526034059121" velocity="2.71540943019156"/>
+			<limit effort="1000" lower="-2.18166156499291" upper="2.70526034059121" velocity="2.71540943019156"/> #effort value is arbitary for make gazebo simulation runs without gravity problems
 			<dynamics damping="0" friction="0"/>
 		</joint>
@@ -131,5 +131,5 @@
 			<origin rpy="0.000000 0.000000 0.000000" xyz="-0.010000 0.000000 0.164500"/>
 			<axis xyz="-0.000000 -0.000000 1.000000"/>
-			<limit effort="1" lower="-4.71238898038469" upper="4.71238898038469" velocity="3.73064127613788"/>
+			<limit effort="1000" lower="-4.71238898038469" upper="4.71238898038469" velocity="3.73064127613788"/> #effort value is arbitary for make gazebo simulation runs without gravity problems
 			<dynamics damping="0" friction="0"/>
 		</joint>
@@ -158,5 +158,5 @@
 			<origin rpy="0.000000 0.000000 0.000000" xyz="0.000000 0.000000 0.135500"/>
 			<axis xyz="-0.000000 1.000000 -0.000000"/>
-			<limit effort="1" lower="-2.0943951023932" upper="2.0943951023932" velocity="2.87060410727889"/>
+			<limit effort="1000" lower="-2.0943951023932" upper="2.0943951023932" velocity="2.87060410727889"/> #effort value is arbitary for make gazebo simulation runs without gravity problems
 			<dynamics damping="0" friction="0"/>
 		</joint>
@@ -185,5 +185,5 @@
 			<origin rpy="0.000000 0.000000 0.000000" xyz="0.000000 0.000000 0.070000"/>
 			<axis xyz="-0.000000 -0.000000 1.000000"/>
-			<limit effort="1" lower="-6.28318530717959" upper="6.28318530717959" velocity="5.96902604182061"/>
+			<limit effort="1000" lower="-6.28318530717959" upper="6.28318530717959" velocity="5.96902604182061"/> #effort value is arbitary for make gazebo simulation runs without gravity problems
 			<dynamics damping="0" friction="0"/>
 		</joint>

Commit message: fix: comments syntax wrong

File: denso_robot_descriptions/robots/vs050/urdf/denso_robot_kinematics.xacro (robot description, xacro)
@@ -50,5 +50,5 @@
 			<origin rpy="0.000000 0.000000 0.000000" xyz="0.000000 0.000000 0.181500"/>
 			<axis xyz="-0.000000 -0.000000 1.000000"/>
-			<limit effort="1000" lower="-2.96705972839036" upper="2.96705972839036" velocity="3.73064127613788"/> #effort value is arbitary for make gazebo simulation runs without gravity problems
+			<limit effort="1000" lower="-2.96705972839036" upper="2.96705972839036" velocity="3.73064127613788"/> <!-- effort value is arbitary for make gazebo simulation runs without gravity problems -->
 			<dynamics damping="0" friction="0"/>
 		</joint>
@@ -77,5 +77,5 @@
 			<origin rpy="0.000000 0.000000 0.000000" xyz="0.000000 0.000000 0.163500"/>
 			<axis xyz="-0.000000 1.000000 -0.000000"/>
-			<limit effort="1000" lower="-2.0943951023932" upper="2.0943951023932" velocity="2.48709418409192"/> #effort value is arbitary for make gazebo simulation runs without gravity problems
+			<limit effort="1000" lower="-2.0943951023932" upper="2.0943951023932" velocity="2.48709418409192"/> <!-- effort value is arbitary for make gazebo simulation runs without gravity problems -->
 			<dynamics damping="0" friction="0"/>
 		</joint>
@@ -104,5 +104,5 @@
 			<origin rpy="0.000000 0.000000 0.000000" xyz="0.000000 0.000000 0.250000"/>
 			<axis xyz="-0.000000 1.000000 -0.000000"/>
-			<limit effort="1000" lower="-2.18166156499291" upper="2.70526034059121" velocity="2.71540943019156"/> #effort value is arbitary for make gazebo simulation runs without gravity problems
+			<limit effort="1000" lower="-2.18166156499291" upper="2.70526034059121" velocity="2.71540943019156"/> <!-- effort value is arbitary for make gazebo simulation runs without gravity problems -->
 			<dynamics damping="0" friction="0"/>
 		</joint>
@@ -131,5 +131,5 @@
 			<origin rpy="0.000000 0.000000 0.000000" xyz="-0.010000 0.000000 0.119500"/>
 			<axis xyz="-0.000000 -0.000000 1.000000"/>
-			<limit effort="1000" lower="-4.71238898038469" upper="4.71238898038469" velocity="3.73064127613788"/> #effort value is arbitary for make gazebo simulation runs without gravity problems
+			<limit effort="1000" lower="-4.71238898038469" upper="4.71238898038469" velocity="3.73064127613788"/> <!-- effort value is arbitary for make gazebo simulation runs without gravity problems -->
 			<dynamics damping="0" friction="0"/>
 		</joint>
@@ -158,5 +158,5 @@
 			<origin rpy="0.000000 0.000000 0.000000" xyz="0.000000 0.000000 0.135500"/>
 			<axis xyz="-0.000000 1.000000 -0.000000"/>
-			<limit effort="1000" lower="-2.0943951023932" upper="2.0943951023932" velocity="2.87060410727889"/> #effort value is arbitary for make gazebo simulation runs without gravity problems
+			<limit effort="1000" lower="-2.0943951023932" upper="2.0943951023932" velocity="2.87060410727889"/> <!-- effort value is arbitary for make gazebo simulation runs without gravity problems -->
 			<dynamics damping="0" friction="0"/>
 		</joint>
@@ -185,5 +185,5 @@
 			<origin rpy="0.000000 0.000000 0.000000" xyz="0.000000 0.000000 0.070000"/>
 			<axis xyz="-0.000000 -0.000000 1.000000"/>
-			<limit effort="1000" lower="-6.28318530717959" upper="6.28318530717959" velocity="5.96902604182061"/> #effort value is arbitary for make gazebo simulation runs without gravity problems
+			<limit effort="1000" lower="-6.28318530717959" upper="6.28318530717959" velocity="5.96902604182061"/> <!-- effort value is arbitary for make gazebo simulation runs without gravity problems -->
 			<dynamics damping="0" friction="0"/>
 		</joint>

File: denso_robot_descriptions/robots/vs060/urdf/denso_robot_kinematics.xacro (robot description, xacro)
@@ -50,5 +50,5 @@
 			<origin rpy="0.000000 0.000000 0.000000" xyz="0.000000 0.000000 0.181500"/>
 			<axis xyz="-0.000000 -0.000000 1.000000"/>
-			<limit effort="1000" lower="-2.96705972839036" upper="2.96705972839036" velocity="3.73064127613788"/> #effort value is arbitary for make gazebo simulation runs without gravity problems
+			<limit effort="1000" lower="-2.96705972839036" upper="2.96705972839036" velocity="3.73064127613788"/>   <!-- effort value is arbitary for make gazebo simulation runs without gravity problems -->
 			<dynamics damping="0" friction="0"/>
 		</joint>
@@ -77,6 +77,5 @@
 			<origin rpy="0.000000 0.000000 0.000000" xyz="0.000000 0.000000 0.163500"/>
 			<axis xyz="-0.000000 1.000000 -0.000000"/>
-			<limit effort="1000" lower="-2.0943951023932" upper="2.0943951023932" velocity="2.48709418409192"/> #effort value is arbitary for make gazebo simulation runs without gravity problems
-			<dynamics damping="0" friction="0"/>
+			<limit effort="1000" lower="-2.0943951023932" upper="2.0943951023932" velocity="2.48709418409192"/> <!-- effort value is arbitary for make gazebo simulation runs without gravity problems -->
 		</joint>
 		<link name="$(arg namespace)J3">
@@ -104,5 +103,5 @@
 			<origin rpy="0.000000 0.000000 0.000000" xyz="0.000000 0.000000 0.305000"/>
 			<axis xyz="-0.000000 1.000000 -0.000000"/>
-			<limit effort="1000" lower="-2.18166156499291" upper="2.70526034059121" velocity="2.71540943019156"/> #effort value is arbitary for make gazebo simulation runs without gravity problems
+			<limit effort="1000" lower="-2.18166156499291" upper="2.70526034059121" velocity="2.71540943019156"/> <!-- effort value is arbitary for make gazebo simulation runs without gravity problems -->
 			<dynamics damping="0" friction="0"/>
 		</joint>
@@ -131,6 +130,5 @@
 			<origin rpy="0.000000 0.000000 0.000000" xyz="-0.010000 0.000000 0.164500"/>
 			<axis xyz="-0.000000 -0.000000 1.000000"/>
-			<limit effort="1000" lower="-4.71238898038469" upper="4.71238898038469" velocity="3.73064127613788"/> #effort value is arbitary for make gazebo simulation runs without gravity problems
-			<dynamics damping="0" friction="0"/>
+			<limit effort="1000" lower="-4.71238898038469" upper="4.71238898038469" velocity="3.73064127613788"/> <!-- effort value is arbitary for make gazebo simulation runs without gravity problems -->
 		</joint>
 		<link name="$(arg namespace)J5">
@@ -158,5 +156,5 @@
 			<origin rpy="0.000000 0.000000 0.000000" xyz="0.000000 0.000000 0.135500"/>
 			<axis xyz="-0.000000 1.000000 -0.000000"/>
-			<limit effort="1000" lower="-2.0943951023932" upper="2.0943951023932" velocity="2.87060410727889"/> #effort value is arbitary for make gazebo simulation runs without gravity problems
+			<limit effort="1000" lower="-2.0943951023932" upper="2.0943951023932" velocity="2.87060410727889"/> <!-- effort value is arbitary for make gazebo simulation runs without gravity problems -->
 			<dynamics damping="0" friction="0"/>
 		</joint>
@@ -185,5 +183,5 @@
 			<origin rpy="0.000000 0.000000 0.000000" xyz="0.000000 0.000000 0.070000"/>
 			<axis xyz="-0.000000 -0.000000 1.000000"/>
-			<limit effort="1000" lower="-6.28318530717959" upper="6.28318530717959" velocity="5.96902604182061"/> #effort value is arbitary for make gazebo simulation runs without gravity problems
+			<limit effort="1000" lower="-6.28318530717959" upper="6.28318530717959" velocity="5.96902604182061"/> <!-- effort value is arbitary for make gazebo simulation runs without gravity problems -->
 			<dynamics damping="0" friction="0"/>
 		</joint>

Commit message: feat: add camera in vs050

File: denso_robot_descriptions/robots/vs050/urdf/denso_robot_kinematics.xacro (robot description, xacro)
@@ -188,4 +188,25 @@
 			<dynamics damping="0" friction="0"/>
 		</joint>
+		<link name="basic_camera_link">
+			<inertial>
+				<mass value="1"/>
+				<inertia ixx="1" ixy="0" ixz="0" iyy="1" iyz="0" izz="1"/>
+			</inertial>
+			<collision>
+				<geometry>
+					<box size="0.01 0.01 0.01"/>
+				</geometry>
+			</collision>
+				<visual>
+					<geometry>
+						<box size="0.01 0.01 0.01"/>
+					</geometry>
+				</visual>
+		</link>
+		<joint name="basic_camera_joint" type="fixed">
+			<parent link="$(arg namespace)J6"/>
+			<child link="basic_camera_link"/>
+			<origin rpy="0 ${radians(-90)} 0" xyz="0 0 0.01"/>
+		</joint>
 	</xacro:macro>
 </robot>

File: denso_robot_descriptions/robots/vs050/urdf/denso_robot_macro.xacro (robot description, xacro)
@@ -68,4 +68,23 @@
     	</plugin>
   	</gazebo>
+    <gazebo reference="basic_camera_link">
+        <sensor name="basic_camera" type="camera">
+          <camera>
+            <horizontal_fov>1.047</horizontal_fov>
+            <image>
+              <width>320</width>
+              <height>240</height>
+            </image>
+            <clip>
+              <near>0.1</near>
+              <far>100</far>
+            </clip>
+          </camera>
+          <always_on>1</always_on>
+          <update_rate>30</update_rate>
+          <visualize>true</visualize>
+          <topic>basic_camera</topic>
+        </sensor>
+      </gazebo>
   </xacro:macro>
 </robot>

Commit message: feat: add namespace to basic camera

File: denso_robot_descriptions/robots/vs050/urdf/denso_robot_kinematics.xacro (robot description, xacro)
@@ -188,5 +188,5 @@
 			<dynamics damping="0" friction="0"/>
 		</joint>
-		<link name="basic_camera_link">
+		<link name="$(arg namespace)basic_camera_link">
 			<inertial>
 				<mass value="1"/>
@@ -198,13 +198,13 @@
 				</geometry>
 			</collision>
-				<visual>
-					<geometry>
-						<box size="0.01 0.01 0.01"/>
-					</geometry>
-				</visual>
-		</link>
-		<joint name="basic_camera_joint" type="fixed">
+			<visual>
+				<geometry>
+					<box size="0.01 0.01 0.01"/>
+				</geometry>
+			</visual>
+		</link>
+		<joint name="$(arg namespace)basic_camera_joint" type="fixed">
 			<parent link="$(arg namespace)J6"/>
-			<child link="basic_camera_link"/>
+			<child link="$(arg namespace)basic_camera_link"/>
 			<origin rpy="0 ${radians(-90)} 0" xyz="0 0 0.01"/>
 		</joint>

File: denso_robot_descriptions/robots/vs050/urdf/denso_robot_macro.xacro (robot description, xacro)
@@ -68,23 +68,23 @@
     	</plugin>
   	</gazebo>
-    <gazebo reference="basic_camera_link">
-        <sensor name="basic_camera" type="camera">
-          <camera>
-            <horizontal_fov>1.047</horizontal_fov>
-            <image>
-              <width>320</width>
-              <height>240</height>
-            </image>
-            <clip>
-              <near>0.1</near>
-              <far>100</far>
-            </clip>
-          </camera>
-          <always_on>1</always_on>
-          <update_rate>30</update_rate>
-          <visualize>true</visualize>
-          <topic>basic_camera</topic>
-        </sensor>
-      </gazebo>
+    <gazebo reference="$(arg namespace)basic_camera_link">
+      <sensor name="basic_camera" type="camera">
+        <camera>
+          <horizontal_fov>1.047</horizontal_fov>
+          <image>
+            <width>320</width>
+            <height>240</height>
+          </image>
+          <clip>
+            <near>0.1</near>
+            <far>100</far>
+          </clip>
+        </camera>
+        <always_on>1</always_on>
+        <update_rate>30</update_rate>
+        <visualize>true</visualize>
+        <topic>basic_camera</topic>
+      </sensor>
+    </gazebo>
   </xacro:macro>
 </robot>

Commit message: chore: basic_camera modulation

File: denso_robot_descriptions/robots/vs050/urdf/denso_robot_kinematics.xacro (robot description, xacro)
@@ -188,25 +188,4 @@
 			<dynamics damping="0" friction="0"/>
 		</joint>
-		<link name="$(arg namespace)basic_camera_link">
-			<inertial>
-				<mass value="1"/>
-				<inertia ixx="1" ixy="0" ixz="0" iyy="1" iyz="0" izz="1"/>
-			</inertial>
-			<collision>
-				<geometry>
-					<box size="0.01 0.01 0.01"/>
-				</geometry>
-			</collision>
-			<visual>
-				<geometry>
-					<box size="0.01 0.01 0.01"/>
-				</geometry>
-			</visual>
-		</link>
-		<joint name="$(arg namespace)basic_camera_joint" type="fixed">
-			<parent link="$(arg namespace)J6"/>
-			<child link="$(arg namespace)basic_camera_link"/>
-			<origin rpy="0 ${radians(-90)} 0" xyz="0 0 0.01"/>
-		</joint>
 	</xacro:macro>
 </robot>

File: denso_robot_descriptions/robots/vs050/urdf/denso_robot_macro.xacro (robot description, xacro)
@@ -39,4 +39,8 @@
     <!-- ros2 control include -->
     <xacro:include filename="$(find denso_robot_descriptions)/robots/$(arg model)/urdf/denso_robot.ros2_control.xacro" />
+    <!-- For other tools, modify the filename parameter to the path of your tool's xacro file.
+    The line with tag <xacro:tool ... \> passes the parameters defined in your tool's xacro file
+    (see basic_camera.xacro as an example implementation) -->
+    <xacro:include filename="$(find denso_robot_descriptions)/tools/basic_camera/urdf/basic_camera.xacro" />
     <!-- ros2 control instance -->
     <xacro:denso_robot_ros2_control
@@ -63,4 +67,5 @@
     <!-- links -  main serial chain -->
     <xacro:denso_robot_arm_kinematics namespace="$(arg namespace)" model="$(arg model)" />
+    <xacro:tool namespace="$(arg namespace)" />
     <gazebo>
 	    <plugin filename="gz_ros2_control-system" name="gz_ros2_control::GazeboSimROS2ControlPlugin">
@@ -68,23 +73,4 @@
     	</plugin>
   	</gazebo>
-    <gazebo reference="$(arg namespace)basic_camera_link">
-      <sensor name="basic_camera" type="camera">
-        <camera>
-          <horizontal_fov>1.047</horizontal_fov>
-          <image>
-            <width>320</width>
-            <height>240</height>
-          </image>
-          <clip>
-            <near>0.1</near>
-            <far>100</far>
-          </clip>
-        </camera>
-        <always_on>1</always_on>
-        <update_rate>30</update_rate>
-        <visualize>true</visualize>
-        <topic>basic_camera</topic>
-      </sensor>
-    </gazebo>
   </xacro:macro>
 </robot>
