Commit message: refactor(vs060): overhaul MoveIt configurations and URDF kinematics
- Flatten nested `move_group/ros__parameters` structures in the MoveIt configuration YAML files.
- Introduce `flange` and `tool0` dummy links to standardize end-effector attachments.
- Update `denso_robot_joint_limits.xacro` to support velocity command and effort state interfaces.
- Standardize camera arguments to `gz_cam` and fix legacy xacro namespace URLs.

File: denso_robot_descriptions/robots/vs050/urdf/denso_robot_kinematics.xacro (robot description, xacro)
@@ -193,13 +193,13 @@
 		<link name="${namespace}flange"/>
 		<joint name="${namespace}J6-flange" type="fixed">
-		<parent link="${namespace}J6"/>
-		<child link="${namespace}flange"/>
-		<origin rpy="0 0 0" xyz="0 0 0"/>
+      <parent link="${namespace}J6"/>
+      <child link="${namespace}flange"/>
+      <origin rpy="0 0 0" xyz="0 0 0"/>
 		</joint>
 		<link name="${namespace}tool0"/>
 		<joint name="${namespace}J6-tool0" type="fixed">
-		<parent link="${namespace}J6"/>
-		<child link="${namespace}tool0"/>
-		<origin rpy="${radians(pi)} ${radians(-pi/2)} 0" xyz="0 0 0"/>
+      <parent link="${namespace}J6"/>
+      <child link="${namespace}tool0"/>
+      <origin rpy="${radians(pi)} ${radians(-pi/2)} 0" xyz="0 0 0"/>
 		</joint>
 	</xacro:macro>

File: denso_robot_descriptions/robots/vs060/urdf/denso_robot.ros2_control.xacro (robot description, xacro)
@@ -1,19 +1,28 @@
 <?xml version="1.0"?>
 <robot xmlns:xacro="http://www.ros.org/wiki/xacro">
-  <xacro:macro name="denso_robot_ros2_control" params="name namespace
-	robot_name
-    sim:=false fake_sensor_commands:=false
-    ip_address
-    model
-    robot_joints joint_1 joint_2 joint_3 joint_4 joint_5 joint_6
-    arm_group
-    send_format recv_format
-	controller_type
-    verbose
-    initial_positions
-    ">
+  <xacro:macro name="denso_robot_ros2_control"
+               params="name
+                       namespace
+                       robot_name
+                       sim:=false
+                       fake_sensor_commands:=false
+                       ip_address
+                       model
+                       robot_joints
+                       joint_1
+                       joint_2
+                       joint_3
+                       joint_4
+                       joint_5
+                       joint_6
+                       arm_group
+                       send_format
+                       recv_format
+                       controller_type
+                       verbose
+                       initial_positions_file">
     <ros2_control name="${namespace}${name}" type="system">
-	<!-- joint limits include -->
-	<xacro:include filename="$(find denso_robot_descriptions)/robots/$(arg model)/urdf/denso_robot_joint_limits.xacro" />
+	  <!-- joint limits include -->
+	  <xacro:include filename="$(find denso_robot_descriptions)/robots/$(arg model)/urdf/denso_robot_joint_limits.xacro" />
       <hardware>
         <xacro:if value="${sim}">
@@ -23,5 +32,5 @@
           <plugin>denso_robot_control/DensoRobotHW</plugin>
           <param name="ip_address">${ip_address}</param>
-<!-- "robot_name" param must be consistent with the @TYPE_NAME variable of the real robot !!  -->
+          <!-- "robot_name" param must be consistent with the @TYPE_NAME variable of the real robot !!  -->
           <param name="robot_name">${robot_name}</param>
           <param name="node_name">denso_robot_control</param>
@@ -41,5 +50,5 @@
         </xacro:unless>
       </hardware>
-      <xacro:denso_robot_control_limits namespace="${namespace}" initial_positions="${initial_positions}" />
+      <xacro:denso_robot_control_limits namespace="${namespace}" initial_positions_file="${initial_positions_file}" />
     </ros2_control>
   </xacro:macro>

File: denso_robot_descriptions/robots/vs060/urdf/denso_robot_joint_limits.xacro (robot description, xacro)
@@ -1,95 +1,60 @@
 <?xml version='1.0' encoding='UTF-8'?>
 <robot xmlns:xacro="http://www.ros.org/wiki/xacro">
-	<xacro:macro name="denso_robot_control_limits" params="namespace initial_positions">
-		<joint name="${namespace}joint_1">
-			<command_interface name="position">
-				<param name="min">-2.967060</param>
-				<param name="max">2.967060</param>
-			</command_interface>
-			<command_interface name="velocity">
-				<param name="min">0</param>
-				<param name="max">0.392699081698724</param>
-			</command_interface>
-			<state_interface name="position">
-				<param name="initial_value">${initial_positions['joint_1']}</param>
-			</state_interface>
-			<state_interface name="velocity"/>
-			<state_interface name="effort"/>
-		</joint>
-		<joint name="${namespace}joint_2">
-			<command_interface name="position">
-				<param name="min">-2.094395</param>
-				<param name="max">2.094395</param>
-			</command_interface>
-			<command_interface name="velocity">
-				<param name="min">0</param>
-				<param name="max">0.261799387799149</param>
-			</command_interface>
-			<state_interface name="position">
-				<param name="initial_value">${initial_positions['joint_2']}</param>
-			</state_interface>
-			<state_interface name="velocity"/>
-			<state_interface name="effort"/>
-		</joint>
-		<joint name="${namespace}joint_3">
-			<command_interface name="position">
-				<param name="min">-2.181662</param>
-				<param name="max">2.705260</param>
-			</command_interface>
-			<command_interface name="velocity">
-				<param name="min">0</param>
-				<param name="max">0.285832571599111</param>
-			</command_interface>
-			<state_interface name="position">
-				<param name="initial_value">${initial_positions['joint_3']}</param>
-			</state_interface>
-			<state_interface name="velocity"/>
-			<state_interface name="effort"/>
-		</joint>
-		<joint name="${namespace}joint_4">
-			<command_interface name="position">
-				<param name="min">-4.712389</param>
-				<param name="max">4.712389</param>
-			</command_interface>
-			<command_interface name="velocity">
-				<param name="min">0</param>
-				<param name="max">0.392699081698724</param>
-			</command_interface>
-			<state_interface name="position">
-				<param name="initial_value">${initial_positions['joint_4']}</param>
-			</state_interface>
-			<state_interface name="velocity"/>
-			<state_interface name="effort"/>
-		</joint>
-		<joint name="${namespace}joint_5">
-			<command_interface name="position">
-				<param name="min">-2.094395</param>
-				<param name="max">2.094395</param>
-			</command_interface>
-			<command_interface name="velocity">
-				<param name="min">0</param>
-				<param name="max">0.302168853397778</param>
-			</command_interface>
-			<state_interface name="position">
-				<param name="initial_value">${initial_positions['joint_5']}</param>
-			</state_interface>
-			<state_interface name="velocity"/>
-			<state_interface name="effort"/>
-		</joint>
-		<joint name="${namespace}joint_6">
-			<command_interface name="position">
-				<param name="min">-6.283185</param>
-				<param name="max">6.283185</param>
-			</command_interface>
-			<command_interface name="velocity">
-				<param name="min">0</param>
-				<param name="max">0.628318530717959</param>
-			</command_interface>
-			<state_interface name="position">
-				<param name="initial_value">${initial_positions['joint_6']}</param>
-			</state_interface>
-			<state_interface name="velocity"/>
-			<state_interface name="effort"/>
-		</joint>
+	<xacro:macro name="denso_robot_control_limits" params="namespace initial_positions_file">
+    <xacro:property name="initial_positions" value="${xacro.load_yaml(initial_positions_file)['initial_positions']}" />
+	  <joint name="${namespace}joint_1">
+      <command_interface name="position" />
+      <command_interface name="velocity" />
+      <state_interface name="position">
+        <param name="initial_value">${initial_positions['joint_1']}</param>
+      </state_interface>
+      <state_interface name="velocity" />
+      <state_interface name="effort"/>
+    </joint>
+    <joint name="${namespace}joint_2">
+      <command_interface name="position" />
+      <command_interface name="velocity" />
+      <state_interface name="position">
+        <param name="initial_value">${initial_positions['joint_2']}</param>
+      </state_interface>
+      <state_interface name="velocity" />
+      <state_interface name="effort"/>
+    </joint>
+    <joint name="${namespace}joint_3">
+      <command_interface name="position" />
+      <command_interface name="velocity" />
+      <state_interface name="position">
+        <param name="initial_value">${initial_positions['joint_3']}</param>
+      </state_interface>
+      <state_interface name="velocity" />
+      <state_interface name="effort"/>
+    </joint>
+    <joint name="${namespace}joint_4">
+      <command_interface name="position" />
+      <command_interface name="velocity" />
+      <state_interface name="position">
+        <param name="initial_value">${initial_positions['joint_4']}</param>
+      </state_interface>
+      <state_interface name="velocity" />
+      <state_interface name="effort"/>
+    </joint>
+    <joint name="${namespace}joint_5">
+      <command_interface name="position" />
+      <command_interface name="velocity" />
+      <state_interface name="position">
+        <param name="initial_value">${initial_positions['joint_5']}</param>
+      </state_interface>
+      <state_interface name="velocity" />
+      <state_interface name="effort"/>
+    </joint>
+    <joint name="${namespace}joint_6">
+      <command_interface name="position" />
+      <command_interface name="velocity" />
+      <state_interface name="position">
+        <param name="initial_value">${initial_positions['joint_6']}</param>
+      </state_interface>
+      <state_interface name="velocity" />
+      <state_interface name="effort"/>
+    </joint>
 	</xacro:macro>
 </robot>
