Commit message: refactor(vs060): overhaul MoveIt configurations and URDF kinematics
- Flatten nested `move_group/ros__parameters` structures in the MoveIt configuration YAML files.
- Introduce `flange` and `tool0` dummy links to standardize end-effector attachments.
- Update `denso_robot_joint_limits.xacro` to support velocity command and effort state interfaces.
- Standardize camera arguments to `gz_cam` and fix legacy xacro namespace URLs.

File: denso_robot_descriptions/robots/vs060/urdf/denso_robot_kinematics.xacro (robot description, xacro)
@@ -2,187 +2,204 @@
 <robot xmlns:xacro="http://www.ros.org/wiki/xacro">
 	<xacro:macro name="denso_robot_arm_kinematics" params="namespace model parent *origin">
-		<joint name="${namespace}joint_w" type="fixed">
+    <joint name="${namespace}joint_w" type="fixed">
 			<xacro:insert_block name="origin" />
-			<parent link="${parent}"/>
-			<child link="${namespace}base_link"/>
-		</joint>
-		<link name="${namespace}base_link">
-			<visual>
-				<origin rpy="0 0 0" xyz="0 0 0"/>
-				<geometry>
-					<mesh filename="file:///$(find denso_robot_descriptions)/robots/$(arg model)/meshes/base_link.dae" scale="1 1 1"/>
-				</geometry>
-			</visual>
-			<collision>
-				<origin rpy="0 0 0" xyz="0 0 0"/>
-				<geometry>
-					<mesh filename="file:///$(find denso_robot_descriptions)/robots/$(arg model)/meshes/base_link.dae" scale="1 1 1"/>
-				</geometry>
-			</collision>
-			<inertial>
-				<mass value="1"/>
-				<origin rpy="0.000000 0.000000 0.000000" xyz="0.000000 0.000000 0.000000"/>
-				<inertia ixx="1" ixy="0" ixz="0" iyy="1" iyz="0" izz="1"/>
-			</inertial>
-		</link>
-		<link name="${namespace}J1">
-			<visual>
-				<origin rpy="0 0 0" xyz="0 0 0"/>
-				<geometry>
-					<mesh filename="file:///$(find denso_robot_descriptions)/robots/$(arg model)/meshes/J1.dae" scale="1 1 1"/>
-				</geometry>
-			</visual>
-			<collision>
-				<origin rpy="0 0 0" xyz="0 0 0"/>
-				<geometry>
-					<mesh filename="file:///$(find denso_robot_descriptions)/robots/$(arg model)/meshes/J1.dae" scale="1 1 1"/>
-				</geometry>
-			</collision>
-			<inertial>
-				<mass value="1"/>
-				<origin rpy="0.000000 0.000000 0.000000" xyz="0.000000 0.000000 0.000000"/>
-				<inertia ixx="1" ixy="0" ixz="0" iyy="1" iyz="0" izz="1"/>
+			<parent link="${parent}" />
+			<child link="${namespace}base_link" />
+		</joint>
+    <link name="${namespace}base_link">
+			<visual>
+				<origin rpy="0 0 0" xyz="0 0 0" />
+				<geometry>
+					<mesh filename="file:///$(find denso_robot_descriptions)/robots/$(arg model)/meshes/base_link.dae" scale="1 1 1" />
+				</geometry>
+			</visual>
+			<collision>
+				<origin rpy="0 0 0" xyz="0 0 0" />
+				<geometry>
+					<mesh filename="file:///$(find denso_robot_descriptions)/robots/$(arg model)/meshes/base_link.dae" scale="1 1 1" />
+				</geometry>
+			</collision>
+			<inertial>
+				<mass value="1" />
+				<origin rpy="0.000000 0.000000 0.000000" xyz="0.000000 0.000000 0.000000" />
+				<inertia ixx="1" ixy="0" ixz="0" iyy="1" iyz="0" izz="1" />
+			</inertial>
+		</link>
+    <link name="${namespace}J1">
+			<visual>
+				<origin rpy="0 0 0" xyz="0 0 0" />
+				<geometry>
+					<mesh filename="file:///$(find denso_robot_descriptions)/robots/$(arg model)/meshes/J1.dae" scale="1 1 1" />
+				</geometry>
+			</visual>
+			<collision>
+				<origin rpy="0 0 0" xyz="0 0 0" />
+				<geometry>
+					<mesh filename="file:///$(find denso_robot_descriptions)/robots/$(arg model)/meshes/J1.dae" scale="1 1 1" />
+				</geometry>
+			</collision>
+			<inertial>
+				<mass value="1" />
+				<origin rpy="0.000000 0.000000 0.000000" xyz="0.000000 0.000000 0.000000" />
+				<inertia ixx="1" ixy="0" ixz="0" iyy="1" iyz="0" izz="1" />
 			</inertial>
 		</link>
 		<joint name="${namespace}joint_1" type="revolute">
-			<parent link="${namespace}base_link"/>
-			<child link="${namespace}J1"/>
-			<origin rpy="0.000000 0.000000 0.000000" xyz="0.000000 0.000000 0.181500"/>
-			<axis xyz="-0.000000 -0.000000 1.000000"/>
-			<limit effort="1000" lower="-2.96705972839036" upper="2.96705972839036" velocity="3.73064127613788"/>   <!-- effort value is arbitary for make gazebo simulation runs without gravity problems -->
-			<dynamics damping="0" friction="0"/>
-		</joint>
-		<link name="${namespace}J2">
-			<visual>
-				<origin rpy="0 0 0" xyz="0 0 0"/>
-				<geometry>
-					<mesh filename="file:///$(find denso_robot_descriptions)/robots/$(arg model)/meshes/J2.dae" scale="1 1 1"/>
-				</geometry>
-			</visual>
-			<collision>
-				<origin rpy="0 0 0" xyz="0 0 0"/>
-				<geometry>
-					<mesh filename="file:///$(find denso_robot_descriptions)/robots/$(arg model)/meshes/J2.dae" scale="1 1 1"/>
-				</geometry>
-			</collision>
-			<inertial>
-				<mass value="1"/>
-				<origin rpy="0.000000 0.000000 0.000000" xyz="0.000000 0.000000 0.000000"/>
-				<inertia ixx="1" ixy="0" ixz="0" iyy="1" iyz="0" izz="1"/>
+			<parent link="${namespace}base_link" />
+			<child link="${namespace}J1" />
+			<origin rpy="0.000000 0.000000 0.000000" xyz="0.000000 0.000000 0.181500" />
+			<axis xyz="-0.000000 -0.000000 1.000000" />
+      <!-- effort value is arbitary for make gazebo simulation runs without gravity problems -->
+			<limit effort="1000" lower="${radians(-170)}" upper="${radians(170)}" velocity="${radians(425)}"  />
+			<dynamics damping="0" friction="0" />
+		</joint>
+    <link name="${namespace}J2">
+			<visual>
+				<origin rpy="0 0 0" xyz="0 0 0" />
+				<geometry>
+					<mesh filename="file:///$(find denso_robot_descriptions)/robots/$(arg model)/meshes/J2.dae" scale="1 1 1" />
+				</geometry>
+			</visual>
+			<collision>
+				<origin rpy="0 0 0" xyz="0 0 0" />
+				<geometry>
+					<mesh filename="file:///$(find denso_robot_descriptions)/robots/$(arg model)/meshes/J2.dae" scale="1 1 1" />
+				</geometry>
+			</collision>
+			<inertial>
+				<mass value="1" />
+				<origin rpy="0.000000 0.000000 0.000000" xyz="0.000000 0.000000 0.000000" />
+				<inertia ixx="1" ixy="0" ixz="0" iyy="1" iyz="0" izz="1" />
 			</inertial>
 		</link>
 		<joint name="${namespace}joint_2" type="revolute">
-			<parent link="${namespace}J1"/>
-			<child link="${namespace}J2"/>
-			<origin rpy="0.000000 0.000000 0.000000" xyz="0.000000 0.000000 0.163500"/>
-			<axis xyz="-0.000000 1.000000 -0.000000"/>
-			<limit effort="1000" lower="-2.0943951023932" upper="2.0943951023932" velocity="2.48709418409192"/> <!-- effort value is arbitary for make gazebo simulation runs without gravity problems -->
-		</joint>
+			<parent link="${namespace}J1" />
+			<child link="${namespace}J2" />
+			<origin rpy="0.000000 0.000000 0.000000" xyz="0.000000 0.000000 0.163500" />
+			<axis xyz="-0.000000 1.000000 -0.000000" />
+			<!-- effort value is arbitary for make gazebo simulation runs without gravity problems -->
+			<limit effort="1000" lower="${radians(-120)}" upper="${radians(120)}" velocity="${radians(283.33)}" />
+      <dynamics damping="0" friction="0" />
+    </joint>
 		<link name="${namespace}J3">
 			<visual>
-				<origin rpy="0 0 0" xyz="0 0 0"/>
-				<geometry>
-					<mesh filename="file:///$(find denso_robot_descriptions)/robots/$(arg model)/meshes/J3.dae" scale="1 1 1"/>
-				</geometry>
-			</visual>
-			<collision>
-				<origin rpy="0 0 0" xyz="0 0 0"/>
-				<geometry>
-					<mesh filename="file:///$(find denso_robot_descriptions)/robots/$(arg model)/meshes/J3.dae" scale="1 1 1"/>
-				</geometry>
-			</collision>
-			<inertial>
-				<mass value="1"/>
-				<origin rpy="0.000000 0.000000 0.000000" xyz="0.000000 0.000000 0.000000"/>
-				<inertia ixx="1" ixy="0" ixz="0" iyy="1" iyz="0" izz="1"/>
+				<origin rpy="0 0 0" xyz="0 0 0" />
+				<geometry>
+					<mesh filename="file:///$(find denso_robot_descriptions)/robots/$(arg model)/meshes/J3.dae" scale="1 1 1" />
+				</geometry>
+			</visual>
+			<collision>
+				<origin rpy="0 0 0" xyz="0 0 0" />
+				<geometry>
+					<mesh filename="file:///$(find denso_robot_descriptions)/robots/$(arg model)/meshes/J3.dae" scale="1 1 1" />
+				</geometry>
+			</collision>
+			<inertial>
+				<mass value="1" />
+				<origin rpy="0.000000 0.000000 0.000000" xyz="0.000000 0.000000 0.000000" />
+				<inertia ixx="1" ixy="0" ixz="0" iyy="1" iyz="0" izz="1" />
 			</inertial>
 		</link>
 		<joint name="${namespace}joint_3" type="revolute">
-			<parent link="${namespace}J2"/>
-			<child link="${namespace}J3"/>
-			<origin rpy="0.000000 0.000000 0.000000" xyz="0.000000 0.000000 0.305000"/>
-			<axis xyz="-0.000000 1.000000 -0.000000"/>
-			<limit effort="1000" lower="-2.18166156499291" upper="2.70526034059121" velocity="2.71540943019156"/> <!-- effort value is arbitary for make gazebo simulation runs without gravity problems -->
-			<dynamics damping="0" friction="0"/>
+			<parent link="${namespace}J2" />
+			<child link="${namespace}J3" />
+			<origin rpy="0.000000 0.000000 0.000000" xyz="0.000000 0.000000 0.305000" />
+			<axis xyz="-0.000000 1.000000 -0.000000" />
+			<!-- effort value is arbitary for make gazebo simulation runs without gravity problems -->
+			<limit effort="1000" lower="${radians(-25)}" upper="${radians(155)}" velocity="${radians(309.35)}" />
+			<dynamics damping="0" friction="0" />
 		</joint>
 		<link name="${namespace}J4">
 			<visual>
-				<origin rpy="0 0 0" xyz="0 0 0"/>
-				<geometry>
-					<mesh filename="file:///$(find denso_robot_descriptions)/robots/$(arg model)/meshes/J4.dae" scale="1 1 1"/>
-				</geometry>
-			</visual>
-			<collision>
-				<origin rpy="0 0 0" xyz="0 0 0"/>
-				<geometry>
-					<mesh filename="file:///$(find denso_robot_descriptions)/robots/$(arg model)/meshes/J4.dae" scale="1 1 1"/>
-				</geometry>
-			</collision>
-			<inertial>
-				<mass value="1"/>
-				<origin rpy="0.000000 0.000000 0.000000" xyz="0.000000 0.000000 0.000000"/>
-				<inertia ixx="1" ixy="0" ixz="0" iyy="1" iyz="0" izz="1"/>
+				<origin rpy="0 0 0" xyz="0 0 0" />
+				<geometry>
+					<mesh filename="file:///$(find denso_robot_descriptions)/robots/$(arg model)/meshes/J4.dae" scale="1 1 1" />
+				</geometry>
+			</visual>
+			<collision>
+				<origin rpy="0 0 0" xyz="0 0 0" />
+				<geometry>
+					<mesh filename="file:///$(find denso_robot_descriptions)/robots/$(arg model)/meshes/J4.dae" scale="1 1 1" />
+				</geometry>
+			</collision>
+			<inertial>
+				<mass value="1" />
+				<origin rpy="0.000000 0.000000 0.000000" xyz="0.000000 0.000000 0.000000" />
+				<inertia ixx="1" ixy="0" ixz="0" iyy="1" iyz="0" izz="1" />
 			</inertial>
 		</link>
 		<joint name="${namespace}joint_4" type="revolute">
-			<parent link="${namespace}J3"/>
-			<child link="${namespace}J4"/>
-			<origin rpy="0.000000 0.000000 0.000000" xyz="-0.010000 0.000000 0.164500"/>
-			<axis xyz="-0.000000 -0.000000 1.000000"/>
-			<limit effort="1000" lower="-4.71238898038469" upper="4.71238898038469" velocity="3.73064127613788"/> <!-- effort value is arbitary for make gazebo simulation runs without gravity problems -->
+			<parent link="${namespace}J3" />
+			<child link="${namespace}J4" />
+			<origin rpy="0.000000 0.000000 0.000000" xyz="-0.010000 0.000000 0.164500" />
+			<axis xyz="-0.000000 -0.000000 1.000000" />
+			<limit effort="6.66" lower="${radians(-270)}" upper="${radians(270)}" velocity="${radians(425)}" />
+      <dynamics damping="0" friction="0" />
 		</joint>
 		<link name="${namespace}J5">
 			<visual>
-				<origin rpy="0 0 0" xyz="0 0 0"/>
-				<geometry>
-					<mesh filename="file:///$(find denso_robot_descriptions)/robots/$(arg model)/meshes/J5.dae" scale="1 1 1"/>
-				</geometry>
-			</visual>
-			<collision>
-				<origin rpy="0 0 0" xyz="0 0 0"/>
-				<geometry>
-					<mesh filename="file:///$(find denso_robot_descriptions)/robots/$(arg model)/meshes/J5.dae" scale="1 1 1"/>
-				</geometry>
-			</collision>
-			<inertial>
-				<mass value="1"/>
-				<origin rpy="0.000000 0.000000 0.000000" xyz="0.000000 0.000000 0.000000"/>
-				<inertia ixx="1" ixy="0" ixz="0" iyy="1" iyz="0" izz="1"/>
+				<origin rpy="0 0 0" xyz="0 0 0" />
+				<geometry>
+					<mesh filename="file:///$(find denso_robot_descriptions)/robots/$(arg model)/meshes/J5.dae" scale="1 1 1" />
+				</geometry>
+			</visual>
+			<collision>
+				<origin rpy="0 0 0" xyz="0 0 0" />
+				<geometry>
+					<mesh filename="file:///$(find denso_robot_descriptions)/robots/$(arg model)/meshes/J5.dae" scale="1 1 1" />
+				</geometry>
+			</collision>
+			<inertial>
+				<mass value="1" />
+				<origin rpy="0.000000 0.000000 0.000000" xyz="0.000000 0.000000 0.000000" />
+				<inertia ixx="1" ixy="0" ixz="0" iyy="1" iyz="0" izz="1" />
 			</inertial>
 		</link>
 		<joint name="${namespace}joint_5" type="revolute">
-			<parent link="${namespace}J4"/>
-			<child link="${namespace}J5"/>
-			<origin rpy="0.000000 0.000000 0.000000" xyz="0.000000 0.000000 0.135500"/>
-			<axis xyz="-0.000000 1.000000 -0.000000"/>
-			<limit effort="1000" lower="-2.0943951023932" upper="2.0943951023932" velocity="2.87060410727889"/> <!-- effort value is arbitary for make gazebo simulation runs without gravity problems -->
-			<dynamics damping="0" friction="0"/>
+			<parent link="${namespace}J4" />
+			<child link="${namespace}J5" />
+			<origin rpy="0.000000 0.000000 0.000000" xyz="0.000000 0.000000 0.135500" />
+			<axis xyz="-0.000000 1.000000 -0.000000" />
+			<limit effort="6.66" lower="${radians(-120)}" upper="${radians(120)}" velocity="${radians(327.01)}" />
+			<dynamics damping="0" friction="0" />
 		</joint>
 		<link name="${namespace}J6">
 			<visual>
-				<origin rpy="0 0 0" xyz="0 0 0"/>
-				<geometry>
-					<mesh filename="file:///$(find denso_robot_descriptions)/robots/$(arg model)/meshes/J6.dae" scale="1 1 1"/>
-				</geometry>
-			</visual>
-			<collision>
-				<origin rpy="0 0 0" xyz="0 0 0"/>
-				<geometry>
-					<mesh filename="file:///$(find denso_robot_descriptions)/robots/$(arg model)/meshes/J6.dae" scale="1 1 1"/>
-				</geometry>
-			</collision>
-			<inertial>
-				<mass value="1"/>
-				<origin rpy="0.000000 0.000000 0.000000" xyz="0.000000 0.000000 0.000000"/>
-				<inertia ixx="1" ixy="0" ixz="0" iyy="1" iyz="0" izz="1"/>
+				<origin rpy="0 0 0" xyz="0 0 0" />
+				<geometry>
+					<mesh filename="file:///$(find denso_robot_descriptions)/robots/$(arg model)/meshes/J6.dae" scale="1 1 1" />
+				</geometry>
+			</visual>
+			<collision>
+				<origin rpy="0 0 0" xyz="0 0 0" />
+				<geometry>
+					<mesh filename="file:///$(find denso_robot_descriptions)/robots/$(arg model)/meshes/J6.dae" scale="1 1 1" />
+				</geometry>
+			</collision>
+			<inertial>
+				<mass value="1" />
+				<origin rpy="0.000000 0.000000 0.000000" xyz="0.000000 0.000000 0.000000" />
+				<inertia ixx="1" ixy="0" ixz="0" iyy="1" iyz="0" izz="1" />
 			</inertial>
 		</link>
 		<joint name="${namespace}joint_6" type="revolute">
-			<parent link="${namespace}J5"/>
-			<child link="${namespace}J6"/>
-			<origin rpy="0.000000 0.000000 0.000000" xyz="0.000000 0.000000 0.070000"/>
-			<axis xyz="-0.000000 -0.000000 1.000000"/>
-			<limit effort="1000" lower="-6.28318530717959" upper="6.28318530717959" velocity="5.96902604182061"/> <!-- effort value is arbitary for make gazebo simulation runs without gravity problems -->
-			<dynamics damping="0" friction="0"/>
+			<parent link="${namespace}J5" />
+			<child link="${namespace}J6" />
+			<origin rpy="0.000000 0.000000 0.000000" xyz="0.000000 0.000000 0.070000" />
+			<axis xyz="-0.000000 -0.000000 1.000000" />
+			<limit effort="3.13" lower="${radians(-360)}" upper="${radians(360)}" velocity="${radians(680)}" />
+			<dynamics damping="0" friction="0" />
+		</joint>
+    <link name="${namespace}flange" />
+		<joint name="${namespace}J6-flange" type="fixed">
+      <parent link="${namespace}J6" />
+      <child link="${namespace}flange" />
+      <origin rpy="0 0 0" xyz="0 0 0" />
+		</joint>
+		<link name="${namespace}tool0" />
+		<joint name="${namespace}J6-tool0" type="fixed">
+      <parent link="${namespace}J6" />
+      <child link="${namespace}tool0" />
+      <origin rpy="${radians(pi)} ${radians(-pi/2)} 0" xyz="0 0 0" />
 		</joint>
 	</xacro:macro>
