Commit message: refactor(vs060): overhaul MoveIt configurations and URDF kinematics
- Flatten nested `move_group/ros__parameters` structures in the MoveIt configuration YAML files.
- Introduce `flange` and `tool0` dummy links to standardize end-effector attachments.
- Update `denso_robot_joint_limits.xacro` to support velocity command and effort state interfaces.
- Standardize camera arguments to `gz_cam` and fix legacy xacro namespace URLs.

File: denso_robot_descriptions/robots/vs060/urdf/denso_robot_macro.xacro (robot description, xacro)
@@ -1,4 +1,4 @@
 <?xml version="1.0"?>
-<robot xmlns:xacro="http://wiki.ros.org/xacro">
+<robot xmlns:xacro="http://www.ros.org/wiki/xacro">
   <!--
     Base Denso robot xacro macro.
@@ -9,77 +9,73 @@
     Author DENSO WAVE INCORPORATED
   -->
-  <xacro:macro name="denso_robot" params="
-    model
-    namespace
-    parent
-    *origin
-    transmission_hw_interface:=hardware_interface/PositionJointInterface
-    sim:=false
-    basic_camera:=false
-    ip_address
-    send_format
-    recv_format
-    verbose:=false"
-  >
-    <!-- Robot data required by the denso driver -->
-    <xacro:arg name="ip_address" default="192.168.0.1"/>
-    <xacro:arg name="robot_name" default="VS060A3-AV6-NNN-NNN A"/> <!-- "robot_name" param must be consistent with the @TYPE_NAME variable of the real robot !! -->
-    <xacro:arg name="robot_joints" default="6"/> <!-- number of total joints in the kinematic chain -->
-    <xacro:arg name="joint_1" default="1"/> <!-- 0 = prismatic , 1 = revolute -->
-    <xacro:arg name="joint_2" default="1"/> <!-- 0 = prismatic , 1 = revolute -->
-    <xacro:arg name="joint_3" default="1"/> <!-- 0 = prismatic , 1 = revolute -->
-    <xacro:arg name="joint_4" default="1"/> <!-- 0 = prismatic , 1 = revolute -->
-    <xacro:arg name="joint_5" default="1"/> <!-- 0 = prismatic , 1 = revolute -->
-    <xacro:arg name="joint_6" default="1"/> <!-- 0 = prismatic , 1 = revolute -->
-    <xacro:arg name="controller_type" default="8"/> <!-- 8 = RC8 , 9 = RC9 -->
-    <xacro:arg name="arm_group" default="0"/>
-    <xacro:arg name="send_format" default="288"/>
-    <xacro:arg name="recv_format" default="292"/>
-    <xacro:arg name="verbose" default="false"/>
-    <!-- initial position for simulations-->
-    <xacro:arg name="initial_positions_file" default="$(find denso_robot_descriptions)/robots/$(arg model)/initial_positions.yaml"/>
-    <!-- convert to property to use substitution in function -->
-    <xacro:property name="initial_positions_file" default="$(arg initial_positions_file)"/>
-    <xacro:include filename="$(find denso_robot_descriptions)/robots/$(arg model)/urdf/denso_robot_transmissions.xacro" />
-    <!-- robot kinematics include -->
-    <xacro:include filename="$(find denso_robot_descriptions)/robots/$(arg model)/urdf/denso_robot_kinematics.xacro" />
-    <!-- ros2 control include -->
-    <xacro:include filename="$(find denso_robot_descriptions)/robots/$(arg model)/urdf/denso_robot.ros2_control.xacro" />
-    <!-- For other tools, modify the filename parameter to the path of your tool's xacro file. -->
-    <!-- The line with tag xacro:tool passes the parameters defined in your tool's xacro file -->
-    <!-- (see basic_camera.xacro as an example implementation) -->
-    <xacro:if value="$(arg basic_camera)">
-      <xacro:include filename="$(find denso_robot_gazebo)/sensors/basic_camera/urdf/basic_camera.xacro" />
-    </xacro:if>
-    <!-- ros2 control instance -->
-    <xacro:denso_robot_ros2_control
-      name="GazeboSystem" namespace="${namespace}"
-      sim="$(arg sim)"
-      model="$(arg model)"
-      ip_address="$(arg ip_address)"
-      robot_name="$(arg robot_name)"
-      robot_joints="$(arg robot_joints)"
-      joint_1="$(arg joint_1)"
-      joint_2="$(arg joint_2)"
-      joint_3="$(arg joint_3)"
-      joint_4="$(arg joint_4)"
-      joint_5="$(arg joint_5)"
-      joint_6="$(arg joint_6)"
-      arm_group="$(arg arm_group)"
-      controller_type="$(arg controller_type)"
-      verbose="$(arg verbose)"
-      send_format="$(arg send_format)"
-      recv_format="$(arg recv_format)"
-      initial_positions="${xacro.load_yaml(initial_positions_file)}" />
-    <!-- Add URDF transmission elements (for ros_control) -->
-    <xacro:denso_robot_arm_transmission namespace="${namespace}" hw_interface="$(arg transmission_hw_interface)" />
-    <!-- Placeholder for ros2_control transmission which don't yet exist -->
-    <!-- links -  main serial chain -->
-    <xacro:denso_robot_arm_kinematics namespace="${namespace}" model="$(arg model)" parent="${parent}" >
-      <xacro:insert_block name="origin" />
-    </xacro:denso_robot_arm_kinematics>
-    <xacro:if value="$(arg basic_camera)">
-      <xacro:basic_camera namespace="${namespace}" end_effector="J6" />
-    </xacro:if>
+  <xacro:macro name="denso_robot" params="model
+                                          namespace
+                                          parent
+                                          *origin
+                                          transmission_hw_interface:=hardware_interface/PositionJointInterface
+                                          sim:=false
+                                          basic_camera:=false
+                                          ip_address
+                                          send_format
+                                          recv_format
+                                          verbose:=false">
+  <!-- Robot data required by the denso driver -->
+  <xacro:arg name="ip_address" default=""/>
+  <xacro:arg name="robot_name" default="VS060A3-AV6-NNN-NNN A"/> <!-- "robot_name" param must be consistent with the @TYPE_NAME variable of the real robot !! -->
+  <xacro:arg name="robot_joints" default="6"/> <!-- number of total joints in the kinematic chain -->
+  <xacro:arg name="joint_1" default="1"/> <!-- 0 = prismatic , 1 = revolute -->
+  <xacro:arg name="joint_2" default="1"/> <!-- 0 = prismatic , 1 = revolute -->
+  <xacro:arg name="joint_3" default="1"/> <!-- 0 = prismatic , 1 = revolute -->
+  <xacro:arg name="joint_4" default="1"/> <!-- 0 = prismatic , 1 = revolute -->
+  <xacro:arg name="joint_5" default="1"/> <!-- 0 = prismatic , 1 = revolute -->
+  <xacro:arg name="joint_6" default="1"/> <!-- 0 = prismatic , 1 = revolute -->
+  <xacro:arg name="controller_type" default="8"/> <!-- 8 = RC8 , 9 = RC9 -->
+  <xacro:arg name="arm_group" default="0"/>
+  <xacro:arg name="send_format" default="288"/>
+  <xacro:arg name="recv_format" default="292"/>
+  <xacro:arg name="verbose" default="false"/>
+  <!-- initial position for simulations-->
+  <xacro:arg name="initial_positions_file" default="$(find denso_robot_moveit_config)/robots/$(arg model)/config/initial_positions.yaml" />
+  <xacro:include filename="$(find denso_robot_descriptions)/robots/$(arg model)/urdf/denso_robot_transmissions.xacro" />
+  <!-- robot kinematics include -->
+  <xacro:include filename="$(find denso_robot_descriptions)/robots/$(arg model)/urdf/denso_robot_kinematics.xacro" />
+  <!-- ros2 control include -->
+  <xacro:include filename="$(find denso_robot_descriptions)/robots/$(arg model)/urdf/denso_robot.ros2_control.xacro" />
+  <!-- For other tools, modify the filename parameter to the path of your tool's xacro file. -->
+  <!-- The line with tag xacro:tool passes the parameters defined in your tool's xacro file -->
+  <!-- (see basic_camera.xacro as an example implementation) -->
+  <xacro:if value="$(arg basic_camera)">
+    <xacro:include filename="$(find denso_robot_gazebo)/sensors/basic_camera/urdf/basic_camera.xacro" />
+  </xacro:if>
+  <!-- ros2 control instance -->
+  <xacro:denso_robot_ros2_control name="VS050"
+                                  namespace="${namespace}"
+                                  sim="$(arg sim)"
+                                  model="$(arg model)"
+                                  ip_address="${ip_address}"
+                                  robot_name="$(arg robot_name)"
+                                  robot_joints="$(arg robot_joints)"
+                                  joint_1="$(arg joint_1)"
+                                  joint_2="$(arg joint_2)"
+                                  joint_3="$(arg joint_3)"
+                                  joint_4="$(arg joint_4)"
+                                  joint_5="$(arg joint_5)"
+                                  joint_6="$(arg joint_6)"
+                                  arm_group="$(arg arm_group)"
+                                  controller_type="$(arg controller_type)"
+                                  verbose="$(arg verbose)"
+                                  send_format="$(arg send_format)"
+                                  recv_format="$(arg recv_format)"
+                                  initial_positions_file="$(arg initial_positions_file)" />
+  <!-- Add URDF transmission elements (for ros_control) -->
+  <xacro:denso_robot_arm_transmission namespace="${namespace}" hw_interface="$(arg transmission_hw_interface)" />
+  <!-- Placeholder for ros2_control transmission which don't yet exist -->
+  <!-- links -  main serial chain -->
+  <xacro:denso_robot_arm_kinematics namespace="${namespace}" model="$(arg model)" parent="${parent}">
+    <xacro:insert_block name="origin" />
+  </xacro:denso_robot_arm_kinematics>
+  <xacro:if value="$(arg basic_camera)">
+    <xacro:basic_camera namespace="${namespace}" end_effector="J6" />
+  </xacro:if>
   </xacro:macro>
 </robot>

Commit message: fix(vs050): update acceleration and effort limits for proper simulation
Increases moveit acceleration limits to realistic values to fix slow movements and standardizes URDF joint efforts to 175 to stabilize Gazebo physics.

File: denso_robot_descriptions/robots/vs050/urdf/denso_robot_kinematics.xacro (robot description, xacro)
@@ -50,6 +50,6 @@
 			<origin rpy="0.000000 0.000000 0.000000" xyz="0.000000 0.000000 0.181500" />
 			<axis xyz="-0.000000 -0.000000 1.000000" />
-      <!-- effort value is arbitary for make gazebo simulation runs without gravity problems -->
-			<limit effort="1000" lower="${radians(-170)}" upper="${radians(170)}" velocity="${radians(425)}" />
+      		<!-- effort value is arbitary for make gazebo simulation runs without problems -->
+			<limit effort="175" lower="${radians(-170)}" upper="${radians(170)}" velocity="${radians(425)}" />
 			<dynamics damping="0" friction="0" />
 		</joint>
@@ -78,6 +78,6 @@
 			<origin rpy="0.000000 0.000000 0.000000" xyz="0.000000 0.000000 0.163500" />
 			<axis xyz="-0.000000 1.000000 -0.000000" />
-      <!-- effort value is arbitary for make gazebo simulation runs without gravity problems -->
-			<limit effort="1000" lower="${radians(-120)}" upper="${radians(120)}" velocity="${radians(340)}" />
+      		<!-- effort value is arbitary for make gazebo simulation runs without problems -->
+			<limit effort="175" lower="${radians(-120)}" upper="${radians(120)}" velocity="${radians(340)}" />
 			<dynamics damping="0" friction="0" />
 		</joint>
@@ -106,6 +106,6 @@
 			<origin rpy="0.000000 0.000000 0.000000" xyz="0.000000 0.000000 0.250000" />
 			<axis xyz="-0.000000 1.000000 -0.000000" />
-      <!-- effort value is arbitary for make gazebo simulation runs without gravity problems -->
-			<limit effort="1000" lower="${radians(-120)}" upper="${radians(151)}" velocity="${radians(385.72)}" />
+      		<!-- effort value is arbitary for make gazebo simulation runs without problems -->
+			<limit effort="175" lower="${radians(-120)}" upper="${radians(151)}" velocity="${radians(385.72)}" />
 			<dynamics damping="0" friction="0" />
 		</joint>
@@ -134,5 +134,6 @@
 			<origin rpy="0.000000 0.000000 0.000000" xyz="-0.010000 0.000000 0.119500" />
 			<axis xyz="-0.000000 -0.000000 1.000000" />
-			<limit effort="6.66" lower="${radians(-270)}" upper="${radians(270)}" velocity="${radians(425)}" />
+			<!-- effort value is arbitary for make gazebo simulation runs without problems -->
+			<limit effort="175" lower="${radians(-270)}" upper="${radians(270)}" velocity="${radians(425)}" />
 			<dynamics damping="0" friction="0" />
 		</joint>
@@ -161,5 +162,6 @@
 			<origin rpy="0.000000 0.000000 0.000000" xyz="0.000000 0.000000 0.135500" />
 			<axis xyz="-0.000000 1.000000 -0.000000" />
-			<limit effort="6.66" lower="${radians(-120)}" upper="${radians(120)}" velocity="${radians(327.01)}" />
+			<!-- effort value is arbitary for make gazebo simulation runs without problems -->
+			<limit effort="175" lower="${radians(-120)}" upper="${radians(120)}" velocity="${radians(327.01)}" />
 			<dynamics damping="0" friction="0" />
 		</joint>
@@ -188,5 +190,6 @@
 			<origin rpy="0.000000 0.000000 0.000000" xyz="0.000000 0.000000 0.070000" />
 			<axis xyz="-0.000000 -0.000000 1.000000" />
-			<limit effort="3.13" lower="${radians(-360)}" upper="${radians(360)}" velocity="${radians(680)}" />
+			<!-- effort value is arbitary for make gazebo simulation runs without problems -->
+			<limit effort="175" lower="${radians(-360)}" upper="${radians(360)}" velocity="${radians(680)}" />
 			<dynamics damping="0" friction="0" />
 		</joint>

Commit message: fix(vs050): correct tool0 frame orientation math and indentation
- Remove the incorrect `radians()` function wrapper around `pi` in the `J6-tool0` joint origin. Since `pi` is already in radians, `radians(pi)` resulted in an incorrect rotation.
- Fix XML indentation for the child, parent, and origin tags within the flange and tool0 joints to improve code readability.

File: denso_robot_descriptions/robots/vs050/urdf/denso_robot_kinematics.xacro (robot description, xacro)
@@ -196,13 +196,13 @@
 		<link name="${namespace}flange"/>
 		<joint name="${namespace}J6-flange" type="fixed">
-		<parent link="${namespace}J6"/>
-		<child link="${namespace}flange"/>
-		<origin rpy="0 0 0" xyz="0 0 0"/>
+			<parent link="${namespace}J6"/>
+			<child link="${namespace}flange"/>
+			<origin rpy="0 0 0" xyz="0 0 0"/>
 		</joint>
 		<link name="${namespace}tool0"/>
 		<joint name="${namespace}J6-tool0" type="fixed">
-		<parent link="${namespace}J6"/>
-		<child link="${namespace}tool0"/>
-		<origin rpy="${radians(pi)} ${radians(-pi/2)} 0" xyz="0 0 0"/>
+			<parent link="${namespace}J6"/>
+			<child link="${namespace}tool0"/>
+			<origin rpy="${pi} ${-pi/2} 0" xyz="0 0 0"/>
 		</joint>
 	</xacro:macro>
