Commit message: feat(description): update VS050 physical properties for simulation
- replace placeholder inertial values with calibrated mass, center of mass, and inertia tensors for all links
- update joint effort limits to match the robot specifications
- use unlimited effort (`-1`) for joints driven by position control
- clarify the meaning of negative effort limits with inline documentation

File: denso_robot_descriptions/robots/vs050/urdf/denso_robot_kinematics.xacro (robot description, xacro)
@@ -21,7 +21,7 @@
 			</collision>
 			<inertial>
-				<mass value="1" />
-				<origin rpy="0.000000 0.000000 0.000000" xyz="0.000000 0.000000 0.000000" />
-				<inertia ixx="1" ixy="0" ixz="0" iyy="1" iyz="0" izz="1" />
+				<mass value="10.671" />
+				<origin rpy="0.000000 0.000000 0.000000" xyz="-0.03867582 -0.0001277 0.09016489" />
+				<inertia ixx="2.56206696e-05" ixy="0" ixz="0" iyy="4.04209402e-05" iyz="0" izz="3.52484166e-05" />
 			</inertial>
 		</link>
@@ -40,7 +40,7 @@
 			</collision>
 			<inertial>
-				<mass value="1" />
-				<origin rpy="0.000000 0.000000 0.000000" xyz="0.000000 0.000000 0.000000" />
-				<inertia ixx="1" ixy="0" ixz="0" iyy="1" iyz="0" izz="1" />
+				<mass value="4.955" />
+				<origin rpy="0.000000 0.000000 0.000000" xyz="0.0087579 -0.0012957 0.08320129" />
+				<inertia ixx="2.03430428e-05" ixy="0" ixz="0" iyy="1.43075081e-05" iyz="0" izz="1.33370577e-05" />
 			</inertial>
 		</link>
@@ -50,6 +50,6 @@
 			<origin rpy="0.000000 0.000000 0.000000" xyz="0.000000 0.000000 0.181500" />
 			<axis xyz="-0.000000 -0.000000 1.000000" />
-      		<!-- effort value is arbitary for make gazebo simulation runs without problems -->
-			<limit effort="175" lower="${radians(-170)}" upper="${radians(170)}" velocity="${radians(425)}" />
+      		<!-- a negative effort value acts as a sentinel meaning "no limit" (treated as infinite) -->
+			<limit effort="-1" lower="${radians(-170)}" upper="${radians(170)}" velocity="${radians(425)}" />
 			<dynamics damping="0" friction="0" />
 		</joint>
@@ -68,7 +68,7 @@
 			</collision>
 			<inertial>
-				<mass value="1" />
-				<origin rpy="0.000000 0.000000 0.000000" xyz="0.000000 0.000000 0.000000" />
-				<inertia ixx="1" ixy="0" ixz="0" iyy="1" iyz="0" izz="1" />
+				<mass value="6.184" />
+				<origin rpy="0.000000 0.000000 0.000000" xyz="-0.01386069 -0.00042137 0.08832005" />
+				<inertia ixx="3.54063103e-05" ixy="0" ixz="0" iyy="3.25785729e-05" iyz="0" izz="9.77018345e-06" />
 			</inertial>
 		</link>
@@ -78,6 +78,6 @@
 			<origin rpy="0.000000 0.000000 0.000000" xyz="0.000000 0.000000 0.163500" />
 			<axis xyz="-0.000000 1.000000 -0.000000" />
-      		<!-- effort value is arbitary for make gazebo simulation runs without problems -->
-			<limit effort="175" lower="${radians(-120)}" upper="${radians(120)}" velocity="${radians(340)}" />
+      		<!-- a negative effort value acts as a sentinel meaning "no limit" (treated as infinite) -->
+			<limit effort="-1" lower="${radians(-120)}" upper="${radians(120)}" velocity="${radians(340)}" />
 			<dynamics damping="0" friction="0" />
 		</joint>
@@ -96,7 +96,7 @@
 			</collision>
 			<inertial>
-				<mass value="1" />
-				<origin rpy="0.000000 0.000000 0.000000" xyz="0.000000 0.000000 0.000000" />
-				<inertia ixx="1" ixy="0" ixz="0" iyy="1" iyz="0" izz="1" />
+				<mass value="2.645" />
+				<origin rpy="0.000000 0.000000 0.000000" xyz="-0.00406821 0.0016604 0.03603942" />
+				<inertia ixx="4.41330319e-06" ixy="0" ixz="0" iyy="4.45791777e-06" iyz="0" izz="2.03895005e-06" />
 			</inertial>
 		</link>
@@ -106,6 +106,6 @@
 			<origin rpy="0.000000 0.000000 0.000000" xyz="0.000000 0.000000 0.250000" />
 			<axis xyz="-0.000000 1.000000 -0.000000" />
-      		<!-- effort value is arbitary for make gazebo simulation runs without problems -->
-			<limit effort="175" lower="${radians(-120)}" upper="${radians(151)}" velocity="${radians(385.72)}" />
+      		<!-- a negative effort value acts as a sentinel meaning "no limit" (treated as infinite) -->
+			<limit effort="-1" lower="${radians(-120)}" upper="${radians(151)}" velocity="${radians(385.72)}" />
 			<dynamics damping="0" friction="0" />
 		</joint>
@@ -124,7 +124,7 @@
 			</collision>
 			<inertial>
-				<mass value="1" />
-				<origin rpy="0.000000 0.000000 0.000000" xyz="0.000000 0.000000 0.000000" />
-				<inertia ixx="1" ixy="0" ixz="0" iyy="1" iyz="0" izz="1" />
+				<mass value="1.770" />
+				<origin rpy="0.000000 0.000000 0.000000" xyz="-0.00090245 0.00241103 0.0619847" />
+				<inertia ixx="2.99417953e-06" ixy="0" ixz="0" iyy="2.61053927e-06" iyz="0" izz="1.50605741e-06" />
 			</inertial>
 		</link>
@@ -134,6 +134,5 @@
 			<origin rpy="0.000000 0.000000 0.000000" xyz="-0.010000 0.000000 0.119500" />
 			<axis xyz="-0.000000 -0.000000 1.000000" />
-			<!-- effort value is arbitary for make gazebo simulation runs without problems -->
-			<limit effort="175" lower="${radians(-270)}" upper="${radians(270)}" velocity="${radians(425)}" />
+			<limit effort="6.66" lower="${radians(-270)}" upper="${radians(270)}" velocity="${radians(425)}" />
 			<dynamics damping="0" friction="0" />
 		</joint>
@@ -152,7 +151,7 @@
 			</collision>
 			<inertial>
-				<mass value="1" />
-				<origin rpy="0.000000 0.000000 0.000000" xyz="0.000000 0.000000 0.000000" />
-				<inertia ixx="1" ixy="0" ixz="0" iyy="1" iyz="0" izz="1" />
+				<mass value="0.735" />
+				<origin rpy="0.000000 0.000000 0.000000" xyz="0.00125985 -0.00178539 0.00593704" />
+				<inertia ixx="4.39629328e-07" ixy="0" ixz="0" iyy="5.25922017e-07" iyz="0" izz="2.67062349e-07" />
 			</inertial>
 		</link>
@@ -162,6 +161,5 @@
 			<origin rpy="0.000000 0.000000 0.000000" xyz="0.000000 0.000000 0.135500" />
 			<axis xyz="-0.000000 1.000000 -0.000000" />
-			<!-- effort value is arbitary for make gazebo simulation runs without problems -->
-			<limit effort="175" lower="${radians(-120)}" upper="${radians(120)}" velocity="${radians(327.01)}" />
+			<limit effort="6.66" lower="${radians(-120)}" upper="${radians(120)}" velocity="${radians(327.01)}" />
 			<dynamics damping="0" friction="0" />
 		</joint>
@@ -180,7 +178,7 @@
 			</collision>
 			<inertial>
-				<mass value="1" />
-				<origin rpy="0.000000 0.000000 0.000000" xyz="0.000000 0.000000 0.000000" />
-				<inertia ixx="1" ixy="0" ixz="0" iyy="1" iyz="0" izz="1" />
+				<mass value="0.041" />
+				<origin rpy="0.000000 0.000000 0.000000" xyz="-4.13833459e-07 -7.00967243e-05 -1.06200824e-02" />
+				<inertia ixx="2.96285977e-09" ixy="0" ixz="0" iyy="2.98822098e-09" iyz="0" izz="4.55917832e-09" />
 			</inertial>
 		</link>
@@ -190,6 +188,5 @@
 			<origin rpy="0.000000 0.000000 0.000000" xyz="0.000000 0.000000 0.070000" />
 			<axis xyz="-0.000000 -0.000000 1.000000" />
-			<!-- effort value is arbitary for make gazebo simulation runs without problems -->
-			<limit effort="175" lower="${radians(-360)}" upper="${radians(360)}" velocity="${radians(680)}" />
+			<limit effort="3.13" lower="${radians(-360)}" upper="${radians(360)}" velocity="${radians(680)}" />
 			<dynamics damping="0" friction="0" />
 		</joint>

Commit message: fix(description): replace unlimited joint effort sentinel with large effort limit
- replace negative effort limits with `1e6` for joints 1–3
- document the reason for using a large finite effort limit instead of the previous sentinel value

File: denso_robot_descriptions/robots/vs050/urdf/denso_robot_kinematics.xacro (robot description, xacro)
@@ -50,6 +50,8 @@
 			<origin rpy="0.000000 0.000000 0.000000" xyz="0.000000 0.000000 0.181500" />
 			<axis xyz="-0.000000 -0.000000 1.000000" />
-      		<!-- a negative effort value acts as a sentinel meaning "no limit" (treated as infinite) -->
-			<limit effort="-1" lower="${radians(-170)}" upper="${radians(170)}" velocity="${radians(425)}" />
+      		<!-- Initially, a negative effort value acting as a sentinel indicating "no limit" (treated as infinity) was used,
+			but this was changed following the error on line 175 of
+			https://github.com/gazebosim/gz-physics/blob/ign-physics5/dartsim/src/JointFeatures.cc -->
+			<limit effort="1e6" lower="${radians(-170)}" upper="${radians(170)}" velocity="${radians(425)}" />
 			<dynamics damping="0" friction="0" />
 		</joint>
@@ -78,6 +80,8 @@
 			<origin rpy="0.000000 0.000000 0.000000" xyz="0.000000 0.000000 0.163500" />
 			<axis xyz="-0.000000 1.000000 -0.000000" />
-      		<!-- a negative effort value acts as a sentinel meaning "no limit" (treated as infinite) -->
-			<limit effort="-1" lower="${radians(-120)}" upper="${radians(120)}" velocity="${radians(340)}" />
+      		<!-- Initially, a negative effort value acting as a sentinel indicating "no limit" (treated as infinity) was used,
+			but this was changed following the error on line 175 of
+			https://github.com/gazebosim/gz-physics/blob/ign-physics5/dartsim/src/JointFeatures.cc -->
+			<limit effort="1e6" lower="${radians(-120)}" upper="${radians(120)}" velocity="${radians(340)}" />
 			<dynamics damping="0" friction="0" />
 		</joint>
@@ -106,6 +110,8 @@
 			<origin rpy="0.000000 0.000000 0.000000" xyz="0.000000 0.000000 0.250000" />
 			<axis xyz="-0.000000 1.000000 -0.000000" />
-      		<!-- a negative effort value acts as a sentinel meaning "no limit" (treated as infinite) -->
-			<limit effort="-1" lower="${radians(-120)}" upper="${radians(151)}" velocity="${radians(385.72)}" />
+      		<!-- Initially, a negative effort value acting as a sentinel indicating "no limit" (treated as infinity) was used,
+			but this was changed following the error on line 175 of
+			https://github.com/gazebosim/gz-physics/blob/ign-physics5/dartsim/src/JointFeatures.cc -->
+			<limit effort="1e6" lower="${radians(-120)}" upper="${radians(151)}" velocity="${radians(385.72)}" />
 			<dynamics damping="0" friction="0" />
 		</joint>

Commit message: fix(description): align flange and tool0 frames with robot convention
- rotate the flange frame to match the expected orientation
- reset the `tool0` frame transform to the robot base convention

File: denso_robot_descriptions/robots/vs050/urdf/denso_robot_kinematics.xacro (robot description, xacro)
@@ -201,5 +201,5 @@
 			<parent link="${namespace}J6"/>
 			<child link="${namespace}flange"/>
-			<origin rpy="0 0 0" xyz="0 0 0"/>
+			<origin rpy="0 ${radians(-90)} 0" xyz="0 0 0"/>
 		</joint>
 		<link name="${namespace}tool0"/>
@@ -207,5 +207,5 @@
 			<parent link="${namespace}J6"/>
 			<child link="${namespace}tool0"/>
-			<origin rpy="${pi} ${-pi/2} 0" xyz="0 0 0"/>
+			<origin rpy="0 0 0" xyz="0 0 0"/>
 		</joint>
 	</xacro:macro>

Commit message: fix(description): replace unlimited joint effort sentinel with large effort limit
- replace negative effort limits with `1e6` for joints 1–3
- document the reason for using a large finite effort limit instead of the previous sentinel value

(cherry picked from commit df1dda3e1f5687aba68d788c636ef6b6b7d7b7e2)

File: denso_robot_descriptions/robots/vs050/urdf/denso_robot_kinematics.xacro (robot description, xacro)
@@ -50,6 +50,8 @@
 			<origin rpy="0.000000 0.000000 0.000000" xyz="0.000000 0.000000 0.181500" />
 			<axis xyz="-0.000000 -0.000000 1.000000" />
-      		<!-- a negative effort value acts as a sentinel meaning "no limit" (treated as infinite) -->
-			<limit effort="-1" lower="${radians(-170)}" upper="${radians(170)}" velocity="${radians(425)}" />
+      		<!-- Initially, a negative effort value acting as a sentinel indicating "no limit" (treated as infinity) was used,
+			but this was changed following the error on line 175 of
+			https://github.com/gazebosim/gz-physics/blob/gz-physics7/dartsim/src/JointFeatures.cc -->
+			<limit effort="1e6" lower="${radians(-170)}" upper="${radians(170)}" velocity="${radians(425)}" />
 			<dynamics damping="0" friction="0" />
 		</joint>
@@ -78,6 +80,8 @@
 			<origin rpy="0.000000 0.000000 0.000000" xyz="0.000000 0.000000 0.163500" />
 			<axis xyz="-0.000000 1.000000 -0.000000" />
-      		<!-- a negative effort value acts as a sentinel meaning "no limit" (treated as infinite) -->
-			<limit effort="-1" lower="${radians(-120)}" upper="${radians(120)}" velocity="${radians(340)}" />
+      		<!-- Initially, a negative effort value acting as a sentinel indicating "no limit" (treated as infinity) was used,
+			but this was changed following the error on line 175 of
+			https://github.com/gazebosim/gz-physics/blob/gz-physics7/dartsim/src/JointFeatures.cc -->
+			<limit effort="1e6" lower="${radians(-120)}" upper="${radians(120)}" velocity="${radians(340)}" />
 			<dynamics damping="0" friction="0" />
 		</joint>
@@ -106,6 +110,8 @@
 			<origin rpy="0.000000 0.000000 0.000000" xyz="0.000000 0.000000 0.250000" />
 			<axis xyz="-0.000000 1.000000 -0.000000" />
-      		<!-- a negative effort value acts as a sentinel meaning "no limit" (treated as infinite) -->
-			<limit effort="-1" lower="${radians(-120)}" upper="${radians(151)}" velocity="${radians(385.72)}" />
+      		<!-- Initially, a negative effort value acting as a sentinel indicating "no limit" (treated as infinity) was used,
+			but this was changed following the error on line 175 of
+			https://github.com/gazebosim/gz-physics/blob/gz-physics7/dartsim/src/JointFeatures.cc -->
+			<limit effort="1e6" lower="${radians(-120)}" upper="${radians(151)}" velocity="${radians(385.72)}" />
 			<dynamics damping="0" friction="0" />
 		</joint>
