Commit message: refactor(sensors): convert gz_cam link to a virtual frame
- Remove physical properties (mass, inertia, collision, and visual box) from the camera link definition in `gz_cam.xacro`.
- Clean up the overall XML indentation and formatting.

File: denso_robot_gazebo/sensors/gz_cam/urdf/gz_cam.xacro (robot description, xacro)
@@ -1,49 +1,34 @@
-<?xml version='1.0' encoding='UTF-8'?>
+<?xml version='1.0'?>
 <robot xmlns:xacro="http://www.ros.org/wiki/xacro">
     <!-- here you define the parameters you want your xacro file to receive. -->
     <xacro:macro name="gz_cam" params="namespace">
-    <!-- if your tool has meshes, define the path to it in geometry tag. -->
-    <!-- see the vs050 robot urdf implementation as an example. -->
-    <link name="${namespace}gz_cam_link">
-		<inertial>
-			<mass value="1"/>
-			<inertia ixx="1" ixy="0" ixz="0" iyy="1" iyz="0" izz="1"/>
-		</inertial>
-		<collision>
-			<geometry>
-				<box size="0.01 0.01 0.01"/>
-			</geometry>
-		</collision>
-		<visual>
-			<geometry>
-				<box size="0.01 0.01 0.01"/>
-			</geometry>
-		</visual>
-	</link>
-	<joint name="${namespace}gz_cam_joint" type="fixed">
-        <!-- here you define where your tool will connect. In this case, it's at joint 6. -->
-		<parent link="${namespace}flange"/>
-		<child link="${namespace}gz_cam_link"/>
-		<origin rpy="0 ${radians(-90)} 0" xyz="0 0 0.01"/>
-	</joint>
-    <gazebo reference="${namespace}gz_cam_link">
-      <sensor name="${namespace}gz_cam" type="camera">
-        <camera>
-          <horizontal_fov>1.047</horizontal_fov>
-          <image>
-            <width>640</width>
-            <height>480</height>
-          </image>
-          <clip>
-            <near>0.1</near>
-            <far>100</far>
-          </clip>
-        </camera>
-        <always_on>1</always_on>
-        <update_rate>30</update_rate>
-        <visualize>true</visualize>
-        <topic>${namespace}gz_cam</topic>
-      </sensor>
-    </gazebo>
+      <!-- if your tool has meshes, define the path to it in geometry tag. -->
+      <!-- see the vs050 robot urdf implementation as an example. -->
+      <link name="${namespace}gz_cam_link" />
+      <joint name="${namespace}gz_cam_joint" type="fixed">
+            <!-- here you define where your tool will connect. In this case, it's at joint 6. -->
+        <parent link="${namespace}flange"/>
+        <child link="${namespace}gz_cam_link"/>
+        <origin rpy="0 ${radians(-90)} 0" xyz="0 0 0.01"/>
+      </joint>
+      <gazebo reference="${namespace}gz_cam_link">
+        <sensor name="${namespace}gz_cam" type="camera">
+          <camera>
+            <horizontal_fov>1.047</horizontal_fov>
+            <image>
+              <width>640</width>
+              <height>480</height>
+            </image>
+            <clip>
+              <near>0.1</near>
+              <far>100</far>
+            </clip>
+          </camera>
+          <always_on>1</always_on>
+          <update_rate>30</update_rate>
+          <visualize>true</visualize>
+          <topic>${namespace}gz_cam</topic>
+        </sensor>
+      </gazebo>
     </xacro:macro>
 </robot>
