Commit message: refactor(gazebo): attach camera sensor directly to the flange
- remove the intermediate camera link and fixed joint
- attach the Gazebo camera sensor directly to the flange frame
- simplify the sensor description and update inline documentation

File: denso_robot_gazebo/sensors/gz_cam/urdf/gz_cam.xacro (robot description, xacro)
@@ -1,16 +1,8 @@
 <?xml version='1.0'?>
 <robot xmlns:xacro="http://www.ros.org/wiki/xacro">
-    <!-- here you define the parameters you want your xacro file to receive. -->
     <xacro:macro name="gz_cam" params="namespace">
-      <!-- if your tool has meshes, define the path to it in geometry tag. -->
-      <!-- see the vs050 robot urdf implementation as an example. -->
-      <link name="${namespace}gz_cam_link" />
-      <joint name="${namespace}gz_cam_joint" type="fixed">
-        <!-- You should always attach the flange -->
-        <parent link="${namespace}flange"/>
-        <child link="${namespace}gz_cam_link"/>
-        <origin rpy="0 ${radians(-90)} 0" xyz="0 0 0.01"/>
-      </joint>
-      <gazebo reference="${namespace}gz_cam_link">
+      <!-- You should always attach the flange -->
+      <gazebo reference="${namespace}flange">
+      <!-- others specs can be add for camera sensor https://sdformat.org/spec/1.9/sensor/#sensor_camera -->
         <sensor name="${namespace}gz_cam" type="camera">
           <camera>
