Commit message: refactor(vs060): modernize SRDF structure and collision matrix
- Streamline the `arm` planning group definition using the `<chain>` element.
- Add standard `tool0` end-effector definitions and a predefined `home` posture.
- Expand the `disable_collisions` matrix to explicitly cover all safe adjacent and never-colliding link pairs, improving planner performance.

File: denso_robot_moveit_config/robots/vs060/srdf/denso_robot_macro.srdf.xacro (robot description, xacro)
@@ -1,4 +1,4 @@
-<?xml version="1.0" encoding="UTF-8"?>
-<robot xmlns:xacro="http://wiki.ros.org/xacro">
+<?xml version="1.0"?>
+<robot xmlns:xacro="http://www.ros.org/wiki/xacro">
 <!--This does not replace URDF, and is not an extension of URDF.
     This is a format for representing semantic information about the robot structure.
@@ -12,24 +12,37 @@
     <!--SUBGROUPS - Groups can also be formed by referencing to already defined group names-->
     <group name="${namespace}arm">
-		<joint name="${namespace}joint_1"/>
-		<joint name="${namespace}joint_2"/>
-		<joint name="${namespace}joint_3"/>
-		<joint name="${namespace}joint_4"/>
-		<joint name="${namespace}joint_5"/>
-		<joint name="${namespace}joint_6"/>
-	</group>
+      <chain base_link="${namespace}base_link" tip_link="${namespace}tool0" />
+    </group>
+    <group name="${namespace}end_effector">
+        <link name="${namespace}tool0"/>
+    </group>
     <!--GROUP STATES - Purpose - Define a named state for a particular group, in terms of joint values. This is useful to define states like 'folded arms'-->
+    <group_state name="${namespace}home" group="${namespace}arm">
+      <joint name="${namespace}joint_1" value="0"/>
+      <joint name="${namespace}joint_2" value="-0.5"/>
+      <joint name="${namespace}joint_3" value="1.2"/>
+      <joint name="${namespace}joint_4" value="0"/>
+      <joint name="${namespace}joint_5" value="1.5"/>
+      <joint name="${namespace}joint_6" value="0"/>
+    </group_state>
     <!--END EFFECTOR - Purpose - Represent information about an end effector.-->
+    <end_effector name="${namespace}eff" parent_link="${namespace}tool0" group="${namespace}end_effector" parent_group="${namespace}arm"/>
     <!--VIRTUAL JOINT - Purpose - this element defines a virtual joint between a robot link and an external frame of reference (considered fixed with respect to the robot)-->
     <virtual_joint name="${namespace}fixed_base" type="fixed" parent_frame="world" child_link="${namespace}base_link" />
     <!--DISABLE COLLISIONS - By default it is assumed that any link of the robot could potentially come into collision with any other link in the robot. This tag disables collision checking between a specified pair of links. -->
-	<disable_collisions link1="${namespace}J6" link2="${namespace}J3" reason="Never"/>
-	<disable_collisions link1="${namespace}J6" link2="${namespace}J5" reason="Adjacent"/>
-	<disable_collisions link1="${namespace}J1" link2="${namespace}J2" reason="Adjacent"/>
-	<disable_collisions link1="${namespace}J1" link2="${namespace}base_link" reason="Adjacent"/>
-	<disable_collisions link1="${namespace}J2" link2="${namespace}J3" reason="Adjacent"/>
-	<disable_collisions link1="${namespace}J3" link2="${namespace}J4" reason="Adjacent"/>
-	<disable_collisions link1="${namespace}J3" link2="${namespace}J5" reason="Never"/>
-	<disable_collisions link1="${namespace}J4" link2="${namespace}J5" reason="Adjacent"/>
+	  <disable_collisions link1="${namespace}J1" link2="${namespace}J2" reason="Adjacent"/>
+    <disable_collisions link1="${namespace}J1" link2="${namespace}J3" reason="Never"/>
+    <disable_collisions link1="${namespace}J1" link2="${namespace}base_link" reason="Adjacent"/>
+    <disable_collisions link1="${namespace}J2" link2="${namespace}J3" reason="Adjacent"/>
+    <disable_collisions link1="${namespace}J2" link2="${namespace}J4" reason="Never"/>
+    <disable_collisions link1="${namespace}J2" link2="${namespace}J5" reason="Never"/>
+    <disable_collisions link1="${namespace}J2" link2="${namespace}J6" reason="Never"/>
+    <disable_collisions link1="${namespace}J2" link2="${namespace}base_link" reason="Never"/>
+    <disable_collisions link1="${namespace}J3" link2="${namespace}J4" reason="Adjacent"/>
+    <disable_collisions link1="${namespace}J3" link2="${namespace}J5" reason="Never"/>
+    <disable_collisions link1="${namespace}J3" link2="${namespace}J6" reason="Never"/>
+    <disable_collisions link1="${namespace}J4" link2="${namespace}J5" reason="Adjacent"/>
+    <disable_collisions link1="${namespace}J4" link2="${namespace}J6" reason="Never"/>
+    <disable_collisions link1="${namespace}J5" link2="${namespace}J6" reason="Adjacent"/>
   </xacro:macro>
 </robot>
