Commit message: fix(hsr065a1): fix xacro namespaces, flatten YAMLs, and optimize collisions
Resolves broken namespace prefixes, updates the MoveIt configuration files to the flattened ROS 2 structure, adds gz_cam/origin support, and significantly improves Gazebo simulation performance by using primitive collision shapes.

File: denso_robot_descriptions/robots/hsr065a1_n32/urdf/denso_robot.ros2_control.xacro (robot description, xacro)
@@ -1,29 +1,36 @@
 <?xml version="1.0"?>
 <robot xmlns:xacro="http://www.ros.org/wiki/xacro">
-  <xacro:macro name="denso_robot_ros2_control" params="name namespace
-	robot_name
-    sim:=false fake_sensor_commands:=false
-    ip_address
-    model
-    robot_joints joint_1 joint_2 joint_3 joint_4
-    arm_group
-    send_format recv_format
-	controller_type
-    verbose
-    ">
+  <xacro:macro name="denso_robot_ros2_control"
+               params="name
+                       namespace
+                       robot_name
+                       sim:=false
+                       fake_sensor_commands:=false
+                       ip_address
+                       model
+                       robot_joints
+                       joint_1
+                       joint_2
+                       joint_3
+                       joint_4
+                       arm_group
+                       send_format
+                       recv_format
+                       controller_type
+                       verbose">
     <ros2_control name="${namespace}${name}" type="system">
-	<!-- joint limits include -->
-	<xacro:include filename="$(find denso_robot_descriptions)/robots/$(arg model)/urdf/denso_robot_joint_limits.xacro" />
+      <!-- joint limits include -->
+      <xacro:include filename="$(find denso_robot_descriptions)/robots/$(arg model)/urdf/denso_robot_joint_limits.xacro" />
       <hardware>
         <xacro:if value="${sim}">
-      	  <plugin>gz_ros2_control/GazeboSimSystem</plugin>
+          <plugin>gz_ros2_control/GazeboSimSystem</plugin>
         </xacro:if>
         <xacro:unless value="${sim}">
           <plugin>denso_robot_control/DensoRobotHW</plugin>
           <param name="ip_address">${ip_address}</param>
-<!-- "robot_name" param must be consistent with the @TYPE_NAME variable of the real robot !!  -->
+          <!-- "robot_name" param must be consistent with the @TYPE_NAME variable of the real robot !! -->
           <param name="robot_name">${robot_name}</param>
           <param name="node_name">denso_robot_control</param>
-          <param name="node_namespace">${namespace}${model}</param>
+          <param name="node_namespace">${namespace}$(arg model)</param>
           <param name="robot_joints">${robot_joints}</param>
           <param name="joint_1">${joint_1}</param>
@@ -38,5 +45,5 @@
         </xacro:unless>
       </hardware>
-      <xacro:denso_robot_control_limits namespace="$(arg namespace)" />
+      <xacro:denso_robot_control_limits namespace="${namespace}" />
     </ros2_control>
   </xacro:macro>

File: denso_robot_descriptions/robots/hsr065a1_n32/urdf/denso_robot_kinematics.xacro (robot description, xacro)
@@ -1,11 +1,11 @@
 <?xml version='1.0' encoding='UTF-8'?>
 <robot xmlns:xacro="http://www.ros.org/wiki/xacro">
-	<xacro:macro name="denso_robot_arm_kinematics" params="namespace model">
-		<link name="world"/>
-		<joint name="$(arg namespace)joint_w" type="fixed">
-			<parent link="world"/>
-			<child link="$(arg namespace)base_link"/>
+	<xacro:macro name="denso_robot_arm_kinematics" params="namespace model parent *origin">
+		<joint name="${namespace}joint_w" type="fixed">
+			<xacro:insert_block name="origin" />
+			<parent link="${parent}" />
+			<child link="${namespace}base_link" />
 		</joint>
-		<link name="$(arg namespace)base_link">
+		<link name="${namespace}base_link">
 			<visual>
 				<origin rpy="0 0 0" xyz="0 0 0"/>
@@ -15,16 +15,16 @@
 			</visual>
 			<collision>
-				<origin rpy="0 0 0" xyz="0 0 0"/>
+				<origin rpy="0 0 0" xyz="0 0 0.050"/>
 				<geometry>
-					<mesh filename="file:///$(find denso_robot_descriptions)/robots/$(arg model)/meshes/base_link.dae" scale="1 1 1"/>
+					<cylinder radius="0.100" length="0.100"/>
 				</geometry>
 			</collision>
 			<inertial>
 				<mass value="1"/>
-				<origin rpy="0.000000 0.000000 0.000000" xyz="0.000000 0.000000 0.000000"/>
+				<origin rpy="0 0 0" xyz="0 0 0"/>
 				<inertia ixx="1" ixy="0" ixz="0" iyy="1" iyz="0" izz="1"/>
 			</inertial>
 		</link>
-		<link name="$(arg namespace)J1">
+		<link name="${namespace}J1">
 			<visual>
 				<origin rpy="0 0 0" xyz="0 0 0"/>
@@ -33,25 +33,26 @@
 				</geometry>
 			</visual>
+			<!-- J1 arm: extends 0.375 m along X to joint_2 -->
 			<collision>
-				<origin rpy="0 0 0" xyz="0 0 0"/>
+				<origin rpy="0 0 0" xyz="0.187 0 0"/>
 				<geometry>
-					<mesh filename="file:///$(find denso_robot_descriptions)/robots/$(arg model)/meshes/J1.dae" scale="1 1 1"/>
+					<box size="0.375 0.080 0.060"/>
 				</geometry>
 			</collision>
 			<inertial>
 				<mass value="1"/>
-				<origin rpy="0.000000 0.000000 0.000000" xyz="0.000000 0.000000 0.000000"/>
+				<origin rpy="0 0 0" xyz="0 0 0"/>
 				<inertia ixx="1" ixy="0" ixz="0" iyy="1" iyz="0" izz="1"/>
 			</inertial>
 		</link>
-		<joint name="$(arg namespace)joint_1" type="revolute">
-			<parent link="$(arg namespace)base_link"/>
-			<child link="$(arg namespace)J1"/>
-			<origin rpy="0.000000 0.000000 0.000000" xyz="0.000000 0.000000 0.000000"/>
-			<axis xyz="-0.000000 -0.000000 1.000000"/>
+		<joint name="${namespace}joint_1" type="revolute">
+			<parent link="${namespace}base_link"/>
+			<child link="${namespace}J1"/>
+			<origin rpy="0 0 0" xyz="0 0 0"/>
+			<axis xyz="0 0 1"/>
 			<limit effort="1" lower="-2.26892802759263" upper="2.26892802759263" velocity="3.08615226990019"/>
 			<dynamics damping="0" friction="0"/>
 		</joint>
-		<link name="$(arg namespace)J2">
+		<link name="${namespace}J2">
 			<visual>
 				<origin rpy="0 0 0" xyz="0 0 0"/>
@@ -60,25 +61,26 @@
 				</geometry>
 			</visual>
+			<!-- J2 arm: goes -0.375 m back along X then 0.650 m forward to joint_4 -->
 			<collision>
-				<origin rpy="0 0 0" xyz="0 0 0"/>
+				<origin rpy="0 0 0" xyz="0.138 0 0"/>
 				<geometry>
-					<mesh filename="file:///$(find denso_robot_descriptions)/robots/$(arg model)/meshes/J2.dae" scale="1 1 1"/>
+					<box size="0.375 0.080 0.060"/>
 				</geometry>
 			</collision>
 			<inertial>
 				<mass value="1"/>
-				<origin rpy="0.000000 0.000000 0.000000" xyz="0.000000 0.000000 0.000000"/>
+				<origin rpy="0 0 0" xyz="0 0 0"/>
 				<inertia ixx="1" ixy="0" ixz="0" iyy="1" iyz="0" izz="1"/>
 			</inertial>
 		</link>
-		<joint name="$(arg namespace)joint_2" type="revolute">
-			<parent link="$(arg namespace)J1"/>
-			<child link="$(arg namespace)J2"/>
-			<origin rpy="0.000000 0.000000 0.000000" xyz="0.375000 0.000000 0.000000"/>
-			<axis xyz="-0.000000 -0.000000 1.000000"/>
+		<joint name="${namespace}joint_2" type="revolute">
+			<parent link="${namespace}J1"/>
+			<child link="${namespace}J2"/>
+			<origin rpy="0 0 0" xyz="0.375000 0 0"/>
+			<axis xyz="0 0 1"/>
 			<limit effort="1" lower="-2.61799387799149" upper="2.61799387799149" velocity="5.41357500737341"/>
 			<dynamics damping="0" friction="0"/>
 		</joint>
-		<link name="$(arg namespace)J3">
+		<link name="${namespace}J3">
 			<visual>
 				<origin rpy="0 0 0" xyz="0 0 0"/>
@@ -87,25 +89,26 @@
 				</geometry>
 			</visual>
+			<!-- J3 prismatic: travels 0.32 m along Z -->
 			<collision>
-				<origin rpy="0 0 0" xyz="0 0 0"/>
+				<origin rpy="0 0 0" xyz="0 0 0.060"/>
 				<geometry>
-					<mesh filename="file:///$(find denso_robot_descriptions)/robots/$(arg model)/meshes/J3.dae" scale="1 1 1"/>
+					<cylinder radius="0.030" length="0.320"/>
 				</geometry>
 			</collision>
 			<inertial>
 				<mass value="1"/>
-				<origin rpy="0.000000 0.000000 0.000000" xyz="0.000000 0.000000 0.000000"/>
+				<origin rpy="0 0 0" xyz="0 0 0"/>
 				<inertia ixx="1" ixy="0" ixz="0" iyy="1" iyz="0" izz="1"/>
 			</inertial>
 		</link>
-		<joint name="$(arg namespace)joint_3" type="prismatic">
-			<parent link="$(arg namespace)J2"/>
-			<child link="$(arg namespace)J3"/>
-			<origin rpy="0.000000 0.000000 0.000000" xyz="-0.375000 0.000000 0.000000"/>
-			<axis xyz="0.000000 0.000000 1.000000"/>
+		<joint name="${namespace}joint_3" type="prismatic">
+			<parent link="${namespace}J2"/>
+			<child link="${namespace}J3"/>
+			<origin rpy="0 0 0" xyz="-0.375000 0 0"/>
+			<axis xyz="0 0 1"/>
 			<limit effort="1" lower="-0.1" upper="0.22" velocity="1.9"/>
 			<dynamics damping="0" friction="0"/>
 		</joint>
-		<link name="$(arg namespace)J4">
+		<link name="${namespace}J4">
 			<visual>
 				<origin rpy="0 0 0" xyz="0 0 0"/>
@@ -114,21 +117,22 @@
 				</geometry>
 			</visual>
+			<!-- J4: end-effector / tool attachment -->
 			<collision>
 				<origin rpy="0 0 0" xyz="0 0 0"/>
 				<geometry>
-					<mesh filename="file:///$(find denso_robot_descriptions)/robots/$(arg model)/meshes/J4.dae" scale="1 1 1"/>
+					<cylinder radius="0.040" length="0.060"/>
 				</geometry>
 			</collision>
 			<inertial>
 				<mass value="1"/>
-				<origin rpy="0.000000 0.000000 0.000000" xyz="0.000000 0.000000 0.000000"/>
+				<origin rpy="0 0 0" xyz="0 0 0"/>
 				<inertia ixx="1" ixy="0" ixz="0" iyy="1" iyz="0" izz="1"/>
 			</inertial>
 		</link>
-		<joint name="$(arg namespace)joint_4" type="revolute">
-			<parent link="$(arg namespace)J3"/>
-			<child link="$(arg namespace)J4"/>
-			<origin rpy="0.000000 0.000000 0.000000" xyz="0.650000 0.000000 0.000000"/>
-			<axis xyz="-0.000000 -0.000000 1.000000"/>
+		<joint name="${namespace}joint_4" type="revolute">
+			<parent link="${namespace}J3"/>
+			<child link="${namespace}J4"/>
+			<origin rpy="0 0 0" xyz="0.650000 0 0"/>
+			<axis xyz="0 0 1"/>
 			<limit effort="1" lower="-6.28318530717959" upper="6.28318530717959" velocity="25.2968981715147"/>
 			<dynamics damping="0" friction="0"/>

File: denso_robot_descriptions/robots/hsr065a1_n32/urdf/denso_robot_macro.xacro (robot description, xacro)
@@ -12,11 +12,13 @@
     model
     namespace
+    parent
+    *origin
     transmission_hw_interface:=hardware_interface/PositionJointInterface
     sim:=false
+    gz_cam:=false
     ip_address
     send_format
     recv_format
-    verbose:=false"
-  >
+    verbose:=false">
     <!-- Robot data required by the denso driver -->
     <xacro:arg name="ip_address" default="192.168.0.1"/>
@@ -37,10 +39,17 @@
     <!-- ros2 control include -->
     <xacro:include filename="$(find denso_robot_descriptions)/robots/$(arg model)/urdf/denso_robot.ros2_control.xacro" />
+    <!-- For other tools, modify the filename parameter to the path of your tool's xacro file. -->
+    <!-- The line with tag xacro:tool passes the parameters defined in your tool's xacro file -->
+    <!-- (see gz_cam.xacro as an example implementation) -->
+    <xacro:if value="$(arg gz_cam)">
+      <xacro:include filename="$(find denso_robot_gazebo)/sensors/gz_cam/urdf/gz_cam.xacro" />
+    </xacro:if>
     <!-- ros2 control instance -->
     <xacro:denso_robot_ros2_control
-      name="GazeboSystem" namespace="$(arg namespace)"
+      name="HSR065A1_N32"
+      namespace="${namespace}"
       sim="$(arg sim)"
       model="$(arg model)"
-      ip_address="$(arg ip_address)"
+      ip_address="${ip_address}"
       robot_name="$(arg robot_name)"
       robot_joints="$(arg robot_joints)"
@@ -54,15 +63,14 @@
       send_format="$(arg send_format)"
       recv_format="$(arg recv_format)" />
-      <!-- node_name="$(arg node_name)" -->
     <!-- Add URDF transmission elements (for ros_control) -->
-    <xacro:denso_robot_arm_transmission namespace="$(arg namespace)" hw_interface="$(arg transmission_hw_interface)" />
+    <xacro:denso_robot_arm_transmission namespace="${namespace}" hw_interface="$(arg transmission_hw_interface)" />
     <!-- Placeholder for ros2_control transmission which don't yet exist -->
-    <!-- links -  main serial chain -->
-    <xacro:denso_robot_arm_kinematics namespace="$(arg namespace)" model="$(arg model)" />
-    <gazebo>
-	    <plugin filename="gz_ros2_control-system" name="gz_ros2_control::GazeboSimROS2ControlPlugin">
-      		<parameters>$(find denso_robot_moveit_config)/robots/$(arg model)/config/denso_robot_controllers.yaml</parameters>
-    	</plugin>
-  	</gazebo>
+    <!-- links - main serial chain -->
+    <xacro:denso_robot_arm_kinematics namespace="${namespace}" model="$(arg model)" parent="${parent}">
+      <xacro:insert_block name="origin" />
+    </xacro:denso_robot_arm_kinematics>
+    <xacro:if value="$(arg gz_cam)">
+      <xacro:gz_cam namespace="${namespace}" />
+    </xacro:if>
   </xacro:macro>
 </robot>

File: denso_robot_moveit_config/robots/hsr065a1_n32/srdf/denso_robot_macro.srdf.xacro (robot description, xacro)
@@ -5,5 +5,5 @@
     A URDF file must exist for this robot as well, where the joints and the links that are referenced are defined
 -->
-  <xacro:macro name="denso_robot_srdf" params="name namespace">
+  <xacro:macro name="denso_robot_srdf" params="namespace">
     <!--GROUPS - Representation of a set of joints and links. This can be useful for specifying DOF to plan for, defining arms, end effectors, etc-->
     <!--LINKS - When a link is specified, the parent joint of that link (if it exists) is automatically included-->
@@ -12,9 +12,9 @@
     <!--SUBGROUPS - Groups can also be formed by referencing to already defined group names-->
     <group name="${namespace}arm">
-		<joint name="$(arg namespace)joint_1"/>
-		<joint name="$(arg namespace)joint_2"/>
-		<joint name="$(arg namespace)joint_3"/>
-		<joint name="$(arg namespace)joint_4"/>
-	</group>
+      <joint name="${namespace}joint_1"/>
+      <joint name="${namespace}joint_2"/>
+      <joint name="${namespace}joint_3"/>
+      <joint name="${namespace}joint_4"/>
+    </group>
     <!--GROUP STATES - Purpose - Define a named state for a particular group, in terms of joint values. This is useful to define states like 'folded arms'-->
     <!--END EFFECTOR - Purpose - Represent information about an end effector.-->
@@ -22,13 +22,13 @@
     <virtual_joint name="${namespace}fixed_base" type="fixed" parent_frame="world" child_link="${namespace}base_link" />
     <!--DISABLE COLLISIONS - By default it is assumed that any link of the robot could potentially come into collision with any other link in the robot. This tag disables collision checking between a specified pair of links. -->
-	<disable_collisions link1="$(arg namespace)J1" link2="$(arg namespace)J2" reason="Adjacent"/>
-	<disable_collisions link1="$(arg namespace)J1" link2="$(arg namespace)J3" reason="Never"/>
-	<disable_collisions link1="$(arg namespace)J1" link2="$(arg namespace)J4" reason="Never"/>
-	<disable_collisions link1="$(arg namespace)J1" link2="$(arg namespace)base_link" reason="Adjacent"/>
-	<disable_collisions link1="$(arg namespace)J2" link2="$(arg namespace)J3" reason="Adjacent"/>
-	<disable_collisions link1="$(arg namespace)J2" link2="$(arg namespace)J4" reason="Never"/>
-	<disable_collisions link1="$(arg namespace)J2" link2="$(arg namespace)base_link" reason="Never"/>
-	<disable_collisions link1="$(arg namespace)J3" link2="$(arg namespace)J4" reason="Adjacent"/>
-	<disable_collisions link1="$(arg namespace)J4" link2="$(arg namespace)base_link" reason="Never"/>
+    <disable_collisions link1="${namespace}J1" link2="${namespace}J2" reason="Adjacent"/>
+    <disable_collisions link1="${namespace}J1" link2="${namespace}J3" reason="Never"/>
+    <disable_collisions link1="${namespace}J1" link2="${namespace}J4" reason="Never"/>
+    <disable_collisions link1="${namespace}J1" link2="${namespace}base_link" reason="Adjacent"/>
+    <disable_collisions link1="${namespace}J2" link2="${namespace}J3" reason="Adjacent"/>
+    <disable_collisions link1="${namespace}J2" link2="${namespace}J4" reason="Never"/>
+    <disable_collisions link1="${namespace}J2" link2="${namespace}base_link" reason="Never"/>
+    <disable_collisions link1="${namespace}J3" link2="${namespace}J4" reason="Adjacent"/>
+    <disable_collisions link1="${namespace}J4" link2="${namespace}base_link" reason="Never"/>
   </xacro:macro>
 </robot>
